Commit message: Added joints and links

File: cogimon_urdf/urdf/gazebo/cogimon_materials.gazebo.xacro (robot description, xacro)
@@ -8,4 +8,7 @@
   <material>Gazebo/Green</material>
 </gazebo>
+<gazebo reference="RThighUpLeg">
+  <material>Gazebo/DarkGrey</material>
+</gazebo>
 </xacro:if>
 <xacro:if value="${COGIMON_LEFT_LEG}" >
@@ -13,4 +16,7 @@
   <material>Gazebo/Green</material>
 </gazebo>
+<gazebo reference="LThighUpLeg">
+  <material>Gazebo/DarkGrey</material>
+</gazebo>
 </xacro:if>
 </robot>

File: cogimon_urdf/urdf/parts/legs.urdf.xacro (robot description, xacro)
@@ -23,4 +23,24 @@
     </collision>
   </link>
+<link name ="LThighUpLeg">
+    <inertial>
+      <origin xyz="${5.8688639e-01*mmTom} ${-6.2440385e+01*mmTom} ${-8.5057072e+01*mmTom}" rpy="0 0 0"/>
+      <mass value="1.6115687"/>
+      <inertia ixx="${1.6169151e+04*mm2Tom2}"  ixy="${-2.1886129e+01*mm2Tom2}"  ixz="${6.0058109e+01*mm2Tom2}" iyy="${1.4437800e+04*mm2Tom2}" iyz="${-2.7173225e+03*mm2Tom2}" izz="${3.9254506e+03*mm2Tom2}" />
+    </inertial>
+    <visual>
+      <origin xyz="0. 0. 0." rpy="0 0 0."/>
+      <material name="dark_grey"/>
+      <geometry name="LThighUpLeg_visual">
+        <mesh filename="package://cogimon_urdf/meshes/HipPitch.stl" scale="${mmTom} ${mmTom} ${mmTom}" />
+      </geometry>
+    </visual>
+    <collision>
+      <origin xyz="0.0 0. 0" rpy="0 0 0."/>
+      <geometry name="LThighUpLeg_collision">
+        <mesh filename="package://cogimon_urdf/meshes/simple/HipPitch.stl" scale="${mmTom} ${mmTom} ${mmTom}" />
+      </geometry>
+    </collision>
+  </link>
 <!-- JOINTS -->
 <joint name="LHipLat" type="revolute">
@@ -29,4 +49,12 @@
     <origin xyz="${15.45*mmTom} ${112.0*mmTom} ${-50.0*mmTom}" rpy="0 0 0" />
     <axis xyz="1 0 0" />
+    <limit velocity="3.67" effort="176" lower="${-90.*toRad}" upper="${90.*toRad}" />
+    <dynamics friction="0" damping="3.0"/>
+</joint>
+<joint name="LHipSag" type="revolute">
+    <parent link="LHipMot"/>
+    <child link="LThighUpLeg"/>
+    <origin xyz="${-59.*mmTom} ${78.65*mmTom} ${-118.5*mmTom}" rpy="0 0 0" />
+    <axis xyz="0 1 0" />
     <limit velocity="3.67" effort="176" lower="${-90.*toRad}" upper="${90.*toRad}" />
     <dynamics friction="0" damping="3.0"/>
@@ -55,4 +83,24 @@
     </collision>
 </link>
+<link name ="RThighUpLeg">
+    <inertial>
+      <origin xyz="${5.8688639e-01*mmTom} ${6.2440385e+01*mmTom} ${-8.5057072e+01*mmTom}" rpy="0 0 0"/>
+      <mass value="1.6115687"/>
+      <inertia ixx="${1.6169151e+04*mm2Tom2}"  ixy="${2.1886129e+01*mm2Tom2}"  ixz="${6.0058109e+01*mm2Tom2}" iyy="${1.4437800e+04*mm2Tom2}" iyz="${2.7173225e+03*mm2Tom2}" izz="${3.9254506e+03*mm2Tom2}" />
+    </inertial>
+    <visual>
+      <origin xyz="0. 0. 0." rpy="0 0 0."/>
+      <material name="dark_grey"/>
+      <geometry name="RThighUpLeg_visual">
+        <mesh filename="package://cogimon_urdf/meshes/HipPitch.stl" scale="${mmTom} ${-mmTom} ${mmTom}" />
+      </geometry>
+    </visual>
+    <collision>
+      <origin xyz="0.0 0. 0" rpy="0 0 0."/>
+      <geometry name="RThighUpLeg_collision">
+        <mesh filename="package://cogimon_urdf/meshes/simple/HipPitch.stl" scale="${mmTom} ${-mmTom} ${mmTom}" />
+      </geometry>
+    </collision>
+  </link>
 <!-- JOINTS -->
 <joint name="RHipLat" type="revolute">
@@ -64,4 +112,12 @@
     <dynamics friction="0" damping="3.0"/>
 </joint>
+<joint name="RHipSag" type="revolute">
+    <parent link="RHipMot"/>
+    <child link="RThighUpLeg"/>
+    <origin xyz="${-59.*mmTom} ${-78.65*mmTom} ${-118.5*mmTom}" rpy="0 0 0" />
+    <axis xyz="0 1 0" />
+    <limit velocity="3.67" effort="176" lower="${-90.*toRad}" upper="${90.*toRad}" />
+    <dynamics friction="0" damping="3.0"/>
+</joint>
 </xacro:if>
 </robot>

Commit message: Added new joints and links

File: cogimon_urdf/urdf/gazebo/cogimon_materials.gazebo.xacro (robot description, xacro)
@@ -11,4 +11,7 @@
   <material>Gazebo/DarkGrey</material>
 </gazebo>
+<gazebo reference="RThighLowLeg">
+  <material>Gazebo/Green</material>
+</gazebo>
 </xacro:if>
 <xacro:if value="${COGIMON_LEFT_LEG}" >
@@ -19,4 +22,7 @@
   <material>Gazebo/DarkGrey</material>
 </gazebo>
+<gazebo reference="LThighLowLeg">
+  <material>Gazebo/Green</material>
+</gazebo>
 </xacro:if>
 </robot>

File: cogimon_urdf/urdf/parts/legs.urdf.xacro (robot description, xacro)
@@ -22,5 +22,5 @@
       </geometry>
     </collision>
-  </link>
+</link>
 <link name ="LThighUpLeg">
     <inertial>
@@ -42,5 +42,25 @@
       </geometry>
     </collision>
-  </link>
+</link>
+<link name ="LThighLowLeg">
+    <inertial>
+      <origin xyz="${-2.1136410e+01*mmTom} ${-4.2862386e+00*mmTom} ${-3.8232267e+01*mmTom}" rpy="0 0 0"/>
+      <mass value="1.7454681"/>
+      <inertia ixx="${8.5691728e+03*mm2Tom2}"  ixy="${-1.9828734e+02*mm2Tom2}"  ixz="${-2.2121863e+03*mm2Tom2}" iyy="${9.9794948e+03*mm2Tom2}" iyz="${-4.0039407e+02*mm2Tom2}" izz="${5.2783547e+03*mm2Tom2}" />
+    </inertial>
+    <visual>
+      <origin xyz="0. 0. 0." rpy="0 0 0."/>
+      <material name="green"/>
+      <geometry name="LThighLowLeg_visual">
+        <mesh filename="package://cogimon_urdf/meshes/HipYaw.stl" scale="${mmTom} ${mmTom} ${mmTom}" />
+      </geometry>
+    </visual>
+    <collision>
+      <origin xyz="0.0 0. 0" rpy="0 0 0."/>
+      <geometry name="LThighLowLeg_collision">
+        <mesh filename="package://cogimon_urdf/meshes/simple/HipYaw.stl" scale="${mmTom} ${mmTom} ${mmTom}" />
+      </geometry>
+    </collision>
+</link>
 <!-- JOINTS -->
 <joint name="LHipLat" type="revolute">
@@ -57,4 +77,12 @@
     <origin xyz="${-59.*mmTom} ${78.65*mmTom} ${-118.5*mmTom}" rpy="0 0 0" />
     <axis xyz="0 1 0" />
+    <limit velocity="3.67" effort="176" lower="${-90.*toRad}" upper="${90.*toRad}" />
+    <dynamics friction="0" damping="3.0"/>
+</joint>
+<joint name="LHipYaw" type="revolute">
+    <parent link="LThighUpLeg"/>
+    <child link="LThighLowLeg"/>
+    <origin xyz="${0.*mmTom} ${-90.*mmTom} ${-256.45*mmTom}" rpy="0 0 0" />
+    <axis xyz="0 0 1" />
     <limit velocity="3.67" effort="176" lower="${-90.*toRad}" upper="${90.*toRad}" />
     <dynamics friction="0" damping="3.0"/>
@@ -103,4 +131,24 @@
     </collision>
   </link>
+<link name ="RThighLowLeg">
+    <inertial>
+      <origin xyz="${-2.1136410e+01*mmTom} ${4.2862386e+00*mmTom} ${-3.8232267e+01*mmTom}" rpy="0 0 0"/>
+      <mass value="1.7454681"/>
+      <inertia ixx="${8.5691728e+03*mm2Tom2}"  ixy="${1.9828734e+02*mm2Tom2}"  ixz="${-2.2121863e+03*mm2Tom2}" iyy="${9.9794948e+03*mm2Tom2}" iyz="${4.0039407e+02*mm2Tom2}" izz="${5.2783547e+03*mm2Tom2}" />
+    </inertial>
+    <visual>
+      <origin xyz="0. 0. 0." rpy="0 0 0."/>
+      <material name="green"/>
+      <geometry name="RThighLowLeg_visual">
+        <mesh filename="package://cogimon_urdf/meshes/HipYaw.stl" scale="${mmTom} ${-mmTom} ${mmTom}" />
+      </geometry>
+    </visual>
+    <collision>
+      <origin xyz="0.0 0. 0" rpy="0 0 0."/>
+      <geometry name="RThighLowLeg_collision">
+        <mesh filename="package://cogimon_urdf/meshes/simple/HipYaw.stl" scale="${mmTom} ${-mmTom} ${mmTom}" />
+      </geometry>
+    </collision>
+</link>
 <!-- JOINTS -->
 <joint name="RHipLat" type="revolute">
@@ -120,4 +168,12 @@
     <dynamics friction="0" damping="3.0"/>
 </joint>
+<joint name="RHipYaw" type="revolute">
+    <parent link="RThighUpLeg"/>
+    <child link="RThighLowLeg"/>
+    <origin xyz="${0.*mmTom} ${90.*mmTom} ${-256.45*mmTom}" rpy="0 0 0" />
+    <axis xyz="0 0 1" />
+    <limit velocity="3.67" effort="176" lower="${-90.*toRad}" upper="${90.*toRad}" />
+    <dynamics friction="0" damping="3.0"/>
+</joint>
 </xacro:if>
 </robot>

Commit message: Added joints and links

File: cogimon_urdf/urdf/gazebo/cogimon_materials.gazebo.xacro (robot description, xacro)
@@ -17,4 +17,7 @@
   <material>Gazebo/DarkGrey</material>
 </gazebo>
+<gazebo reference="RFootmot">
+  <material>Gazebo/DarkGrey</material>
+</gazebo>
 </xacro:if>
 <xacro:if value="${COGIMON_LEFT_LEG}" >
@@ -31,4 +34,7 @@
   <material>Gazebo/DarkGrey</material>
 </gazebo>
+<gazebo reference="LFootmot">
+  <material>Gazebo/DarkGrey</material>
+</gazebo>
 </xacro:if>
 </robot>

File: cogimon_urdf/urdf/parts/legs.urdf.xacro (robot description, xacro)
@@ -7,5 +7,5 @@
       <origin xyz="${-4.1435899e+01*mmTom} ${-2.4099021e-01*mmTom} ${-6.7437774e+01*mmTom}" rpy="0 0 0"/>
       <mass value="2.0936467"/>
-      <inertia ixx="${2.0328644e+04*mm2Tom2}"  ixy="${1.2836757e+01*mm2Tom2}"  ixz="${-7.1832791e+03*mm2Tom2}" iyy="${2.4404941e+04*mm2Tom2}" iyz="${2.2892687e+01*mm2Tom2}" izz="${8.9864540e+03*mm2Tom2}" />
+      <inertia ixx="${1.0806924e+04*mm2Tom2}"  ixy="${3.3743172e+01*mm2Tom2}"  ixz="${-1.3329083e+03*mm2Tom2}" iyy="${1.1288691e+04*mm2Tom2}" iyz="${5.6918305e+01*mm2Tom2}" izz="${5.3916798e+03*mm2Tom2}" />
     </inertial>
     <visual>
@@ -47,5 +47,5 @@
       <origin xyz="${-2.1136410e+01*mmTom} ${-4.2862386e+00*mmTom} ${-3.8232267e+01*mmTom}" rpy="0 0 0"/>
       <mass value="1.7454681"/>
-      <inertia ixx="${8.5691728e+03*mm2Tom2}"  ixy="${-1.9828734e+02*mm2Tom2}"  ixz="${-2.2121863e+03*mm2Tom2}" iyy="${9.9794948e+03*mm2Tom2}" iyz="${-4.0039407e+02*mm2Tom2}" izz="${5.2783547e+03*mm2Tom2}" />
+      <inertia ixx="${5.9857438e+03*mm2Tom2}"  ixy="${-4.0155441e+01*mm2Tom2}"  ixz="${-8.0168603e+02*mm2Tom2}" iyy="${6.6483492e+03*mm2Tom2}" iyz="${-1.1435964e+02*mm2Tom2}" izz="${4.4665032e+03*mm2Tom2}" />
     </inertial>
     <visual>
@@ -80,4 +80,24 @@
       <geometry name="LLowLeg_collision">
         <mesh filename="package://cogimon_urdf/meshes/simple/KneePitch.stl" scale="${mmTom} ${mmTom} ${mmTom}" />
+      </geometry>
+    </collision>
+</link>
+<link name ="LFootmot">
+    <inertial>
+      <origin xyz="${1.1213007e+00*mmTom} ${4.6152281e-01*mmTom} ${-1.1449670e-03*mmTom}" rpy="0 0 0"/>
+      <mass value="1.7723821e-01"/>
+      <inertia ixx="${2.8142035e+01*mm2Tom2}"  ixy="${9.1715528e-02*mm2Tom2}"  ixz="${-2.1701012e-04*mm2Tom2}" iyy="${9.7378402e+01*mm2Tom2}" iyz="${3.7303915e-04*mm2Tom2}" izz="${1.1570584e+02*mm2Tom2}" />
+    </inertial>
+    <visual>
+      <origin xyz="0 0 0" rpy="0 0 0"/>
+      <geometry name="LFootmot_visual">
+        <mesh filename="package://cogimon_urdf/meshes/AnklePitch.stl" scale="${mmTom} ${mmTom} ${mmTom}" />
+      </geometry>
+      <material name="dark_grey"/>
+    </visual>
+    <collision>
+      <origin xyz="0 0 0" rpy="0 0 0"/>
+      <geometry name="LFootmot_collision">
+        <mesh filename="package://cogimon_urdf/meshes/simple/AnklePitch.stl" scale="${mmTom} ${mmTom} ${mmTom}" />
       </geometry>
     </collision>
@@ -116,4 +136,12 @@
     <dynamics friction="0" damping="3.0"/>
 </joint>
+<joint name="LAnklePitch" type="revolute">
+    <parent link="LLowLeg"/>
+    <child link="LFootmot"/>
+    <origin xyz="${39.*mmTom} ${-61.6*mmTom} ${-425.294*mmTom}" rpy="0 0 0" />
+    <axis xyz="0 1 0" />
+    <limit velocity="3.67" effort="176" lower="${-90.*toRad}" upper="${90.*toRad}" />
+    <dynamics friction="0" damping="0.1"/>
+</joint>
 </xacro:if>
 <xacro:if value="${COGIMON_RIGHT_LEG}" >
@@ -123,5 +151,5 @@
       <origin xyz="${-4.1435899e+01*mmTom} ${2.4099021e-01*mmTom} ${-6.7437774e+01*mmTom}" rpy="0 0 0"/>
       <mass value="2.0936467"/>
-      <inertia ixx="${2.0328644e+04*mm2Tom2}"  ixy="${-1.2836757e+01*mm2Tom2}"  ixz="${-7.1832791e+03*mm2Tom2}" iyy="${2.4404941e+04*mm2Tom2}" iyz="${-2.2892687e+01*mm2Tom2}" izz="${8.9864540e+03*mm2Tom2}" />
+      <inertia ixx="${1.0806924e+04*mm2Tom2}"  ixy="${-3.3743172e+01*mm2Tom2}"  ixz="${-1.3329083e+03*mm2Tom2}" iyy="${1.1288691e+04*mm2Tom2}" iyz="${-5.6918305e+01*mm2Tom2}" izz="${5.3916798e+03*mm2Tom2}" />
     </inertial>
     <visual>
@@ -163,5 +191,5 @@
       <origin xyz="${-2.1136410e+01*mmTom} ${4.2862386e+00*mmTom} ${-3.8232267e+01*mmTom}" rpy="0 0 0"/>
       <mass value="1.7454681"/>
-      <inertia ixx="${8.5691728e+03*mm2Tom2}"  ixy="${1.9828734e+02*mm2Tom2}"  ixz="${-2.2121863e+03*mm2Tom2}" iyy="${9.9794948e+03*mm2Tom2}" iyz="${4.0039407e+02*mm2Tom2}" izz="${5.2783547e+03*mm2Tom2}" />
+      <inertia ixx="${5.9857438e+03*mm2Tom2}"  ixy="${4.0155441e+01*mm2Tom2}"  ixz="${-8.0168603e+02*mm2Tom2}" iyy="${6.6483492e+03*mm2Tom2}" iyz="${1.1435964e+02*mm2Tom2}" izz="${4.4665032e+03*mm2Tom2}" />
     </inertial>
     <visual>
@@ -196,4 +224,24 @@
       <geometry name="RLowLeg_collision">
         <mesh filename="package://cogimon_urdf/meshes/simple/KneePitch.stl" scale="${mmTom} ${-mmTom} ${mmTom}" />
+      </geometry>
+    </collision>
+</link>
+<link name ="RFootmot">
+    <inertial>
+      <origin xyz="${1.1213007e+00*mmTom} ${4.6152281e-01*mmTom} ${-1.1449670e-03*mmTom}" rpy="0 0 0"/>
+      <mass value="1.7723821e-01"/>
+      <inertia ixx="${2.8142035e+01*mm2Tom2}"  ixy="${9.1715528e-02*mm2Tom2}"  ixz="${-2.1701012e-04*mm2Tom2}" iyy="${9.7378402e+01*mm2Tom2}" iyz="${3.7303915e-04*mm2Tom2}" izz="${1.1570584e+02*mm2Tom2}" />
+    </inertial>
+    <visual>
+      <origin xyz="0 0 0" rpy="0 0 0"/>
+      <geometry name="RFootmot_visual">
+        <mesh filename="package://cogimon_urdf/meshes/AnklePitch.stl" scale="${mmTom} ${mmTom} ${mmTom}" />
+      </geometry>
+      <material name="dark_grey"/>
+    </visual>
+    <collision>
+      <origin xyz="0 0 0" rpy="0 0 0"/>
+      <geometry name="RFootmot_collision">
+        <mesh filename="package://cogimon_urdf/meshes/simple/AnklePitch.stl" scale="${mmTom} ${mmTom} ${mmTom}" />
       </geometry>
     </collision>
@@ -232,4 +280,12 @@
     <dynamics friction="0" damping="3.0"/>
 </joint>
+<joint name="RAnklePitch" type="revolute">
+    <parent link="RLowLeg"/>
+    <child link="RFootmot"/>
+    <origin xyz="${39.*mmTom} ${61.6*mmTom} ${-425.294*mmTom}" rpy="0 0 0" />
+    <axis xyz="0 1 0" />
+    <limit velocity="3.67" effort="176" lower="${-90.*toRad}" upper="${90.*toRad}" />
+    <dynamics friction="0" damping="0.1"/>
+</joint>
 </xacro:if>
 </robot>
