Commit message: fixed script to be updated with last version of xacro. Removed some useless definition in xacro files

File: cogimon_urdf/urdf/gazebo/force_torque.gazebo.xacro (robot description, xacro)
@@ -6,5 +6,5 @@
 and we will add a revolute joint between foot_flange and sensor and a fixed joint (where we will measure the wrench) between sensor and sole.
 -->
-<robot xmlns:xacro="http:/ros.org/wiki/xacro">
+<robot xmlns:xacro="http://ros.org/wiki/xacro">
 <xacro:if value="${COGIMON_LEFT_ARM}" >
        <gazebo reference="LWrMot3">

File: cogimon_urdf/urdf/gazebo/imu.gazebo.xacro (robot description, xacro)
@@ -3,5 +3,5 @@
 This IMU does not exist in the actual robot
 -->
-<robot xmlns:xacro="http:/ros.org/wiki/xacro">
+<robot xmlns:xacro="http://ros.org/wiki/xacro">
 <gazebo reference="imu_link">
     <sensor name="imu_link" type="imu">

File: cogimon_urdf/urdf/parts/arms.urdf.xacro (robot description, xacro)
@@ -1,8 +1,7 @@
 <?xml version="1.0"?>
 <robot xmlns:xacro="http://ros.org/wiki/xacro">
-<xacro:property name="PI" value="3.14159265359" />
+<!--xacro:property name="PI" value="3.14159265359" />
 <xacro:property name="mmTom" value="0.001" />
-<xacro:property name="mm2Tom2" value="${0.001*0.001}" />
-<xacro:property name="DEG2RAD" value="${PI/180.}" />
+<xacro:property name="mm2Tom2" value="${0.001*0.001}" /-->
 <xacro:if value="${COGIMON_RIGHT_ARM}">
 <!-- RIGHT ARM -->

File: cogimon_urdf/urdf/parts/soft_hands.urdf.xacro (robot description, xacro)
@@ -1,6 +1,6 @@
 <?xml version="1.0"?>
 <robot xmlns:xacro="http://ros.org/wiki/xacro" name="SoftHand">
-<xacro:property name="PI" value="3.14159265359" />
-<xacro:property name="PI_2" value="1.57079632679" />
+<!--xacro:property name="PI" value="3.14159265359" />
+<xacro:property name="PI_2" value="1.57079632679" /-->
 <xacro:if value="${COGIMON_RIGHT_ARM}">
 <!-- LINKS -->
