Commit message: added link state sensor

File: cogimon_urdf/urdf/gazebo/xbot_control.gazebo.xacro (robot description, xacro)
@@ -2,4 +2,9 @@
 <robot xmlns:xacro="http://ros.org/wiki/xacro">
 <gazebo>
+    <plugin name="xbot2_link_state_sensor" filename="libxbot2_gz_link_state_sensor.so">
+        <links>
+            <link name="base_link"/>
+        </links>
+    </plugin>
     <plugin name="xbot2_gz_ft_server" filename="libxbot2_gz_ft_server.so"/>
     <plugin name="xbot2_gz_imu_server" filename="libxbot2_gz_imu_server.so"/>
