Commit message: Changed lenghts in legs and torso

File: cogimon_urdf/urdf/parts/legs.urdf.xacro (robot description, xacro)
@@ -316,5 +316,5 @@
     <parent link="RThighUpLeg"/>
     <child link="RThighLowLeg"/>
-    <origin xyz="0.0 0.0 ${-0.1024-hco}" rpy="0 0 0" />
+    <origin xyz="0.0 0.0 ${-0.1024-hco-0.025}" rpy="0 0 0" />
     <axis xyz="0 0 1" />
     <limit velocity="4.0" effort="80" lower="-0.8727" upper="0.8727" />
@@ -332,5 +332,5 @@
     <parent link="RLowLeg"/>
     <child link="RFootmot"/>
-    <origin xyz="0.0 0.0 ${-0.201-hco}" rpy="0 0 0" />
+    <origin xyz="0.0 0.0 ${-0.201-hco-0.025}" rpy="0 0 0" />
     <axis xyz="1 0 0" />
     <limit velocity="4.0" effort="80" lower="-0.6109" upper="0.6109" />
@@ -365,5 +365,5 @@
     <parent link="LThighUpLeg"/>
     <child link="LThighLowLeg"/>
-    <origin xyz="0.0 0.0 ${-0.1024-hco}" rpy="0 0 0" />
+    <origin xyz="0.0 0.0 ${-0.1024-hco-0.025}" rpy="0 0 0" />
     <axis xyz="0 0 1" />
     <limit velocity="4.0" effort="80" lower="-0.8727" upper="0.8727" />
@@ -381,5 +381,5 @@
     <parent link="LLowLeg"/>
     <child link="LFootmot"/>
-    <origin xyz="0.0 0.0 ${-0.201-hco}" rpy="0 0 0" />
+    <origin xyz="0.0 0.0 ${-0.201-hco-0.025}" rpy="0 0 0" />
     <axis xyz="1 0 0" />
     <limit velocity="4.0" effort="80" lower="-0.6109" upper="0.6109" />

File: cogimon_urdf/urdf/parts/torso.urdf.xacro (robot description, xacro)
@@ -91,5 +91,5 @@
     <parent link="DWS"/>
     <child link="DWYTorso"/>
-    <origin xyz="0 0 ${0.04749999+hco}" rpy="0 0 0" />
+    <origin xyz="0 0 ${0.04749999+hco-0.05}" rpy="0 0 0" />
     <axis xyz="0 0 1" />
     <limit velocity="4.0" effort="40" lower="-1.3963" upper="1.3962" />

Commit message: Added left/right hip pitch

File: cogimon_urdf/urdf/parts/legs.urdf.xacro (robot description, xacro)
@@ -23,4 +23,24 @@
     </collision>
 </link>
+<link name ="RThighUpLeg">
+    <inertial>
+      <origin xyz="${2.9898120e-01*mmTom} ${6.5748642e+01*mmTom} ${-8.8443666e+01*mmTom}" rpy="0 0 0"/>
+      <mass value="1.9691802"/>
+      <inertia ixx="${1.6200713e+04*mm2Tom2}"  ixy="${1.9336329e+01*mm2Tom2}"  ixz="${-3.8620029e+01*mm2Tom2}" iyy="${1.4426424e+04*mm2Tom2}" iyz="${3.5985350e+03*mm2Tom2}" izz="${4.8264937e+03*mm2Tom2}" />
+    </inertial>
+    <visual>
+      <origin xyz="0.0 0 0" rpy="0 0 0"/>
+      <material name="dark_grey"/>
+      <geometry name="RThighUpLeg_visual">
+        <mesh filename="package://cogimon_urdf/meshes/Leg1.STL" scale="${mmTom} ${-mmTom} ${mmTom}" />
+      </geometry>
+    </visual>
+    <collision>
+      <origin xyz="0.0 0. 0." rpy="0 0 0"/>
+      <geometry name="RThighUpLeg_collision">
+        <mesh filename="package://cogimon_urdf/meshes/simple/Leg1.STL" scale="${mmTom} ${-mmTom} ${mmTom}" />
+      </geometry>
+    </collision>
+  </link>
 <!-- JOINTS -->
 <joint name="RHipLat" type="revolute">
@@ -32,4 +52,12 @@
     <dynamics friction="0" damping="3.0"/>
   </joint>
+<joint name="RHipSag" type="revolute">
+    <parent link="RHipMot"/>
+    <child link="RThighUpLeg"/>
+    <origin xyz="${-8.5*mmTom} ${-73.9855*mmTom} ${-112.5*mmTom}" rpy="0 0 0" />
+    <axis xyz="0 1 0" />
+    <limit velocity="3.67" effort="176" lower="${-96.*toRad}" upper="${90.*toRad}" />
+    <dynamics friction="0" damping="3.0"/>
+  </joint>
 </xacro:if>
 <xacro:if value="${COGIMON_LEFT_LEG}" >
@@ -52,4 +80,24 @@
       <geometry name="RHipMot_collision">
         <mesh filename="package://cogimon_urdf/meshes/simple/Leg0.STL" scale="${mmTom} ${mmTom} ${mmTom}" />
+      </geometry>
+    </collision>
+  </link>
+  <link name ="LThighUpLeg">
+    <inertial>
+      <origin xyz="${2.9898120e-01*mmTom} ${-6.5748642e+01*mmTom} ${-8.8443666e+01*mmTom}" rpy="0 0 0"/>
+      <mass value="1.9691802"/>
+      <inertia ixx="${1.6200713e+04*mm2Tom2}"  ixy="${-1.9336329e+01*mm2Tom2}"  ixz="${-3.8620029e+01*mm2Tom2}" iyy="${1.4426424e+04*mm2Tom2}" iyz="${-3.5985350e+03*mm2Tom2}" izz="${4.8264937e+03*mm2Tom2}" />
+    </inertial>
+    <visual>
+      <origin xyz="0.0 0 0" rpy="0 0 0"/>
+      <material name="dark_grey"/>
+      <geometry name="LThighUpLeg_visual">
+        <mesh filename="package://cogimon_urdf/meshes/Leg1.STL" scale="${mmTom} ${mmTom} ${mmTom}" />
+      </geometry>
+    </visual>
+    <collision>
+      <origin xyz="0.0 0. 0." rpy="0 0 0"/>
+      <geometry name="LThighUpLeg_collision">
+        <mesh filename="package://cogimon_urdf/meshes/simple/Leg1.STL" scale="${mmTom} ${mmTom} ${mmTom}" />
       </geometry>
     </collision>
@@ -62,4 +110,12 @@
     <axis xyz="1 0 0" />
     <limit velocity="3.67" effort="176" lower="${-25.*toRad}" upper="${85.*toRad}" />
+    <dynamics friction="0" damping="3.0"/>
+  </joint>
+<joint name="LHipSag" type="revolute">
+    <parent link="LHipMot"/>
+    <child link="LThighUpLeg"/>
+    <origin xyz="${-8.5*mmTom} ${73.9855*mmTom} ${-112.5*mmTom}" rpy="0 0 0" />
+    <axis xyz="0 1 0" />
+    <limit velocity="3.67" effort="176" lower="${-96.*toRad}" upper="${90.*toRad}" />
     <dynamics friction="0" damping="3.0"/>
   </joint>
@@ -195,44 +251,4 @@
 <!-- ********************LEFT LEG******************** -->
 <!--
-  <link name ="LHipMot">
-    <inertial>
-      <origin xyz="-3.269678E-4 0.023587321 -2.6496509E-4" rpy="0 0 0"/>
-      <mass value="${wcf*0.89258227}"/>
-      <inertia ixx="${wcf*4.7672294E-4}"  ixy="${wcf*3.9936567E-6}"  ixz="${wcf*-2.4802574E-6}" iyy="${wcf*5.458038E-4}" iyz="${wcf*3.3389575E-6}" izz="${wcf*5.126859E-4}" />
-    </inertial>
-    <visual>
-      <origin xyz="0.0 -0.023 -0.52" rpy="0 0 ${PI}"/>
-      <material name="dark_grey"/>
-      <geometry name="RHipMot_visual">
-        <mesh filename="package://cogimon_urdf/meshes/Leg0.STL" scale="${SF} -${SF} ${SF}" />
-      </geometry>
-    </visual>
-    <collision>
-      <origin xyz="0.0 -0.023 -0.52" rpy="0 0 ${PI}"/>
-      <geometry name="RHipMot_collision">
-        <mesh filename="package://cogimon_urdf/meshes/simple/Leg0.STL" scale="${SF} -${SF} ${SF}" />
-      </geometry>
-    </collision>
-  </link>
-  <link name ="LThighUpLeg">
-    <inertial>
-      <origin xyz="0.0012591632 0.016896372 -0.058903336" rpy="0 0 0"/>
-      <mass value="${wcf*1.0246101}"/>
-      <inertia ixx="${wcf*9.165719E-4}"  ixy="${wcf*1.4449904E-6}"  ixz="${wcf*-1.6685011E-5}" iyy="${wcf*0.00104849584}" iyz="${wcf*-2.5492874E-5}" izz="${wcf*6.8637197E-4}" />
-    </inertial>
-    <visual>
-      <origin xyz="0.0 -0.0726 -0.52" rpy="0 0 ${PI}"/>
-      <material name="dark_grey"/>
-      <geometry name="LThighUpLeg_visual">
-        <mesh filename="package://cogimon_urdf/meshes/Leg1.STL" scale="${SF} -${SF} ${SF}" />
-      </geometry>
-    </visual>
-    <collision>
-      <origin xyz="0.0 -0.0726 -0.52" rpy="0 0 ${PI}"/>
-      <geometry name="LThighUpLeg_collision">
-        <mesh filename="package://cogimon_urdf/meshes/simple/Leg1.STL" scale="${SF} -${SF} ${SF}" />
-      </geometry>
-    </collision>
-  </link>
   <link name ="LThighLowLeg">
     <inertial>

Commit message: Updated joint limits up to Left/Right KneePitch

File: cogimon_urdf/urdf/parts/legs.urdf.xacro (robot description, xacro)
@@ -129,5 +129,5 @@
     <origin xyz="${15.45*mmTom} ${112.0*mmTom} ${-50.0*mmTom}" rpy="0 0 0" />
     <axis xyz="1 0 0" />
-    <limit velocity="3.67" effort="176" lower="${-90.*toRad}" upper="${90.*toRad}" />
+    <limit velocity="3.67" effort="176" lower="${-30.*toRad}" upper="${95.*toRad}" />
     <dynamics friction="0" damping="3.0"/>
 </joint>
@@ -137,5 +137,5 @@
     <origin xyz="${-59.*mmTom} ${78.65*mmTom} ${-118.5*mmTom}" rpy="0 0 0" />
     <axis xyz="0 1 0" />
-    <limit velocity="3.67" effort="176" lower="${-90.*toRad}" upper="${90.*toRad}" />
+    <limit velocity="3.67" effort="176" lower="${-110.*toRad}" upper="${89.*toRad}" />
     <dynamics friction="0" damping="3.0"/>
 </joint>
@@ -145,5 +145,5 @@
     <origin xyz="${0.*mmTom} ${-90.*mmTom} ${-256.45*mmTom}" rpy="0 0 0" />
     <axis xyz="0 0 1" />
-    <limit velocity="3.67" effort="176" lower="${-90.*toRad}" upper="${90.*toRad}" />
+    <limit velocity="3.67" effort="176" lower="${-32.*toRad}" upper="${90.*toRad}" />
     <dynamics friction="0" damping="3.0"/>
 </joint>
@@ -153,5 +153,5 @@
     <origin xyz="${-39.*mmTom} ${64.1*mmTom} ${-60.7*mmTom}" rpy="0 0 0" />
     <axis xyz="0 1 0" />
-    <limit velocity="3.67" effort="176" lower="${-90.*toRad}" upper="${90.*toRad}" />
+    <limit velocity="3.67" effort="176" lower="${0.*toRad}" upper="${140.*toRad}" />
     <dynamics friction="0" damping="3.0"/>
 </joint>
@@ -301,5 +301,5 @@
     <origin xyz="${15.45*mmTom} ${-112.0*mmTom} ${-50.0*mmTom}" rpy="0 0 0" />
     <axis xyz="1 0 0" />
-    <limit velocity="3.67" effort="176" lower="${-90.*toRad}" upper="${90.*toRad}" />
+    <limit velocity="3.67" effort="176" lower="${-95.*toRad}" upper="${30.*toRad}" />
     <dynamics friction="0" damping="3.0"/>
 </joint>
@@ -309,5 +309,5 @@
     <origin xyz="${-59.*mmTom} ${-78.65*mmTom} ${-118.5*mmTom}" rpy="0 0 0" />
     <axis xyz="0 1 0" />
-    <limit velocity="3.67" effort="176" lower="${-90.*toRad}" upper="${90.*toRad}" />
+    <limit velocity="3.67" effort="176" lower="${-110.*toRad}" upper="${89.*toRad}" />
     <dynamics friction="0" damping="3.0"/>
 </joint>
@@ -317,5 +317,5 @@
     <origin xyz="${0.*mmTom} ${90.*mmTom} ${-256.45*mmTom}" rpy="0 0 0" />
     <axis xyz="0 0 1" />
-    <limit velocity="3.67" effort="176" lower="${-90.*toRad}" upper="${90.*toRad}" />
+    <limit velocity="3.67" effort="176" lower="${-90.*toRad}" upper="${32.*toRad}" />
     <dynamics friction="0" damping="3.0"/>
 </joint>
@@ -325,5 +325,5 @@
     <origin xyz="${-39.*mmTom} ${-64.1*mmTom} ${-60.7*mmTom}" rpy="0 0 0" />
     <axis xyz="0 1 0" />
-    <limit velocity="3.67" effort="176" lower="${-90.*toRad}" upper="${90.*toRad}" />
+    <limit velocity="3.67" effort="176" lower="${0.*toRad}" upper="${140.*toRad}" />
     <dynamics friction="0" damping="3.0"/>
 </joint>

Commit message: Updated joint limits for the ankles (we are using safety margins here)

File: cogimon_urdf/urdf/parts/legs.urdf.xacro (robot description, xacro)
@@ -156,4 +156,5 @@
     <dynamics friction="0" damping="3.0"/>
 </joint>
+<!-- Here we do an assumption: Ankle Pitch can go -50/+40 while Ankle Roll -15/+15-->
 <joint name="LAnklePitch" type="revolute">
     <parent link="LLowLeg"/>
@@ -161,5 +162,5 @@
     <origin xyz="${39.*mmTom} ${-61.6*mmTom} ${-425.294*mmTom}" rpy="0 0 0" />
     <axis xyz="0 1 0" />
-    <limit velocity="3.67" effort="176" lower="${-90.*toRad}" upper="${90.*toRad}" />
+    <limit velocity="3.67" effort="176" lower="${-50.*toRad}" upper="${40.*toRad}" />
     <dynamics friction="0" damping="0.1"/>
 </joint>
@@ -169,5 +170,5 @@
     <origin xyz="0 0 0" rpy="0 0 0" />
     <axis xyz="1 0 0" />
-    <limit velocity="3.67" effort="176" lower="${-90.*toRad}" upper="${90.*toRad}" />
+    <limit velocity="3.67" effort="176" lower="${-15.*toRad}" upper="${15.*toRad}" />
     <dynamics friction="0" damping="3.0"/>
 </joint>
@@ -328,4 +329,5 @@
     <dynamics friction="0" damping="3.0"/>
 </joint>
+<!-- Here we do an assumption: Ankle Pitch can go -50/+40 while Ankle Roll -15/+15-->
 <joint name="RAnklePitch" type="revolute">
     <parent link="RLowLeg"/>
@@ -333,5 +335,5 @@
     <origin xyz="${39.*mmTom} ${61.6*mmTom} ${-425.294*mmTom}" rpy="0 0 0" />
     <axis xyz="0 1 0" />
-    <limit velocity="3.67" effort="176" lower="${-90.*toRad}" upper="${90.*toRad}" />
+    <limit velocity="3.67" effort="176" lower="${-50.*toRad}" upper="${40.*toRad}" />
     <dynamics friction="0" damping="0.1"/>
 </joint>
@@ -341,5 +343,5 @@
     <origin xyz="0 0 0" rpy="0 0 0" />
     <axis xyz="1 0 0" />
-    <limit velocity="3.67" effort="176" lower="${-90.*toRad}" upper="${90.*toRad}" />
+    <limit velocity="3.67" effort="176" lower="${-15.*toRad}" upper="${15.*toRad}" />
     <dynamics friction="0" damping="3.0"/>
 </joint>

Commit message: added torque and vel limits

File: cogimon_urdf/urdf/parts/legs.urdf.xacro (robot description, xacro)
@@ -129,5 +129,5 @@
     <origin xyz="${15.45*mmTom} ${112.0*mmTom} ${-50.0*mmTom}" rpy="0 0 0" />
     <axis xyz="1 0 0" />
-    <limit velocity="3.67" effort="176" lower="${-30.*toRad}" upper="${95.*toRad}" />
+    <limit velocity="7.4" effort="235" lower="${-30.*toRad}" upper="${95.*toRad}" />
     <dynamics friction="0" damping="3.0"/>
 </joint>
@@ -137,5 +137,5 @@
     <origin xyz="${-59.*mmTom} ${78.65*mmTom} ${-118.5*mmTom}" rpy="0 0 0" />
     <axis xyz="0 1 0" />
-    <limit velocity="3.67" effort="176" lower="${-110.*toRad}" upper="${89.*toRad}" />
+    <limit velocity="7.4" effort="235" lower="${-110.*toRad}" upper="${89.*toRad}" />
     <dynamics friction="0" damping="3.0"/>
 </joint>
@@ -145,5 +145,5 @@
     <origin xyz="${0.*mmTom} ${-90.*mmTom} ${-256.45*mmTom}" rpy="0 0 0" />
     <axis xyz="0 0 1" />
-    <limit velocity="3.67" effort="176" lower="${-32.*toRad}" upper="${90.*toRad}" />
+    <limit velocity="4.6" effort="153" lower="${-32.*toRad}" upper="${90.*toRad}" />
     <dynamics friction="0" damping="3.0"/>
 </joint>
@@ -153,5 +153,5 @@
     <origin xyz="${-39.*mmTom} ${64.1*mmTom} ${-60.7*mmTom}" rpy="0 0 0" />
     <axis xyz="0 1 0" />
-    <limit velocity="3.67" effort="176" lower="${0.*toRad}" upper="${140.*toRad}" />
+    <limit velocity="5.5" effort="313" lower="${0.*toRad}" upper="${140.*toRad}" />
     <dynamics friction="0" damping="3.0"/>
 </joint>
@@ -162,5 +162,5 @@
     <origin xyz="${39.*mmTom} ${-61.6*mmTom} ${-425.294*mmTom}" rpy="0 0 0" />
     <axis xyz="0 1 0" />
-    <limit velocity="3.67" effort="176" lower="${-50.*toRad}" upper="${40.*toRad}" />
+    <limit velocity="4.9" effort="179" lower="${-50.*toRad}" upper="${40.*toRad}" />
     <dynamics friction="0" damping="0.1"/>
 </joint>
@@ -170,5 +170,5 @@
     <origin xyz="0 0 0" rpy="0 0 0" />
     <axis xyz="1 0 0" />
-    <limit velocity="3.67" effort="176" lower="${-15.*toRad}" upper="${15.*toRad}" />
+    <limit velocity="3.2" effort="230" lower="${-15.*toRad}" upper="${15.*toRad}" />
     <dynamics friction="0" damping="3.0"/>
 </joint>
@@ -302,5 +302,5 @@
     <origin xyz="${15.45*mmTom} ${-112.0*mmTom} ${-50.0*mmTom}" rpy="0 0 0" />
     <axis xyz="1 0 0" />
-    <limit velocity="3.67" effort="176" lower="${-95.*toRad}" upper="${30.*toRad}" />
+    <limit velocity="7.4" effort="235" lower="${-95.*toRad}" upper="${30.*toRad}" />
     <dynamics friction="0" damping="3.0"/>
 </joint>
@@ -310,5 +310,5 @@
     <origin xyz="${-59.*mmTom} ${-78.65*mmTom} ${-118.5*mmTom}" rpy="0 0 0" />
     <axis xyz="0 1 0" />
-    <limit velocity="3.67" effort="176" lower="${-110.*toRad}" upper="${89.*toRad}" />
+    <limit velocity="7.4" effort="235" lower="${-110.*toRad}" upper="${89.*toRad}" />
     <dynamics friction="0" damping="3.0"/>
 </joint>
@@ -318,5 +318,5 @@
     <origin xyz="${0.*mmTom} ${90.*mmTom} ${-256.45*mmTom}" rpy="0 0 0" />
     <axis xyz="0 0 1" />
-    <limit velocity="3.67" effort="176" lower="${-90.*toRad}" upper="${32.*toRad}" />
+    <limit velocity="4.9" effort="153" lower="${-90.*toRad}" upper="${32.*toRad}" />
     <dynamics friction="0" damping="3.0"/>
 </joint>
@@ -326,5 +326,5 @@
     <origin xyz="${-39.*mmTom} ${-64.1*mmTom} ${-60.7*mmTom}" rpy="0 0 0" />
     <axis xyz="0 1 0" />
-    <limit velocity="3.67" effort="176" lower="${0.*toRad}" upper="${140.*toRad}" />
+    <limit velocity="5.5" effort="313" lower="${0.*toRad}" upper="${140.*toRad}" />
     <dynamics friction="0" damping="3.0"/>
 </joint>
@@ -335,5 +335,5 @@
     <origin xyz="${39.*mmTom} ${61.6*mmTom} ${-425.294*mmTom}" rpy="0 0 0" />
     <axis xyz="0 1 0" />
-    <limit velocity="3.67" effort="176" lower="${-50.*toRad}" upper="${40.*toRad}" />
+    <limit velocity="4.9" effort="179" lower="${-50.*toRad}" upper="${40.*toRad}" />
     <dynamics friction="0" damping="0.1"/>
 </joint>
@@ -343,5 +343,5 @@
     <origin xyz="0 0 0" rpy="0 0 0" />
     <axis xyz="1 0 0" />
-    <limit velocity="3.67" effort="176" lower="${-15.*toRad}" upper="${15.*toRad}" />
+    <limit velocity="3.2" effort="230" lower="${-15.*toRad}" upper="${15.*toRad}" />
     <dynamics friction="0" damping="3.0"/>
 </joint>

Commit message: Fixed feet collision with new feet

File: cogimon_urdf/urdf/parts/legs.urdf.xacro (robot description, xacro)
@@ -118,5 +118,5 @@
     </visual>
     <collision>
-      <origin xyz="0.0 0.0 -0.046" rpy="0 0 0"/>
+      <origin xyz="0.0 0.0 -0.061" rpy="0 0 0"/>
        <geometry>
         <box size="0.21 0.11 0.015" />
@@ -315,5 +315,5 @@
     </visual>
     <collision>
-      <origin xyz="0.0 0.0 -0.046" rpy="0 0 0"/>
+      <origin xyz="0.0 0.0 -0.061" rpy="0 0 0"/>
        <geometry>
         <box size="0.21 0.11 0.015" />
