Commit message: Updated maximum torques

File: cogimon_urdf/urdf/parts/arms.urdf.xacro (robot description, xacro)
@@ -173,5 +173,5 @@
     <origin xyz="-0.014976503999999998 -0.0825 0.15770847" rpy="0 0 0" />
     <axis xyz="0 1 0" />
-    <limit velocity="4.0" effort="40" lower="-3.4034" upper="1.6581" />
+    <limit velocity="4.0" effort="120" lower="-3.4034" upper="1.6581" />
     <dynamics friction="0" damping="3.0"/>
 </joint>
@@ -181,5 +181,5 @@
     <origin xyz="0.0 -0.07329999999999999 0.0" rpy="0 0 0" />
     <axis xyz="1 0 0" />
-    <limit velocity="4.0" effort="40" lower="-2.094" upper="0.31415" />
+    <limit velocity="4.0" effort="120" lower="-2.094" upper="0.31415" />
     <dynamics friction="0" damping="3.0"/>
 </joint>
@@ -189,5 +189,5 @@
     <origin xyz="0.0 0.0 -0.04480846999999999" rpy="0 0 0" />
     <axis xyz="0 0 1" />
-    <limit velocity="4.0" effort="40" lower="-1.5708" upper="1.5708" />
+    <limit velocity="4.0" effort="120" lower="-1.5708" upper="1.5708" />
     <dynamics friction="0" damping="3.0"/>
 </joint>
@@ -197,5 +197,5 @@
     <origin xyz="0.015 0.0 -0.13519152999999998" rpy="0 0 0" />
     <axis xyz="0 1 0" />
-    <limit velocity="4.0" effort="40" lower="-2.3562" upper="0.0" />
+    <limit velocity="4.0" effort="90" lower="-2.3562" upper="0.0" />
     <dynamics friction="0" damping="3.0"/>
   </joint>
@@ -206,5 +206,5 @@
     <origin xyz="-0.014976503999999998 0.0825 0.15770847" rpy="0 0 0" />
     <axis xyz="0 1 0" />
-    <limit velocity="4.0" effort="40" lower="-3.4034" upper="1.6581" />
+    <limit velocity="4.0" effort="120" lower="-3.4034" upper="1.6581" />
     <dynamics friction="0" damping="3.0"/>
 </joint>
@@ -222,5 +222,5 @@
     <origin xyz="0.0 0.0 -0.04480846999999999" rpy="0 0 0" />
     <axis xyz="0 0 1" />
-    <limit velocity="4.0" effort="40" lower="-1.5708" upper="1.5708" />
+    <limit velocity="4.0" effort="120" lower="-1.5708" upper="1.5708" />
     <dynamics friction="0" damping="3.0"/>
 </joint>
@@ -230,5 +230,5 @@
     <origin xyz="0.015 0.0 -0.13519152999999998" rpy="0 0 0" />
     <axis xyz="0 1 0" />
-    <limit velocity="4.0" effort="40" lower="-2.3562" upper="0.0" />
+    <limit velocity="4.0" effort="90" lower="-2.3562" upper="0.0" />
     <dynamics friction="0" damping="3.0"/>
   </joint>

File: cogimon_urdf/urdf/parts/forearms.urdf.xacro (robot description, xacro)
@@ -149,5 +149,5 @@
     <origin xyz="-0.015 0.0 ${-0.051 - Wrj1_to_FT}" rpy="0 0 0"/>
     <axis xyz="0 0 1" />
-    <limit velocity="4.0" effort="15" lower="-1.5708" upper="1.5708" />
+    <limit velocity="4.0" effort="40" lower="-1.5708" upper="1.5708" />
     <dynamics friction="0" damping="0.03"/>
   </joint>
@@ -157,5 +157,5 @@
     <origin xyz="0 0 ${-0.14368 + Wrj1_to_FT}" rpy="0 0 0"/>
     <axis xyz="0 1 0"/>
-    <limit velocity="4.0" effort="15" lower="-0.524" upper="0.524" />
+    <limit velocity="4.0" effort="40" lower="-0.524" upper="0.524" />
     <dynamics friction="0" damping="0.03"/>
   </joint>
@@ -165,5 +165,5 @@
     <origin xyz="0 0 0.0" rpy="0 0 0"/>
     <axis xyz="1 0 0"/>
-    <limit velocity="4.0" effort="15" lower="-0.785375" upper="1.395" />
+    <limit velocity="4.0" effort="40" lower="-0.785375" upper="1.395" />
     <dynamics friction="0" damping="0.03"/>
   </joint>
@@ -179,5 +179,5 @@
     <origin xyz="-0.015 0.0 ${-0.051 - Wrj1_to_FT}" rpy="0 0 0"/>
     <axis xyz="0 0 1" />
-    <limit velocity="4.0" effort="15" lower="-1.5708" upper="1.5708" />
+    <limit velocity="4.0" effort="40" lower="-1.5708" upper="1.5708" />
     <dynamics friction="0" damping="0.03"/>
   </joint>
@@ -187,5 +187,5 @@
     <origin xyz="0 0 ${-0.14368 + Wrj1_to_FT}" rpy="0 0 0"/>
     <axis xyz="0 1 0"/>
-    <limit velocity="4.0" effort="15" lower="-0.524" upper="0.524" />
+    <limit velocity="4.0" effort="40" lower="-0.524" upper="0.524" />
     <dynamics friction="0" damping="0.03"/>
   </joint>
@@ -195,5 +195,5 @@
     <origin xyz="0 0 0.0" rpy="0 0 0"/>
     <axis xyz="1 0 0"/>
-    <limit velocity="4.0" effort="15" lower="-1.395" upper="0.785375" />
+    <limit velocity="4.0" effort="40" lower="-1.395" upper="0.785375" />
     <dynamics friction="0" damping="0.03"/>
   </joint>

File: cogimon_urdf/urdf/parts/legs.urdf.xacro (robot description, xacro)
@@ -302,5 +302,5 @@
     <origin xyz="0.0 -0.023 0.0" rpy="0 0 0" />
     <axis xyz="0 1 0" />
-    <limit velocity="4.0" effort="80" lower="-1.9199" upper="0.7854" />
+    <limit velocity="4.0" effort="140" lower="-1.9199" upper="0.7854" />
     <dynamics friction="0" damping="3.0"/>
   </joint>
@@ -310,5 +310,5 @@
     <origin xyz="0.0 -0.0496 0.0" rpy="0 0 0" />
     <axis xyz="1 0 0" />
-    <limit velocity="4.0" effort="80" lower="-1.0472" upper="0.4363" />
+    <limit velocity="4.0" effort="140" lower="-1.0472" upper="0.4363" />
     <dynamics friction="0" damping="3.0"/>
   </joint>
@@ -318,5 +318,5 @@
     <origin xyz="0.0 0.0 ${-0.1024-hco-0.025}" rpy="0 0 0" />
     <axis xyz="0 0 1" />
-    <limit velocity="4.0" effort="80" lower="-0.8727" upper="0.8727" />
+    <limit velocity="4.0" effort="140" lower="-0.8727" upper="0.8727" />
     <dynamics friction="0" damping="3.0"/>
   </joint>
@@ -326,5 +326,5 @@
     <origin xyz="0.0 0.0 -0.1234" rpy="0 0 0" />
     <axis xyz="0 1 0" />
-    <limit velocity="4.0" effort="80" lower="-0.1745" upper="1.9199" />
+    <limit velocity="4.0" effort="140" lower="-0.1745" upper="1.9199" />
     <dynamics friction="0" damping="3.0"/>
   </joint>
@@ -334,5 +334,5 @@
     <origin xyz="0.0 0.0 ${-0.201-hco-0.025}" rpy="0 0 0" />
     <axis xyz="1 0 0" />
-    <limit velocity="4.0" effort="80" lower="-0.6109" upper="0.6109" />
+    <limit velocity="4.0" effort="140" lower="-0.6109" upper="0.6109" />
     <dynamics friction="0" damping="3.0"/>
   </joint>
@@ -342,5 +342,5 @@
       <origin xyz="0.0 0.0 0.0" rpy="0 0 0" />
       <axis xyz="0 1 0" />
-      <limit velocity="4.0" effort="80" lower="-1.2217" upper="1.2217" />
+      <limit velocity="4.0" effort="140" lower="-1.2217" upper="1.2217" />
       <dynamics friction="0" damping="3.0"/>
   </joint>
@@ -351,5 +351,5 @@
     <origin xyz="0.0 0.023 0.0" rpy="0 0 0" />
     <axis xyz="0 1 0" />
-    <limit velocity="4.0" effort="80" lower="-1.9199" upper="0.7854" />
+    <limit velocity="4.0" effort="140" lower="-1.9199" upper="0.7854" />
     <dynamics friction="0" damping="3.0"/>
   </joint>
@@ -359,5 +359,5 @@
     <origin xyz="0.0 0.0496 0.0" rpy="0 0 0" />
     <axis xyz="1 0 0" />
-    <limit velocity="4.0" effort="80" lower="-0.4363" upper="1.0472" />
+    <limit velocity="4.0" effort="140" lower="-0.4363" upper="1.0472" />
     <dynamics friction="0" damping="3.0"/>
   </joint>
@@ -367,5 +367,5 @@
     <origin xyz="0.0 0.0 ${-0.1024-hco-0.025}" rpy="0 0 0" />
     <axis xyz="0 0 1" />
-    <limit velocity="4.0" effort="80" lower="-0.8727" upper="0.8727" />
+    <limit velocity="4.0" effort="140" lower="-0.8727" upper="0.8727" />
     <dynamics friction="0" damping="3.0"/>
   </joint>
@@ -375,5 +375,5 @@
     <origin xyz="0.0 0.0 -0.1234" rpy="0 0 0" />
     <axis xyz="0 1 0" />
-    <limit velocity="4.0" effort="80" lower="-0.1745" upper="1.9199" />
+    <limit velocity="4.0" effort="140" lower="-0.1745" upper="1.9199" />
     <dynamics friction="0" damping="3.0"/>
   </joint>
@@ -383,5 +383,5 @@
     <origin xyz="0.0 0.0 ${-0.201-hco-0.025}" rpy="0 0 0" />
     <axis xyz="1 0 0" />
-    <limit velocity="4.0" effort="80" lower="-0.6109" upper="0.6109" />
+    <limit velocity="4.0" effort="140" lower="-0.6109" upper="0.6109" />
     <dynamics friction="0" damping="3.0"/>
   </joint>
@@ -391,5 +391,5 @@
       <origin xyz="0.0 0.0 0.0" rpy="0 0 0" />
       <axis xyz="0 1 0" />
-      <limit velocity="4.0" effort="80" lower="-1.2217" upper="1.2217" />
+      <limit velocity="4.0" effort="140" lower="-1.2217" upper="1.2217" />
       <dynamics friction="0" damping="3.0"/>
   </joint>

File: cogimon_urdf/urdf/parts/torso.urdf.xacro (robot description, xacro)
@@ -80,5 +80,5 @@
     <origin xyz="0.020281504 0 0.11912053" rpy="0 0 0" />
     <axis xyz="${cos_20} 0 ${sin_20}" />
-    <limit velocity="4.0" effort="80" lower="-0.5236" upper="0.5235" />
+    <limit velocity="4.0" effort="140" lower="-0.5236" upper="0.5235" />
     <!-- dynamics friction="0" damping="0.3"/ -->
     <dynamics friction="0" damping="3.0"/>
@@ -97,5 +97,5 @@
     <origin xyz="0 0 ${0.04749999+hco-0.05}" rpy="0 0 0" />
     <axis xyz="0 0 1" />
-    <limit velocity="4.0" effort="40" lower="-1.3963" upper="1.3962" />
+    <limit velocity="4.0" effort="140" lower="-1.3963" upper="1.3962" />
     <dynamics friction="0" damping="3.0"/>
   </joint>

Commit message: Added offset in arms and forearms

File: cogimon_urdf/urdf/parts/arms.urdf.xacro (robot description, xacro)
@@ -3,4 +3,5 @@
 <xacro:property name="PI" value="3.14159265359" />
 <xacro:property name="SF" value="0.03937" /> <!-- Scale factor for meshes -->
+<xacro:property name="uarm_offset" value="${0.15/2.}" />
 <!-- LINKS -->
 <!-- RIGHT ARM -->
@@ -187,5 +188,5 @@
     <parent link="RShr"/>
     <child link="RShy"/>
-    <origin xyz="0.0 0.0 -0.04480846999999999" rpy="0 0 0" />
+    <origin xyz="0.0 0.0 ${-0.04480846999999999-uarm_offset}" rpy="0 0 0" />
     <axis xyz="0 0 1" />
     <limit velocity="4.0" effort="120" lower="-1.5708" upper="1.5708" />
@@ -195,5 +196,5 @@
     <parent link="RShy"/>
     <child link="RElb"/>
-    <origin xyz="0.015 0.0 -0.13519152999999998" rpy="0 0 0" />
+    <origin xyz="0.015 0.0 ${-0.13519152999999998-uarm_offset}" rpy="0 0 0" />
     <axis xyz="0 1 0" />
     <limit velocity="4.0" effort="90" lower="-2.3562" upper="0.0" />
@@ -220,5 +221,5 @@
     <parent link="LShr"/>
     <child link="LShy"/>
-    <origin xyz="0.0 0.0 -0.04480846999999999" rpy="0 0 0" />
+    <origin xyz="0.0 0.0 ${-0.04480846999999999-uarm_offset}" rpy="0 0 0" />
     <axis xyz="0 0 1" />
     <limit velocity="4.0" effort="120" lower="-1.5708" upper="1.5708" />
@@ -228,5 +229,5 @@
     <parent link="LShy"/>
     <child link="LElb"/>
-    <origin xyz="0.015 0.0 -0.13519152999999998" rpy="0 0 0" />
+    <origin xyz="0.015 0.0 ${-0.13519152999999998-uarm_offset}" rpy="0 0 0" />
     <axis xyz="0 1 0" />
     <limit velocity="4.0" effort="90" lower="-2.3562" upper="0.0" />

File: cogimon_urdf/urdf/parts/forearms.urdf.xacro (robot description, xacro)
@@ -7,4 +7,5 @@
 		and to the z displacement of mass, visual and collision of *Forearm -->
 <xacro:property name="Wrj1_to_FT" value="0.0568" />
+<xacro:property name="larm_offset" value="${0.175/2.}" />
 <!-- ****************LINKS**************** -->
 <!-- ****************LEFT FOREARM**************** -->
@@ -147,5 +148,5 @@
     <parent link="LElb"/>
     <child link="LForearm"/>
-    <origin xyz="-0.015 0.0 ${-0.051 - Wrj1_to_FT}" rpy="0 0 0"/>
+    <origin xyz="-0.015 0.0 ${-0.051 - Wrj1_to_FT - larm_offset}" rpy="0 0 0"/>
     <axis xyz="0 0 1" />
     <limit velocity="4.0" effort="40" lower="-1.5708" upper="1.5708" />
@@ -155,5 +156,5 @@
     <parent link="LForearm"/>
     <child link="LWrMot2"/>
-    <origin xyz="0 0 ${-0.14368 + Wrj1_to_FT}" rpy="0 0 0"/>
+    <origin xyz="0 0 ${-0.14368 + Wrj1_to_FT - larm_offset}" rpy="0 0 0"/>
     <axis xyz="0 1 0"/>
     <limit velocity="4.0" effort="40" lower="-0.524" upper="0.524" />
@@ -177,5 +178,5 @@
     <parent link="RElb"/>
     <child link="RForearm"/>
-    <origin xyz="-0.015 0.0 ${-0.051 - Wrj1_to_FT}" rpy="0 0 0"/>
+    <origin xyz="-0.015 0.0 ${-0.051 - Wrj1_to_FT - larm_offset}" rpy="0 0 0"/>
     <axis xyz="0 0 1" />
     <limit velocity="4.0" effort="40" lower="-1.5708" upper="1.5708" />
@@ -185,5 +186,5 @@
     <parent link="RForearm"/>
     <child link="RWrMot2"/>
-    <origin xyz="0 0 ${-0.14368 + Wrj1_to_FT}" rpy="0 0 0"/>
+    <origin xyz="0 0 ${-0.14368 + Wrj1_to_FT - larm_offset}" rpy="0 0 0"/>
     <axis xyz="0 1 0"/>
     <limit velocity="4.0" effort="40" lower="-0.524" upper="0.524" />

Commit message: updated torque limits

File: cogimon_urdf/urdf/parts/arms.urdf.xacro (robot description, xacro)
@@ -152,5 +152,5 @@
     <origin xyz="${45.7475*mmTom} ${-169.137*mmTom} ${155.126*mmTom}" rpy="-0.174533 0 0.5235988" />
     <axis xyz="0 1 0" />
-    <limit velocity="6.283" effort="147" lower="-3.359" upper="1.606" />
+    <limit velocity="6.283" effort="140" lower="-3.359" upper="1.606" />
     <dynamics friction="0" damping="3.0"/>
 </joint>
@@ -160,5 +160,5 @@
     <origin xyz="${-90.15*mmTom} ${-62*mmTom} 0" rpy="0.1745327 0 0" />
     <axis xyz="1 0 0" />
-    <limit velocity="6.283" effort="120" lower="-3.43" upper="-0.004" />
+    <limit velocity="6.283" effort="140" lower="-3.43" upper="0.0" />
     <dynamics friction="0" damping="3.0"/>
 </joint>
@@ -168,5 +168,5 @@
     <origin xyz="${90.15*mmTom} 0 ${-218.15*mmTom}" rpy="0 0 0" />
     <axis xyz="0 0 1" />
-    <limit velocity="6.283" effort="147" lower="-2.55" upper="2.55" />
+    <limit velocity="6.283" effort="120" lower="-2.55" upper="2.55" />
     <dynamics friction="0" damping="3.0"/>
 </joint>
@@ -176,5 +176,5 @@
     <origin xyz="${45.*mmTom} ${-55.15*mmTom} ${-74.*mmTom}" rpy="0 0 0" />
     <axis xyz="0 1 0" />
-    <limit velocity="6.283" effort="147" lower="-2.488" upper="0.292" />
+    <limit velocity="6.283" effort="120" lower="-2.488" upper="0.292" />
     <dynamics friction="0" damping="3.0"/>
 </joint>
@@ -184,5 +184,5 @@
     <origin xyz="${-15.*mmTom} ${55.15*mmTom} ${-95.*mmTom}" rpy="0 0 0"/>
     <axis xyz="0 0 1" />
-    <limit velocity="6.283" effort="55" lower="-2.55" upper="2.55" />
+    <limit velocity="6.283" effort="35" lower="-2.55" upper="2.55" />
     <dynamics friction="0" damping="0.03"/>
 </joint>
@@ -192,5 +192,5 @@
     <origin xyz="0 ${-49*mmTom} ${-156.*mmTom}" rpy="0 0 0"/>
     <axis xyz="0 1 0"/>
-    <limit velocity="6.283" effort="55" lower="-1.542" upper="1.508" />
+    <limit velocity="6.283" effort="35" lower="-1.542" upper="1.508" />
     <dynamics friction="0" damping="0.03"/>
 </joint>
@@ -200,5 +200,5 @@
        <origin xyz="0 ${49*mmTom} ${-174.*mmTom}" rpy="0 0 0"/>
        <axis xyz="0 0 1"/>
-       <limit velocity="6.283" effort="27" lower="-2.55" upper="2.55" />
+       <limit velocity="6.283" effort="20" lower="-2.55" upper="2.55" />
        <dynamics friction="0" damping="0.03"/>
 </joint>
@@ -351,5 +351,5 @@
     <origin xyz="${45.7475*mmTom} ${169.137*mmTom} ${155.126*mmTom}" rpy="0.174533 0 -0.5235988" />
     <axis xyz="0 1 0" />
-    <limit velocity="6.283" effort="147" lower="-3.352" upper="1.603" />
+    <limit velocity="6.283" effort="140" lower="-3.352" upper="1.603" />
     <dynamics friction="0" damping="3.0"/>
 </joint>
@@ -359,5 +359,5 @@
     <origin xyz="${-90.15*mmTom} ${62*mmTom} 0" rpy="-0.1745327 0 0" />
     <axis xyz="1 0 0" />
-    <limit velocity="6.283" effort="120" lower="0.037" upper="3.517" />
+    <limit velocity="6.283" effort="140" lower="0.0" upper="3.517" />
     <dynamics friction="0" damping="3.0"/>
 </joint>
@@ -367,5 +367,5 @@
     <origin xyz="${90.15*mmTom} 0 ${-218.15*mmTom}" rpy="0 0 0" />
     <axis xyz="0 0 1" />
-    <limit velocity="6.283" effort="147" lower="-2.55" upper="2.55" />
+    <limit velocity="6.283" effort="120" lower="-2.55" upper="2.55" />
     <dynamics friction="0" damping="3.0"/>
 </joint>
@@ -375,5 +375,5 @@
     <origin xyz="${45.*mmTom} ${55.15*mmTom} ${-74.*mmTom}" rpy="0 0 0" />
     <axis xyz="0 1 0" />
-    <limit velocity="6.283" effort="147" lower="-2.492" upper="0.298" />
+    <limit velocity="6.283" effort="120" lower="-2.492" upper="0.298" />
     <dynamics friction="0" damping="3.0"/>
 </joint>
@@ -383,5 +383,5 @@
     <origin xyz="${-15.*mmTom} ${-55.15*mmTom} ${-95.*mmTom}" rpy="0 0 0"/>
     <axis xyz="0 0 1" />
-    <limit velocity="6.283" effort="55" lower="-2.55" upper="2.55" />
+    <limit velocity="6.283" effort="35" lower="-2.55" upper="2.55" />
     <dynamics friction="0" damping="0.03"/>
 </joint>
@@ -391,5 +391,5 @@
     <origin xyz="0 ${49*mmTom} ${-156.*mmTom}" rpy="0 0 0"/>
     <axis xyz="0 1 0"/>
-    <limit velocity="6.283" effort="55" lower="-1.562" upper="1.478" />
+    <limit velocity="6.283" effort="35" lower="-1.562" upper="1.478" />
     <dynamics friction="0" damping="0.03"/>
 </joint>
@@ -399,5 +399,5 @@
        <origin xyz="0 ${-49*mmTom} ${-174.*mmTom}" rpy="0 0 0"/>
        <axis xyz="0 0 1"/>
-       <limit velocity="6.283" effort="27" lower="-2.55" upper="2.55" />
+       <limit velocity="6.283" effort="20" lower="-2.55" upper="2.55" />
        <dynamics friction="0" damping="0.03"/>
 </joint>

File: cogimon_urdf/urdf/parts/legs.urdf.xacro (robot description, xacro)
@@ -129,5 +129,5 @@
     <origin xyz="${15.45*mmTom} ${112.0*mmTom} ${-50.0*mmTom}" rpy="0 0 0" />
     <axis xyz="1 0 0" />
-    <limit velocity="7.4" effort="235" lower="${-30.*toRad}" upper="${95.*toRad}" />
+    <limit velocity="7.4" effort="200" lower="${-30.*toRad}" upper="${95.*toRad}" />
     <dynamics friction="0" damping="3.0"/>
 </joint>
@@ -137,5 +137,5 @@
     <origin xyz="${-59.*mmTom} ${78.65*mmTom} ${-118.5*mmTom}" rpy="0 0 0" />
     <axis xyz="0 1 0" />
-    <limit velocity="7.4" effort="235" lower="${-110.*toRad}" upper="${89.*toRad}" />
+    <limit velocity="7.4" effort="200" lower="${-110.*toRad}" upper="${89.*toRad}" />
     <dynamics friction="0" damping="3.0"/>
 </joint>
@@ -145,5 +145,5 @@
     <origin xyz="${0.*mmTom} ${-90.*mmTom} ${-256.45*mmTom}" rpy="0 0 0" />
     <axis xyz="0 0 1" />
-    <limit velocity="4.6" effort="153" lower="${-32.*toRad}" upper="${90.*toRad}" />
+    <limit velocity="4.6" effort="120" lower="${-32.*toRad}" upper="${90.*toRad}" />
     <dynamics friction="0" damping="3.0"/>
 </joint>
@@ -153,5 +153,5 @@
     <origin xyz="${-39.*mmTom} ${64.1*mmTom} ${-60.7*mmTom}" rpy="0 0 0" />
     <axis xyz="0 1 0" />
-    <limit velocity="5.5" effort="313" lower="${0.*toRad}" upper="${140.*toRad}" />
+    <limit velocity="5.5" effort="200" lower="${0.*toRad}" upper="${140.*toRad}" />
     <dynamics friction="0" damping="3.0"/>
 </joint>
@@ -162,5 +162,5 @@
     <origin xyz="${39.*mmTom} ${-61.6*mmTom} ${-425.294*mmTom}" rpy="0 0 0" />
     <axis xyz="0 1 0" />
-    <limit velocity="4.9" effort="179" lower="${-50.*toRad}" upper="${40.*toRad}" />
+    <limit velocity="4.9" effort="200" lower="${-50.*toRad}" upper="${40.*toRad}" />
     <dynamics friction="0" damping="0.1"/>
 </joint>
@@ -170,5 +170,5 @@
     <origin xyz="0 0 0" rpy="0 0 0" />
     <axis xyz="1 0 0" />
-    <limit velocity="3.2" effort="230" lower="${-15.*toRad}" upper="${15.*toRad}" />
+    <limit velocity="3.2" effort="60" lower="${-15.*toRad}" upper="${15.*toRad}" />
     <dynamics friction="0" damping="3.0"/>
 </joint>
@@ -302,5 +302,5 @@
     <origin xyz="${15.45*mmTom} ${-112.0*mmTom} ${-50.0*mmTom}" rpy="0 0 0" />
     <axis xyz="1 0 0" />
-    <limit velocity="7.4" effort="235" lower="${-95.*toRad}" upper="${30.*toRad}" />
+    <limit velocity="7.4" effort="200" lower="${-95.*toRad}" upper="${30.*toRad}" />
     <dynamics friction="0" damping="3.0"/>
 </joint>
@@ -310,5 +310,5 @@
     <origin xyz="${-59.*mmTom} ${-78.65*mmTom} ${-118.5*mmTom}" rpy="0 0 0" />
     <axis xyz="0 1 0" />
-    <limit velocity="7.4" effort="235" lower="${-110.*toRad}" upper="${89.*toRad}" />
+    <limit velocity="7.4" effort="200" lower="${-110.*toRad}" upper="${89.*toRad}" />
     <dynamics friction="0" damping="3.0"/>
 </joint>
@@ -318,5 +318,5 @@
     <origin xyz="${0.*mmTom} ${90.*mmTom} ${-256.45*mmTom}" rpy="0 0 0" />
     <axis xyz="0 0 1" />
-    <limit velocity="4.9" effort="153" lower="${-90.*toRad}" upper="${32.*toRad}" />
+    <limit velocity="4.9" effort="120" lower="${-90.*toRad}" upper="${32.*toRad}" />
     <dynamics friction="0" damping="3.0"/>
 </joint>
@@ -326,5 +326,5 @@
     <origin xyz="${-39.*mmTom} ${-64.1*mmTom} ${-60.7*mmTom}" rpy="0 0 0" />
     <axis xyz="0 1 0" />
-    <limit velocity="5.5" effort="313" lower="${0.*toRad}" upper="${140.*toRad}" />
+    <limit velocity="5.5" effort="200" lower="${0.*toRad}" upper="${140.*toRad}" />
     <dynamics friction="0" damping="3.0"/>
 </joint>
@@ -335,5 +335,5 @@
     <origin xyz="${39.*mmTom} ${61.6*mmTom} ${-425.294*mmTom}" rpy="0 0 0" />
     <axis xyz="0 1 0" />
-    <limit velocity="4.9" effort="179" lower="${-50.*toRad}" upper="${40.*toRad}" />
+    <limit velocity="4.9" effort="200" lower="${-50.*toRad}" upper="${40.*toRad}" />
     <dynamics friction="0" damping="0.1"/>
 </joint>
@@ -343,5 +343,5 @@
     <origin xyz="0 0 0" rpy="0 0 0" />
     <axis xyz="1 0 0" />
-    <limit velocity="3.2" effort="230" lower="${-15.*toRad}" upper="${15.*toRad}" />
+    <limit velocity="3.2" effort="60" lower="${-15.*toRad}" upper="${15.*toRad}" />
     <dynamics friction="0" damping="3.0"/>
 </joint>

File: cogimon_urdf/urdf/parts/torso.urdf.xacro (robot description, xacro)
@@ -117,5 +117,5 @@
     <origin xyz="${12.00*mmTom} 0.0 0.0" rpy="0 0 0" />
     <axis xyz="1 0 0" />
-    <limit velocity="7.4" effort="150" lower="${-30.*toRad}" upper="${30.*toRad}" />
+    <limit velocity="7.4" effort="140" lower="${-30.*toRad}" upper="${30.*toRad}" />
     <dynamics friction="0" damping="3.0"/>
 </joint>
