Commit message: Added macro to specify joint names in arms

File: cogimon_urdf/urdf/parts/arms.urdf.xacro (robot description, xacro)
@@ -4,451 +4,10 @@
 <xacro:property name="mmTom" value="0.001" />
 <xacro:property name="mm2Tom2" value="${0.001*0.001}" /-->
+<xacro:include filename="$(find cogimon_urdf)/urdf/parts/arms_macro.urdf.xacro" />
 <xacro:if value="${COGIMON_RIGHT_ARM}">
-<!-- RIGHT ARM -->
-<link name ="RShp">
-    <inertial>
-      <origin xyz="${-7.4457212*mmTom} ${-3.4107960e+01*mmTom} ${1.0978102e-01*mmTom}" rpy="0 0 0"/>
-      <mass value="1.9628675"/>
-      <inertia ixx="${5.3547717e+03*mm2Tom2}"  ixy="${-3.6428926e+02*mm2Tom2}"  ixz="${1.5089568e+01*mm2Tom2}" iyy="${3.3923328e+03*mm2Tom2}" iyz="${-5.5692312e+01*mm2Tom2}" izz="${6.8921413e+03*mm2Tom2}" />
-    </inertial>
-    <visual>
-      <origin xyz="0 0 0" rpy="0 0 0"/>
-      <geometry name="RShp_visual">
-        <mesh filename="package://cogimon_urdf/meshes/ShoulderPitch.STL" scale="0.001 0.001 0.001" />
-      </geometry>
-      <material name="green"/>
-    </visual>
-    <collision>
-      <origin xyz="0 0 0" rpy="0 0 0"/>
-      <geometry name="RShp_collision">
-        <mesh filename="package://cogimon_urdf/meshes/simple/ShoulderPitch.STL" scale="0.001 0.001 0.001" />
-      </geometry>
-    </collision>
-</link>
-<link name ="RShr">
-    <inertial>
-      <origin xyz="${5.8142302e+01*mmTom} ${-5.7450803e-02*mmTom} ${-7.7477683e+01*mmTom}" rpy="0 0 0"/>
-      <mass value="1.8595811"/>
-      <inertia ixx="${1.3776643e+04*mm2Tom2}"  ixy="${-3.7788675e+01*mm2Tom2}"  ixz="${3.7690171e+03*mm2Tom2}" iyy="${1.5677464e+04*mm2Tom2}" iyz="${9.4893549*mm2Tom2}" izz="${4.6317657e+03*mm2Tom2}" />
-    </inertial>
-    <visual>
-      <origin xyz="0 0 0" rpy="0 0 0"/>
-      <geometry name="RShr_visual">
-        <mesh filename="package://cogimon_urdf/meshes/ShoulderRoll.STL" scale="0.001 0.001 0.001" />
-      </geometry>
-      <material name="dark_grey"/>
-    </visual>
-    <collision>
-      <origin xyz="0 0 0" rpy="0 0 0"/>
-      <geometry name="RShr_collision">
-        <mesh filename="package://cogimon_urdf/meshes/simple/ShoulderRoll.STL" scale="0.001 0.001 0.001" />
-      </geometry>
-    </collision>
-</link>
-<link name ="RShy">
-    <inertial>
-      <origin xyz="${1.4625194e+01*mmTom} ${-8.1726720e-01*mmTom} ${-2.8333545e+01*mmTom}" rpy="0 0 0"/>
-      <mass value="1.6678109"/>
-      <inertia ixx="${6.4480435e+03*mm2Tom2}"  ixy="${1.5639093e+02*mm2Tom2}"  ixz="${1.2205359e+03*mm2Tom2}" iyy="${7.3372077e+03*mm2Tom2}" iyz="${-8.9941532e+01*mm2Tom2}" izz="${3.6738448e+03*mm2Tom2}" />
-    </inertial>
-    <visual>
-      <origin xyz="0 0 0" rpy="0 0 0"/>
-      <geometry name="RShy_visual">
-        <mesh filename="package://cogimon_urdf/meshes/ShoulderYaw.STL" scale="0.001 0.001 0.001" />
-      </geometry>
-      <material name="green"/>
-    </visual>
-    <collision>
-      <origin xyz="0 0 0" rpy="0 0 0"/>
-      <geometry name="RShy_collision">
-        <mesh filename="package://cogimon_urdf/meshes/simple/ShoulderYaw.STL" scale="0.001 0.001 0.001" />
-      </geometry>
-    </collision>
-</link>
-<link name ="RElb">
- <inertial>
-   <origin xyz="${-7.6833067*mmTom} ${4.0302205e+01*mmTom} ${-4.3492779e+01*mmTom}" rpy="0 0 0"/>
-   <mass value="1.3157289"/>
-   <inertia ixx="${4.3303940e+03*mm2Tom2}"  ixy="${1.1737391e+02*mm2Tom2}"  ixz="${-4.1923199e+02*mm2Tom2}" iyy="${3.8539919e+03*mm2Tom2}" iyz="${7.9573038e+02*mm2Tom2}" izz="${1.7594689e+03*mm2Tom2}" />
- </inertial>
- <visual>
-   <origin xyz="0 0 0" rpy="0 0 0"/>
-   <geometry name="RElb_visual">
-     <mesh filename="package://cogimon_urdf/meshes/Elbow.STL" scale="0.001 0.001 0.001" />
-   </geometry>
-  <material name="dark_grey"/>
- </visual>
- <collision>
-   <origin xyz="0 0 0" rpy="0 0 0"/>
-   <geometry name="RElb_collision">
-     <mesh filename="package://cogimon_urdf/meshes/simple/Elbow.STL" scale="0.001 0.001 0.001" />
-   </geometry>
- </collision>
-</link>
-<link name ="RForearm">
- <inertial>
-   <origin xyz="${-1.1079615e-01*mmTom} ${-1.1590836e+01*mmTom} ${-7.8160260e+01*mmTom}" rpy="0 0 0"/>
-   <mass value="1.4908547"/>
-   <inertia ixx="${8.5692128e+03*mm2Tom2}"  ixy="${-1.7856252e+01*mm2Tom2}"  ixz="${1.9379365e+01*mm2Tom2}" iyy="${7.7454159e+03*mm2Tom2}" iyz="${3.2860094e+02*mm2Tom2}" izz="${2.7441921e+03*mm2Tom2}" />
- </inertial>
- <visual>
-   <origin xyz="0 0 0" rpy="0 0 0"/>
-   <geometry name="RForearm_visual">
-     <mesh filename="package://cogimon_urdf/meshes/Forearm.STL" scale="0.001 0.001 0.001" />
-   </geometry>
-  <material name="green"/>
- </visual>
- <collision>
-   <origin xyz="0 0 0" rpy="0 0 0"/>
-   <geometry name="RForearm_collision">
-     <mesh filename="package://cogimon_urdf/meshes/simple/Forearm.STL" scale="0.001 0.001 0.001" />
-   </geometry>
- </collision>
-</link>
-<link name="RWrMot2">
- <inertial>
-   <origin xyz="${-4.6502396e-03*mmTom} ${3.8014094e+01*mmTom} ${-6.9926878e+01*mmTom}" rpy="0 0 0"/>
-   <mass value="1.1263612"/>
-   <inertia ixx="${5.1871784e+03*mm2Tom2}"  ixy="${-2.7244370e+01*mm2Tom2}"  ixz="${2.2833496*mm2Tom2}" iyy="${4.8037789e+03*mm2Tom2}" iyz="${7.2165653e+02*mm2Tom2}" izz="${1.2771388e+03*mm2Tom2}" />
- </inertial>
- <visual>
-   <origin xyz="0 0 0" rpy="0 0 0"/>
-   <geometry name="RWrMot2_visual">
-     <mesh filename="package://cogimon_urdf/meshes/ForearmPitch.STL" scale="0.001 0.001 0.001" />
-   </geometry>
-  <material name="dark_grey"/>
- </visual>
- <collision>
-   <origin xyz="0 0 0" rpy="0 0 0"/>
-   <geometry name="RWrMot2_collision">
-     <mesh filename="package://cogimon_urdf/meshes/simple/ForearmPitch.STL" scale="0.001 0.001 0.001" />
-   </geometry>
- </collision>
-</link>
-<link name="RWrMot3">
- <inertial>
-   <origin xyz="0 0 ${3.1270570e+01*mmTom}" rpy="0 0 0"/>
-   <mass value="2.7966428e-01"/>
-   <inertia ixx="${1.4415192e+02*mm2Tom2}"  ixy="${9.8651826e-02*mm2Tom2}"  ixz="0" iyy="${1.4417010e+02*mm2Tom2}" iyz="0" izz="${6.0500616e+01*mm2Tom2}" />
- </inertial>
- <visual>
-   <origin xyz="0 0 0" rpy="0 0 0"/>
-   <geometry name="RWrMot3_visual">
-     <mesh filename="package://cogimon_urdf/meshes/ForearmYaw.STL" scale="0.001 0.001 0.001" />
-   </geometry>
-  <material name="green"/>
- </visual>
- <collision>
-   <origin xyz="0 0 0" rpy="0 0 0"/>
-   <geometry name="RWrMot3_collision">
-     <mesh filename="package://cogimon_urdf/meshes/simple/ForearmYaw.STL" scale="0.001 0.001 0.001" />
-   </geometry>
- </collision>
-</link>
-<link name="r_wrist">
-    <inertial>
-      <origin xyz="${8.2161929e-02*mmTom} ${-2.6334189*mmTom} ${-1.6465877e+01*mmTom}" rpy="0 0 0"/>
-      <mass value="3.7827821e-01"/>
-      <inertia ixx="${2.3321716e+02*mm2Tom2}"  ixy="${-2.3681435*mm2Tom2}"  ixz="${-1.8039102*mm2Tom2}" iyy="${2.0626291e+02*mm2Tom2}" iyz="${-3.1588290e+01*mm2Tom2}" izz="${2.7399881e+02*mm2Tom2}" />
-    </inertial>
-    <visual>
-      <origin xyz="0 0 0" rpy="${PI} 0 0"/>
-      <geometry name="RShp_visual">
-        <mesh filename="package://cogimon_urdf/meshes/Wrist.STL" scale="0.001 0.001 0.001" />
-      </geometry>
-      <material name="dark_grey"/>
-    </visual>
-    <collision>
-      <origin xyz="0 0 0" rpy="${PI} 0 0"/>
-      <geometry name="RShp_collision">
-        <mesh filename="package://cogimon_urdf/meshes/simple/Wrist.STL" scale="0.001 0.001 0.001" />
-      </geometry>
-    </collision>
-</link>
-<joint name="RShSag" type="revolute">
-    <parent link="DWYTorso"/>
-    <child link="RShp"/>
-    <origin xyz="${45.7475*mmTom} ${-169.137*mmTom} ${155.126*mmTom}" rpy="-0.174533 0 0.5235988" />
-    <axis xyz="0 1 0" />
-    <limit velocity="6.283" effort="140" lower="-3.359" upper="1.606" />
-    <dynamics friction="0" damping="3.0"/>
-</joint>
-<joint name="RShLat" type="revolute">
-    <parent link="RShp"/>
-    <child link="RShr"/>
-    <origin xyz="${-90.15*mmTom} ${-62*mmTom} 0" rpy="0.1745327 0 0" />
-    <axis xyz="1 0 0" />
-    <limit velocity="6.283" effort="140" lower="-3.43" upper="0.0" />
-    <dynamics friction="0" damping="3.0"/>
-</joint>
-<joint name="RShYaw" type="revolute">
-    <parent link="RShr"/>
-    <child link="RShy"/>
-    <origin xyz="${90.15*mmTom} 0 ${-218.15*mmTom}" rpy="0 0 0" />
-    <axis xyz="0 0 1" />
-    <limit velocity="6.283" effort="120" lower="-2.55" upper="2.55" />
-    <dynamics friction="0" damping="3.0"/>
-</joint>
-<joint name="RElbj" type="revolute">
-    <parent link="RShy"/>
-    <child link="RElb"/>
-    <origin xyz="${45.*mmTom} ${-55.15*mmTom} ${-74.*mmTom}" rpy="0 0 0" />
-    <axis xyz="0 1 0" />
-    <limit velocity="6.283" effort="120" lower="-2.488" upper="0.292" />
-    <dynamics friction="0" damping="3.0"/>
-</joint>
-<joint name="RForearmPlate" type="revolute">
-    <parent link="RElb"/>
-    <child link="RForearm"/>
-    <origin xyz="${-15.*mmTom} ${55.15*mmTom} ${-95.*mmTom}" rpy="0 0 0"/>
-    <axis xyz="0 0 1" />
-    <limit velocity="6.283" effort="35" lower="-2.55" upper="2.55" />
-    <dynamics friction="0" damping="0.03"/>
-</joint>
-<joint name="RWrj1" type="revolute">
-    <parent link="RForearm"/>
-    <child link="RWrMot2"/>
-    <origin xyz="0 ${-49*mmTom} ${-156.*mmTom}" rpy="0 0 0"/>
-    <axis xyz="0 1 0"/>
-    <limit velocity="6.283" effort="35" lower="-1.542" upper="1.508" />
-    <dynamics friction="0" damping="0.03"/>
-</joint>
-<joint name="RWrj2" type="revolute">
-       <parent link="RWrMot2"/>
-       <child link="RWrMot3"/>
-       <origin xyz="0 ${49*mmTom} ${-174.*mmTom}" rpy="0 0 0"/>
-       <axis xyz="0 0 1"/>
-       <limit velocity="6.283" effort="20" lower="-2.55" upper="2.55" />
-       <dynamics friction="0" damping="0.03"/>
-</joint>
-<joint name="r_wrist_joint" type="fixed">
-       <parent link="RWrMot3"/>
-       <child link="r_wrist"/>
-       <origin xyz="0 0 0" rpy="0 0 0" />
-</joint>
+<xacro:right_arm joint1_name="RShSag" joint2_name="RShLat" joint3_name="RShYaw" joint4_name="RElbj" joint5_name="RForearmPlate" joint6_name="RWrj1" joint7_name="RWrj2" />
 </xacro:if>
 <xacro:if value="${COGIMON_LEFT_ARM}">
-<!-- LEFT ARM -->
-<link name ="LShp">
-    <inertial>
-      <origin xyz="${-7.4457212*mmTom} ${3.4107960e+01*mmTom} ${1.0978102e-01*mmTom}" rpy="0 0 0"/>
-      <mass value="1.9628675"/>
-      <inertia ixx="${5.3547717e+03*mm2Tom2}"  ixy="${3.6428926e+02*mm2Tom2}"  ixz="${1.5089568e+01*mm2Tom2}" iyy="${3.3923328e+03*mm2Tom2}" iyz="${5.5692312e+01*mm2Tom2}" izz="${6.8921413e+03*mm2Tom2}" />
-    </inertial>
-    <visual>
-      <origin xyz="0 0 0" rpy="0 0 0"/>
-      <geometry name="LShp_visual">
-        <mesh filename="package://cogimon_urdf/meshes/ShoulderPitch.STL" scale="0.001 -0.001 0.001" />
-      </geometry>
-      <material name="green"/>
-    </visual>
-    <collision>
-      <origin xyz="0 0 0" rpy="0 0 0"/>
-      <geometry name="LShp_collision">
-        <mesh filename="package://cogimon_urdf/meshes/simple/ShoulderPitch.STL" scale="0.001 -0.001 0.001" />
-      </geometry>
-    </collision>
-</link>
-<link name ="LShr">
-    <inertial>
-      <origin xyz="${5.8142302e+01*mmTom} ${5.7450803e-02*mmTom} ${-7.7477683e+01*mmTom}" rpy="0 0 0"/>
-      <mass value="1.8595811"/>
-      <inertia ixx="${1.3776643e+04*mm2Tom2}"  ixy="${3.7788675e+01*mm2Tom2}"  ixz="${3.7690171e+03*mm2Tom2}" iyy="${1.5677464e+04*mm2Tom2}" iyz="${-9.4893549*mm2Tom2}" izz="${4.6317657e+03*mm2Tom2}" />
-    </inertial>
-    <visual>
-      <origin xyz="0 0 0" rpy="0 0 0"/>
-      <geometry name="LShr_visual">
-        <mesh filename="package://cogimon_urdf/meshes/ShoulderRoll.STL" scale="0.001 -0.001 0.001" />
-      </geometry>
-      <material name="dark_grey"/>
-    </visual>
-    <collision>
-      <origin xyz="0 0 0" rpy="0 0 0"/>
-      <geometry name="LShr_collision">
-        <mesh filename="package://cogimon_urdf/meshes/simple/ShoulderRoll.STL" scale="0.001 -0.001 0.001" />
-      </geometry>
-    </collision>
-</link>
-<link name ="LShy">
-    <inertial>
-      <origin xyz="${1.4625194e+01*mmTom} ${8.1726720e-01*mmTom} ${-2.8333545e+01*mmTom}" rpy="0 0 0"/>
-      <mass value="1.6678109"/>
-      <inertia ixx="${6.4480435e+03*mm2Tom2}"  ixy="${-1.5639093e+02*mm2Tom2}"  ixz="${1.2205359e+03*mm2Tom2}" iyy="${7.3372077e+03*mm2Tom2}" iyz="${8.9941532e+01*mm2Tom2}" izz="${3.6738448e+03*mm2Tom2}" />
-    </inertial>
-    <visual>
-      <origin xyz="0 0 0" rpy="0 0 0"/>
-      <geometry name="LShy_visual">
-        <mesh filename="package://cogimon_urdf/meshes/ShoulderYaw.STL" scale="0.001 -0.001 0.001" />
-      </geometry>
-      <material name="green"/>
-    </visual>
-    <collision>
-      <origin xyz="0 0 0" rpy="0 0 0"/>
-      <geometry name="LShy_collision">
-        <mesh filename="package://cogimon_urdf/meshes/simple/ShoulderYaw.STL" scale="0.001 -0.001 0.001" />
-      </geometry>
-    </collision>
-</link>
-<link name ="LElb">
- <inertial>
-   <origin xyz="${-7.6833067*mmTom} ${-4.0302205e+01*mmTom} ${-4.3492779e+01*mmTom}" rpy="0 0 0"/>
-   <mass value="1.3157289"/>
-   <inertia ixx="${4.3303940e+03*mm2Tom2}"  ixy="${-1.1737391e+02*mm2Tom2}"  ixz="${-4.1923199e+02*mm2Tom2}" iyy="${3.8539919e+03*mm2Tom2}" iyz="${-7.9573038e+02*mm2Tom2}" izz="${1.7594689e+03*mm2Tom2}" />
- </inertial>
- <visual>
-   <origin xyz="0 0 0" rpy="0 0 0"/>
-   <geometry name="LElb_visual">
-     <mesh filename="package://cogimon_urdf/meshes/Elbow.STL" scale="0.001 -0.001 0.001" />
-   </geometry>
-  <material name="dark_grey"/>
- </visual>
- <collision>
-   <origin xyz="0 0 0" rpy="0 0 0"/>
-   <geometry name="LElb_collision">
-     <mesh filename="package://cogimon_urdf/meshes/simple/Elbow.STL" scale="0.001 -0.001 0.001" />
-   </geometry>
- </collision>
-</link>
-<link name ="LForearm">
- <inertial>
-   <origin xyz="${-1.1079615e-01*mmTom} ${1.1590836e+01*mmTom} ${-7.8160260e+01*mmTom}" rpy="0 0 0"/>
-   <mass value="1.4908547"/>
-   <inertia ixx="${8.5692128e+03*mm2Tom2}"  ixy="${1.7856252e+01*mm2Tom2}"  ixz="${1.9379365e+01*mm2Tom2}" iyy="${7.7454159e+03*mm2Tom2}" iyz="${-3.2860094e+02*mm2Tom2}" izz="${2.7441921e+03*mm2Tom2}" />
- </inertial>
- <visual>
-   <origin xyz="0 0 0" rpy="0 0 0"/>
-   <geometry name="LForearm_visual">
-     <mesh filename="package://cogimon_urdf/meshes/Forearm.STL" scale="0.001 -0.001 0.001" />
-   </geometry>
-  <material name="green"/>
- </visual>
- <collision>
-   <origin xyz="0 0 0" rpy="0 0 0"/>
-   <geometry name="LForearm_collision">
-     <mesh filename="package://cogimon_urdf/meshes/simple/Forearm.STL" scale="0.001 -0.001 0.001" />
-   </geometry>
- </collision>
-</link>
-<link name="LWrMot2">
- <inertial>
-   <origin xyz="${-4.6502396e-03*mmTom} ${-3.8014094e+01*mmTom} ${-6.9926878e+01*mmTom}" rpy="0 0 0"/>
-   <mass value="1.1263612"/>
-   <inertia ixx="${5.1871784e+03*mm2Tom2}"  ixy="${2.7244370e+01*mm2Tom2}"  ixz="${2.2833496*mm2Tom2}" iyy="${4.8037789e+03*mm2Tom2}" iyz="${-7.2165653e+02*mm2Tom2}" izz="${1.2771388e+03*mm2Tom2}" />
- </inertial>
- <visual>
-   <origin xyz="0 0 0" rpy="0 0 0"/>
-   <geometry name="LWrMot2_visual">
-     <mesh filename="package://cogimon_urdf/meshes/ForearmPitch.STL" scale="0.001 -0.001 0.001" />
-   </geometry>
-  <material name="dark_grey"/>
- </visual>
- <collision>
-   <origin xyz="0 0 0" rpy="0 0 0"/>
-   <geometry name="LWrMot2_collision">
-     <mesh filename="package://cogimon_urdf/meshes/simple/ForearmPitch.STL" scale="0.001 -0.001 0.001" />
-   </geometry>
- </collision>
-</link>
-<link name="LWrMot3">
- <inertial>
-   <origin xyz="0 0 ${3.1270570e+01*mmTom}" rpy="0 0 0"/>
-   <mass value="2.7966428e-01"/>
-   <inertia ixx="${1.4415192e+02*mm2Tom2}"  ixy="${9.8651826e-02*mm2Tom2}"  ixz="0" iyy="${1.4417010e+02*mm2Tom2}" iyz="0" izz="${6.0500616e+01*mm2Tom2}" />
- </inertial>
- <visual>
-   <origin xyz="0 0 0" rpy="0 0 0"/>
-   <geometry name="LWrMot3_visual">
-     <mesh filename="package://cogimon_urdf/meshes/ForearmYaw.STL" scale="0.001 -0.001 0.001" />
-   </geometry>
-  <material name="green"/>
- </visual>
- <collision>
-   <origin xyz="0 0 0" rpy="0 0 0"/>
-   <geometry name="LWrMot3_collision">
-     <mesh filename="package://cogimon_urdf/meshes/simple/ForearmYaw.STL" scale="0.001 -0.001 0.001" />
-   </geometry>
- </collision>
-</link>
-<link name="l_wrist">
-    <inertial>
-      <origin xyz="${8.2161929e-02*mmTom} ${2.6334189*mmTom} ${-1.6465877e+01*mmTom}" rpy="0 0 0"/>
-      <mass value="3.7827821e-01"/>
-      <inertia ixx="${2.3321716e+02*mm2Tom2}"  ixy="${2.3681435*mm2Tom2}"  ixz="${-1.8039102*mm2Tom2}" iyy="${2.0626291e+02*mm2Tom2}" iyz="${3.1588290e+01*mm2Tom2}" izz="${2.7399881e+02*mm2Tom2}" />
-    </inertial>
-    <visual>
-      <origin xyz="0 0 0" rpy="${PI} 0 0"/>
-      <geometry name="LShp_visual">
-        <mesh filename="package://cogimon_urdf/meshes/Wrist.STL" scale="0.001 -0.001 0.001" />
-      </geometry>
-      <material name="dark_grey"/>
-    </visual>
-    <collision>
-      <origin xyz="0 0 0" rpy="${PI} 0 0"/>
-      <geometry name="LShp_collision">
-        <mesh filename="package://cogimon_urdf/meshes/simple/Wrist.STL" scale="0.001 -0.001 0.001" />
-      </geometry>
-    </collision>
-</link>
-<joint name="LShSag" type="revolute">
-    <parent link="DWYTorso"/>
-    <child link="LShp"/>
-    <origin xyz="${45.7475*mmTom} ${169.137*mmTom} ${155.126*mmTom}" rpy="0.174533 0 -0.5235988" />
-    <axis xyz="0 1 0" />
-    <limit velocity="6.283" effort="140" lower="-3.352" upper="1.603" />
-    <dynamics friction="0" damping="3.0"/>
-</joint>
-<joint name="LShLat" type="revolute">
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