Commit message: added wcf to torso

File: cogimon_urdf/urdf/parts/torso.urdf.xacro (robot description, xacro)
@@ -12,6 +12,6 @@
     <inertial>
       <origin xyz="4.2999707E-4 -0.0097650317 0.033011157" rpy="0 0 0"/>
-      <mass value="0.54588774"/>
-      <inertia ixx="9.7126578E-4"  ixy="-7.2101244E-7"  ixz="1.1440119E-6" iyy="7.4686706E-4" iyz="-1.7450917E-4" izz="6.2196235E-4" />
+      <mass value="${wcf*0.54588774}"/>
+      <inertia ixx="${wcf*9.7126578E-4}"  ixy="${wcf*-7.2101244E-7}"  ixz="${wcf*1.1440119E-6}" iyy="${wcf*7.4686706E-4}" iyz="${wcf*-1.7450917E-4}" izz="${wcf*6.2196235E-4}" />
     </inertial>
     <visual>
@@ -32,6 +32,6 @@
     <inertial>
       <origin xyz="-0.0021273416 0.0033575235 -0.0010076896" rpy="0 0 0"/>
-      <mass value="0.75398402"/>
-      <inertia ixx="3.4093348E-4"  ixy="-6.2120042E-6"  ixz="-1.3863473E-6" iyy="3.9581916E-4" iyz="1.443019E-6" izz="3.7449753E-4" />
+      <mass value="${wcf*0.75398402}"/>
+      <inertia ixx="${wcf*3.4093348E-4}"  ixy="${wcf*-6.2120042E-6}"  ixz="${wcf*-1.3863473E-6}" iyy="${wcf*3.9581916E-4}" iyz="${wcf*1.443019E-6}" izz="${wcf*3.7449753E-4}" />
     </inertial>
     <visual>
@@ -52,6 +52,6 @@
     <inertial>
       <origin xyz="-0.0358501 1.8286043E-5 0.117557148" rpy="0 0 0"/>
-      <mass value="6.3617175"/>
-      <inertia ixx="0.034089342"  ixy="-9.8308572E-6"  ixz="-7.5649290E-4" iyy="0.030117357" iyz="6.2443771E-6" izz="0.025296582" />
+      <mass value="${wcf*6.3617175}"/>
+      <inertia ixx="${wcf*0.034089342}"  ixy="${wcf*-9.8308572E-6}"  ixz="${wcf*-7.5649290E-4}" iyy="${wcf*0.030117357}" iyz="${wcf*6.2443771E-6}" izz="${wcf*0.025296582}" />
     </inertial>
     <visual>

Commit message: Set torso pitch as fixed, set torso lateral as revolute

File: cogimon_urdf/urdf/parts/torso.urdf.xacro (robot description, xacro)
@@ -75,16 +75,20 @@
     <origin xyz="-0.014976503999999998 0 0.15770847" rpy="0 0 0" />
 </joint>
-<joint name="WaistLat" type="fixed">
+<joint name="WaistLat" type="revolute">
     <parent link="Waist"/>
     <child link="DWL"/>
     <origin xyz="0.020281504 0 0.11912053" rpy="0 0 0" />
+    <axis xyz="${cos_20} 0 ${sin_20}" />
+    <limit velocity="4.0" effort="80" lower="-0.5236" upper="0.5235" />
+    <!-- dynamics friction="0" damping="0.3"/ -->
+    <dynamics friction="0" damping="3.0"/>
 </joint>
-  <joint name="WaistSag" type="revolute">
+  <joint name="WaistSag" type="fixed">
     <parent link="DWL"/>
     <child link="DWS"/>
     <origin xyz="0 0 0" rpy="0 0 0" />
-    <axis xyz="0 1 0" />
+    <!--axis xyz="0 1 0" />
     <limit velocity="4.0" effort="80" lower="-0.3491" upper="0.8727" />
-    <dynamics friction="0" damping="3.0"/>
+    <dynamics friction="0" damping="3.0"/-->
   </joint>
   <joint name="WaistYaw" type="revolute">

Commit message: Added weight

File: cogimon_urdf/urdf/parts/torso.urdf.xacro (robot description, xacro)
@@ -2,4 +2,9 @@
 <robot xmlns:xacro="http://ros.org/wiki/xacro">
 <xacro:if value="${COGIMON_TORSO}" >
+<xacro:property name="d" value="0.11" /> <!-- weight diameter -->
+<xacro:property name="r" value="${d/2.}" /> <!-- weight radius -->
+<xacro:property name="h" value="${3.0*0.02}" /> <!-- weight height, here we consider three discs -->
+<xacro:property name="m" value="30.0" /> <!-- weight mass -->
+<xacro:property name="z" value="0.2" /><!-- weight position -->
 <!-- LINKS -->
 <link name ="DWL">
@@ -24,4 +29,23 @@
 </link>
 <xacro:if value="${COGIMON_PENNACCHIO}" >
+<link name ="weight">
+     <inertial>
+      <origin xyz="0 0 0 " rpy="0 0 0"/>
+      <mass value="${m}"/>
+      <inertia ixx="${(1./12.)*m*(3.*r*r+h*h)}"  ixy="0"  ixz="0" iyy="${(1./12.)*m*(3.*r*r+h*h)}" iyz="0" izz="${(m*r*r)/2.}" />
+    </inertial>
+    <visual>
+      <origin rpy="0 0 0" xyz="0 0 0"/>
+      <geometry>
+       <cylinder length="${h}" radius="${r}"/>
+      </geometry>
+    </visual>
+    <collision>
+      <origin rpy="0 0 0" xyz="0 0 0"/>
+      <geometry>
+       <cylinder length="${h}" radius="${r}"/>
+      </geometry>
+    </collision>
+</link>
 <link name ="pennacchio">
     <inertial>
@@ -60,4 +84,9 @@
     <origin xyz="${-54.0957*mmTom} 0.0 ${66.5*mmTom}" rpy="0 0 0" />
 </joint>
+<joint name="weight_frame" type="fixed">
+    <parent link="pennacchio"/>
+    <child link="weight"/>
+    <origin xyz="0. 0. ${z}" rpy="0 0 0" />
+</joint>
 </xacro:if>
 </xacro:if>

Commit message: Committed files for the mockup of the upperbody

File: cogimon_urdf/urdf/parts/torso.urdf.xacro (robot description, xacro)
@@ -29,5 +29,5 @@
 </link>
 <xacro:if value="${COGIMON_PENNACCHIO}" >
-<link name ="weight">
+<!--link name ="weight">
      <inertial>
       <origin xyz="0 0 0 " rpy="0 0 0"/>
@@ -67,5 +67,5 @@
       </geometry>
     </collision>
-</link>
+</link-->
 </xacro:if>
 <!-- JOINTS -->
@@ -79,5 +79,5 @@
 </joint>
 <xacro:if value="${COGIMON_PENNACCHIO}" >
-<joint name="pennacchio_frame" type="fixed">
+<!--joint name="pennacchio_frame" type="fixed">
     <parent link="DWL"/>
     <child link="pennacchio"/>
@@ -88,5 +88,6 @@
     <child link="weight"/>
     <origin xyz="0. 0. ${z}" rpy="0 0 0" />
-</joint>
+</joint-->
+<xacro:include filename="$(find cogimon_urdf)/urdf/parts/whole_upper_body.urdf.xacro" />
 </xacro:if>
 </xacro:if>

Commit message: Added torso frame

File: cogimon_urdf/urdf/parts/torso.urdf.xacro (robot description, xacro)
@@ -110,4 +110,5 @@
     </collision>
 </link>
+<link name="torso"/>
 </xacro:unless>
 <!-- JOINTS -->
@@ -146,4 +147,9 @@
     <dynamics friction="0" damping="3.0"/>
 </joint>
+<joint name="torso_joint" type="fixed">
+    <parent link="DWYTorso"/>
+    <child link="torso"/>
+    <origin xyz="0.0 0.0 ${155.126*mmTom}" rpy="0 0 0" />
+</joint>
 </xacro:unless>
 </xacro:if>
