Commit message: head limit updated based on Phil suggestion.

File: cogimon_urdf/urdf/parts/head.urdf.xacro (robot description, xacro)
@@ -62,5 +62,5 @@
     <origin xyz="${49.6*mmTom} 0.0 ${90.*mmTom}" rpy="0 0 0" />
     <axis xyz="1 0 0" />
-    <limit velocity="6.283" effort="120" lower="${-355*toRad}" upper="${355*toRad}" /> <!-- TODO: CHECK THESE VALUES!!! -->
+    <limit velocity="6.283" effort="20" lower="-2.5" upper="2.5" /> <!-- TODO: CHECK THESE VALUES!!! -->
     <dynamics friction="0" damping="3.0"/>
   </joint>

Commit message: Fixed angular offset in hokuyo mesh

File: cogimon_urdf/urdf/parts/head.urdf.xacro (robot description, xacro)
@@ -30,5 +30,5 @@
     </inertial>
     <visual>
-      <origin xyz="0.0 0.0 0.0" rpy="0 0 0"/>
+      <origin xyz="0.0 0.0 0.0" rpy="${-45.0*toRad} 0 0"/>
       <geometry name="Neck_visual">
         <mesh filename="package://cogimon_urdf/meshes/HeadRoll.stl" scale="${mmTom} ${mmTom} ${mmTom}" />
@@ -37,5 +37,5 @@
     </visual>
     <collision>
-      <origin xyz="0.0 0.0 0.0" rpy="0 0 0"/>
+      <origin xyz="0.0 0.0 0.0" rpy="${-45.0*toRad} 0 0"/>
       <geometry name="Neck_collision">
         <mesh filename="package://cogimon_urdf/meshes/simple/HeadRoll.stl" scale="${mmTom} ${mmTom} ${mmTom}" />

Commit message: Integrated head in model

File: cogimon_urdf/urdf/parts/head.urdf.xacro (robot description, xacro)
@@ -3,14 +3,14 @@
 <xacro:if value="${COGIMON_HEAD}" >
 <!-- LINKS -->
-<link name ="Neck">
+<link name ="Head">
     <inertial>
-      <origin xyz="${1.9525578e+01*mmTom} ${8.7785097e-02*mmTom} ${7.3374976e+01*mmTom} " rpy="0 0 0"/>
-      <mass value="2.3794941e-01"/>
-      <inertia ixx="${2.8460315e+02*mm2Tom2}"  ixy="${-5.4194691e-01*mm2Tom2}"  ixz="${-7.3250232e+01*mm2Tom2}" iyy="${4.5308750e+02*mm2Tom2}" iyz="${-9.4474115e-02*mm2Tom2}" izz="${2.7675534e+02*mm2Tom2}" />
+      <origin xyz="${5.7448518e+01*mmTom} ${1.6262687e-02*mmTom} ${1.3030019e+02*mmTom} " rpy="0 0 0"/>
+      <mass value="1.2626010"/>
+      <inertia ixx="${8.8669451e+03*mm2Tom2}"  ixy="${-4.5839239e-01*mm2Tom2}"  ixz="${-1.7240170e+03*mm2Tom2}" iyy="${1.1716158e+04*mm2Tom2}" iyz="${-2.6031540e-01*mm2Tom2}" izz="${7.9021213e+03*mm2Tom2}" />
     </inertial>
     <visual>
       <origin xyz="0.0 0.0 0.0" rpy="0 0 0"/>
-      <geometry name="Neck_visual">
-        <mesh filename="package://cogimon_urdf/meshes/NeckFixed.stl" scale="${mmTom} ${mmTom} ${mmTom}" />
+      <geometry name="Head_visual">
+        <mesh filename="package://cogimon_urdf/meshes/Head.stl" scale="${mmTom} ${mmTom} ${mmTom}" />
       </geometry>
       <material name="dark_grey"/>
@@ -18,52 +18,45 @@
     <collision>
       <origin xyz="0.0 0.0 0.0" rpy="0 0 0"/>
-      <geometry name="Neck_collision">
-        <mesh filename="package://cogimon_urdf/meshes/simple/NeckFixed.stl" scale="${mmTom} ${mmTom} ${mmTom}" />
+      <geometry name="Head_collision">
+        <mesh filename="package://cogimon_urdf/meshes/simple/Head.stl" scale="${mmTom} ${mmTom} ${mmTom}" />
       </geometry>
     </collision>
 </link>
-<link name ="HeadHokuyo"> <!-- TODO: CHECK THESE VALUES!!! -->
+<link name ="HeadHokuyo">
     <inertial>
-      <origin xyz="${5.5322369e+01*mmTom} ${1.8472201e+01*mmTom} ${-1.8483703e+01*mmTom} " rpy="0 0 0"/>
-      <mass value="5.4611797e-01"/>
-      <inertia ixx="${1.9756996e+03*mm2Tom2}"  ixy="${-1.1287972e+02*mm2Tom2}"  ixz="${1.1284571e+02*mm2Tom2}" iyy="${4.4030675e+03*mm2Tom2}" iyz="${4.9540219e+02*mm2Tom2}" izz="${4.4027914e+03*mm2Tom2}" />
+      <origin xyz="${5.4246456e+01*mmTom} ${-9.3963721e-03*mmTom} ${-2.5596890e+01*mmTom} " rpy="0 0 0"/>
+      <mass value="5.5751693e-01"/>
+      <inertia ixx="${1.9833413e+03*mm2Tom2}"  ixy="${-7.2298853e-02*mm2Tom2}"  ixz="${1.7498835e+02*mm2Tom2}" iyy="${4.9368962e+03*mm2Tom2}" iyz="${-1.1129001e-01*mm2Tom2}" izz="${3.9384326e+03*mm2Tom2}" />
     </inertial>
-    <visual>
-      <origin xyz="0.0 0.0 0.0" rpy="${-45.0*toRad} 0 0"/>
-      <geometry name="Neck_visual">
-        <mesh filename="package://cogimon_urdf/meshes/HeadRoll.stl" scale="${mmTom} ${mmTom} ${mmTom}" />
-      </geometry>
-      <material name="dark_grey"/>
-    </visual>
-    <collision>
-      <origin xyz="0.0 0.0 0.0" rpy="${-45.0*toRad} 0 0"/>
-      <geometry name="Neck_collision">
-        <mesh filename="package://cogimon_urdf/meshes/simple/HeadRoll.stl" scale="${mmTom} ${mmTom} ${mmTom}" />
-      </geometry>
-    </collision>
 </link>
 <!-- JOINTS -->
 <joint name="neck_frame" type="fixed">
     <parent link="DWYTorso"/>
-    <child link="Neck"/>
-    <origin xyz="${16.*mmTom} 0.0 ${196.5*mmTom}" rpy="0 0 0" />
+    <child link="Head"/>
+    <origin xyz="0.0 0.0 ${196.5*mmTom}" rpy="0 0 0" />
 </joint>
 <xacro:if value="${COGIMON_LASER_FIXED}">
   <joint name="head_roll" type="fixed">
-    <parent link="Neck"/>
+    <parent link="Head"/>
     <child link="HeadHokuyo"/>
-    <origin xyz="${49.6*mmTom} 0.0 ${90.*mmTom}" rpy="0 0 0" />
+    <origin xyz="0.0853 0.0 0.1506" rpy="0 0.3491 0" />
   </joint>
 </xacro:if>
 <xacro:unless value="${COGIMON_LASER_FIXED}">
   <joint name="head_roll" type="revolute">
-    <parent link="Neck"/>
+    <parent link="Head"/>
     <child link="HeadHokuyo"/>
-    <origin xyz="${49.6*mmTom} 0.0 ${90.*mmTom}" rpy="0 0 0" />
+    <origin xyz="0.0853 0.0 0.1506" rpy="0 0.3491 0" />
     <axis xyz="1 0 0" />
-    <limit velocity="6.283" effort="20" lower="-2.5" upper="2.5" /> <!-- TODO: CHECK THESE VALUES!!! -->
+    <limit velocity="6.283" effort="20" lower="-100." upper="100." />
     <dynamics friction="0" damping="3.0"/>
   </joint>
 </xacro:unless>
+<link name="HokuyoLaser"/>
+<joint name="HokuyoLaser_joint" type="fixed">
+    <parent link="HeadHokuyo"/>
+    <child link="HokuyoLaser"/>
+    <origin xyz="${65.2577*mmTom} 0.0 0.0" rpy="0 0 0" />
+  </joint>
 </xacro:if>
 </robot>
