Commit message: added useful ref frame at ball tip

File: cogimon_urdf/urdf/parts/ball_endeff.urdf.xacro (robot description, xacro)
@@ -24,4 +24,5 @@
 </link>
 <link name="r_wrist"/>
+<link name="r_ball_tip"/>
 <joint name="r_wrist_joint" type="fixed">
        <parent link="RWrMot3"/>
@@ -33,4 +34,9 @@
 <child link="RBall"/>
 <origin xyz="0 0 0" rpy="0 0 0"/>
+</joint>
+<joint name="r_ball_tipj" type="fixed">
+<parent link="RBall"/>
+<child link="r_ball_tip"/>
+<origin xyz="0 0 -0.07" rpy="0 0 0"/>
 </joint>
 </xacro:if>
@@ -57,4 +63,5 @@
 </link>
 <link name="l_wrist"/>
+<link name="l_ball_tip"/>
 <joint name="l_wrist_joint" type="fixed">
        <parent link="LWrMot3"/>
@@ -68,4 +75,9 @@
 <origin xyz="0 0 0" rpy="0 0 0"/>
 </joint>
+<joint name="l_ball_tipj" type="fixed">
+<parent link="LBall"/>
+<child link="l_ball_tip"/>
+<origin xyz="0 0 -0.07" rpy="0 0 0"/>
+</joint>
 </xacro:if>
 </robot>

Commit message: Added TCP_L and TCP_R frames in balls

File: cogimon_urdf/urdf/parts/ball_endeff.urdf.xacro (robot description, xacro)
@@ -40,4 +40,10 @@
 <origin xyz="0 0 -0.07" rpy="0 0 0"/>
 </joint>
+<link name="TCP_R"/>
+<joint name="TCP_R_joint" type="fixed">
+       <parent link="r_ball_tip"/>
+       <child link="TCP_R"/>
+       <origin xyz="0 0 0" rpy="0 ${PI} 0" />
+</joint>
 </xacro:if>
 <xacro:if value="${COGIMON_LEFT_ARM}">
@@ -69,4 +75,10 @@
        <origin xyz="0 0 0" rpy="0 0 0" />
 </joint>
+<link name="TCP_L"/>
+<joint name="TCP_L_joint" type="fixed">
+       <parent link="l_ball_tip"/>
+       <child link="TCP_L"/>
+       <origin xyz="0 0 0" rpy="0 ${PI} 0" />
+</joint>
 <!-- JOINTS -->
 <joint name="l_handj" type="fixed">

Commit message: Added extra frames on ball end effector

File: cogimon_urdf/urdf/parts/ball_endeff.urdf.xacro (robot description, xacro)
@@ -40,4 +40,28 @@
 <origin xyz="0 0 -0.07" rpy="0 0 0"/>
 </joint>
+<link name="r_ball_tip_u"/>
+<joint name="r_ball_tipj_u" type="fixed">
+<parent link="RBall"/>
+<child link="r_ball_tip_u"/>
+<origin xyz="0.07 0 0" rpy="0 0 0"/>
+</joint>
+<link name="r_ball_tip_d"/>
+<joint name="r_ball_tipj_d" type="fixed">
+<parent link="RBall"/>
+<child link="r_ball_tip_d"/>
+<origin xyz="-0.07 0 0" rpy="0 0 0"/>
+</joint>
+<link name="r_ball_tip_l"/>
+<joint name="r_ball_tipj_l" type="fixed">
+<parent link="RBall"/>
+<child link="r_ball_tip_l"/>
+<origin xyz="0 0.07 0" rpy="0 0 0"/>
+</joint>
+<link name="r_ball_tip_r"/>
+<joint name="r_ball_tipj_r" type="fixed">
+<parent link="RBall"/>
+<child link="r_ball_tip_r"/>
+<origin xyz="0 -0.07 0" rpy="0 0 0"/>
+</joint>
 <link name="TCP_R"/>
 <joint name="TCP_R_joint" type="fixed">
@@ -75,4 +99,28 @@
        <origin xyz="0 0 0" rpy="0 0 0" />
 </joint>
+<link name="l_ball_tip_u"/>
+<joint name="l_ball_tipj_u" type="fixed">
+<parent link="LBall"/>
+<child link="l_ball_tip_u"/>
+<origin xyz="0.07 0 0" rpy="0 0 0"/>
+</joint>
+<link name="l_ball_tip_d"/>
+<joint name="l_ball_tipj_d" type="fixed">
+<parent link="LBall"/>
+<child link="l_ball_tip_d"/>
+<origin xyz="-0.07 0 0" rpy="0 0 0"/>
+</joint>
+<link name="l_ball_tip_l"/>
+<joint name="l_ball_tipj_l" type="fixed">
+<parent link="LBall"/>
+<child link="l_ball_tip_l"/>
+<origin xyz="0 0.07 0" rpy="0 0 0"/>
+</joint>
+<link name="l_ball_tip_r"/>
+<joint name="l_ball_tipj_r" type="fixed">
+<parent link="LBall"/>
+<child link="l_ball_tip_r"/>
+<origin xyz="0 -0.07 0" rpy="0 0 0"/>
+</joint>
 <link name="TCP_L"/>
 <joint name="TCP_L_joint" type="fixed">
