Commit message: Added new joints and links

File: cogimon_urdf/urdf/cogimon_robot.urdf.xacro (robot description, xacro)
@@ -19,4 +19,4 @@
     <child link="base_link"/>
   </joint>
-<origin xyz="0.0 0.0 0.8" rpy="0 0 0" />
+<origin xyz="0.0 0.0 1.0" rpy="0 0 0" />
 </robot>

File: cogimon_urdf/urdf/gazebo/cogimon_materials.gazebo.xacro (robot description, xacro)
@@ -14,4 +14,7 @@
   <material>Gazebo/Green</material>
 </gazebo>
+<gazebo reference="RLowLeg">
+  <material>Gazebo/DarkGrey</material>
+</gazebo>
 </xacro:if>
 <xacro:if value="${COGIMON_LEFT_LEG}" >
@@ -25,4 +28,7 @@
   <material>Gazebo/Green</material>
 </gazebo>
+<gazebo reference="LLowLeg">
+  <material>Gazebo/DarkGrey</material>
+</gazebo>
 </xacro:if>
 </robot>

File: cogimon_urdf/urdf/parts/legs.urdf.xacro (robot description, xacro)
@@ -60,4 +60,24 @@
       <geometry name="LThighLowLeg_collision">
         <mesh filename="package://cogimon_urdf/meshes/simple/HipYaw.stl" scale="${mmTom} ${mmTom} ${mmTom}" />
+      </geometry>
+    </collision>
+</link>
+<link name ="LLowLeg">
+    <inertial>
+      <origin xyz="${2.7363015e+01*mmTom} ${-5.7802070e+01*mmTom} ${-1.9306454e+02*mmTom}" rpy="0 0 0"/>
+      <mass value="3.7014912"/>
+      <inertia ixx="${6.4669769e+04*mm2Tom2}"  ixy="${3.6914631e+02*mm2Tom2}"  ixz="${5.3710941e+03 *mm2Tom2}" iyy="${6.3323486e+04*mm2Tom2}" iyz="${-2.7319883e+03*mm2Tom2}" izz="${8.1842652e+03*mm2Tom2}" />
+    </inertial>
+    <visual>
+      <origin xyz="0. 0. 0." rpy="0 0 0."/>
+      <material name="dark_grey"/>
+      <geometry name="LLowLeg_visual">
+        <mesh filename="package://cogimon_urdf/meshes/KneePitch.stl" scale="${mmTom} ${mmTom} ${mmTom}" />
+      </geometry>
+    </visual>
+    <collision>
+      <origin xyz="0.0 0. 0" rpy="0 0 0."/>
+      <geometry name="LLowLeg_collision">
+        <mesh filename="package://cogimon_urdf/meshes/simple/KneePitch.stl" scale="${mmTom} ${mmTom} ${mmTom}" />
       </geometry>
     </collision>
@@ -88,4 +108,12 @@
     <dynamics friction="0" damping="3.0"/>
 </joint>
+<joint name="LKneePitch" type="revolute">
+    <parent link="LThighLowLeg"/>
+    <child link="LLowLeg"/>
+    <origin xyz="${-39.*mmTom} ${64.1*mmTom} ${-60.7*mmTom}" rpy="0 0 0" />
+    <axis xyz="0 1 0" />
+    <limit velocity="3.67" effort="176" lower="${-90.*toRad}" upper="${90.*toRad}" />
+    <dynamics friction="0" damping="3.0"/>
+</joint>
 </xacro:if>
 <xacro:if value="${COGIMON_RIGHT_LEG}" >
@@ -148,4 +176,24 @@
       <geometry name="RThighLowLeg_collision">
         <mesh filename="package://cogimon_urdf/meshes/simple/HipYaw.stl" scale="${mmTom} ${-mmTom} ${mmTom}" />
+      </geometry>
+    </collision>
+</link>
+<link name ="RLowLeg">
+    <inertial>
+      <origin xyz="${2.7363015e+01*mmTom} ${5.7802070e+01*mmTom} ${-1.9306454e+02*mmTom}" rpy="0 0 0"/>
+      <mass value="3.7014912"/>
+      <inertia ixx="${6.4669769e+04*mm2Tom2}"  ixy="${-3.6914631e+02*mm2Tom2}"  ixz="${5.3710941e+03 *mm2Tom2}" iyy="${6.3323486e+04*mm2Tom2}" iyz="${2.7319883e+03*mm2Tom2}" izz="${8.1842652e+03*mm2Tom2}" />
+    </inertial>
+    <visual>
+      <origin xyz="0. 0. 0." rpy="0 0 0."/>
+      <material name="dark_grey"/>
+      <geometry name="RLowLeg_visual">
+        <mesh filename="package://cogimon_urdf/meshes/KneePitch.stl" scale="${mmTom} ${-mmTom} ${mmTom}" />
+      </geometry>
+    </visual>
+    <collision>
+      <origin xyz="0.0 0. 0" rpy="0 0 0."/>
+      <geometry name="RLowLeg_collision">
+        <mesh filename="package://cogimon_urdf/meshes/simple/KneePitch.stl" scale="${mmTom} ${-mmTom} ${mmTom}" />
       </geometry>
     </collision>
@@ -176,4 +224,12 @@
     <dynamics friction="0" damping="3.0"/>
 </joint>
+<joint name="RKneePitch" type="revolute">
+    <parent link="RThighLowLeg"/>
+    <child link="RLowLeg"/>
+    <origin xyz="${-39.*mmTom} ${-64.1*mmTom} ${-60.7*mmTom}" rpy="0 0 0" />
+    <axis xyz="0 1 0" />
+    <limit velocity="3.67" effort="176" lower="${-90.*toRad}" upper="${90.*toRad}" />
+    <dynamics friction="0" damping="3.0"/>
+</joint>
 </xacro:if>
 </robot>
