Commit message: Added weight factor correction, changed weight of waist and upper arms

File: cogimon_urdf/urdf/cogimon.urdf.xacro (robot description, xacro)
@@ -27,4 +27,5 @@
 	</joint>
 </xacro:unless>
+<xacro:property name="wcf" value="1.3" />
 <!-- ************ COGIMON BASE ************** -->
 <xacro:include filename="$(find cogimon_urdf)/urdf/cogimon_base.urdf.xacro"/>

File: cogimon_urdf/urdf/cogimon_base.urdf.xacro (robot description, xacro)
@@ -16,6 +16,6 @@
     <inertial>
       <origin xyz="-0.026391145 -5.8216364E-4 0.052632312" rpy="0.0 0.0 0.0"/>
-      <mass value="1.8008695"/>
-      <inertia ixx="0.0051032982"  ixy="-5.7170981E-5"  ixz="0.0016920543" iyy="0.006241636" iyz="1.7225949E-5" izz="0.0024517762" />
+      <mass value="${wcf*1.8008695}"/>
+      <inertia ixx="${wcf*0.0051032982}"  ixy="${wcf*-5.7170981E-5}"  ixz="${wcf*0.0016920543}" iyy="${wcf*0.006241636}" iyz="${wcf*1.7225949E-5}" izz="${wcf*0.0024517762}" />
     </inertial>
     <visual>

File: cogimon_urdf/urdf/parts/arms.urdf.xacro (robot description, xacro)
@@ -8,6 +8,6 @@
     <inertial>
       <origin xyz="0.0099500565 -0.038682024 1.6446924E-4" rpy="0 0 0"/>
-      <mass value="0.56782202"/>
-      <inertia ixx="7.8337456E-4"  ixy="1.9035768E-4"  ixz="-3.0037676E-6" iyy="6.3399921E-4" iyz="4.3840774E-6" izz="0.001008054" />
+      <mass value="${wcf*0.56782202}"/>
+      <inertia ixx="${wcf*7.8337456E-4}"  ixy="${wcf*1.9035768E-4}"  ixz="${wcf*-3.0037676E-6}" iyy="${wcf*6.3399921E-4}" iyz="${wcf*4.3840774E-6}" izz="${wcf*0.001008054}" />
     </inertial>
     <visual>
@@ -28,6 +28,6 @@
     <inertial>
       <origin xyz="-0.0038936743 2.2022151E-6 -0.0048616005" rpy="0 0 0"/>
-      <mass value="0.77683752"/>
-      <inertia ixx="4.5812904E-4"  ixy="-2.4111086E-7"  ixz="9.2521185E-6" iyy="4.3089204E-4" iyz="-4.7216950E-7" izz="3.4174855E-4" />
+      <mass value="${wcf*0.77683752}"/>
+      <inertia ixx="${wcf*4.5812904E-4}"  ixy="${wcf*-2.4111086E-7}"  ixz="${wcf*9.2521185E-6}" iyy="${wcf*4.3089204E-4}" iyz="${wcf*-4.7216950E-7}" izz="${wcf*3.4174855E-4}" />
     </inertial>
     <visual>
@@ -48,6 +48,6 @@
     <inertial>
       <origin xyz="0.0022714213 -0.0071091517 -0.057455221" rpy="0 0 0"/>
-      <mass value="1.0462304"/>
-      <inertia ixx="0.0030934574"  ixy="6.6702837E-5"  ixz="3.0222291E-4" iyy="0.0029181573" iyz="-5.2663661E-4" izz="8.0830389E-4" />
+      <mass value="${wcf*1.0462304}"/>
+      <inertia ixx="${wcf*0.0030934574}"  ixy="${wcf*6.6702837E-5}"  ixz="${wcf*3.0222291E-4}" iyy="${wcf*0.0029181573}" iyz="${wcf*-5.2663661E-4}" izz="${wcf*8.0830389E-4}" />
     </inertial>
     <visual>
@@ -68,6 +68,6 @@
         <inertial>
           <origin xyz="-6.5553403E-4 -9.3464748E-4 -9.3101289E-4" rpy="0 0 0"/>
-          <mass value="0.63306933"/>
-          <inertia ixx="2.2599075E-4"  ixy="-2.6376470E-7"  ixz="-9.8007285E-6" iyy="2.7781302E-4" iyz="-2.0435288E-6" izz="2.1878992E-4" />
+          <mass value="${wcf*0.63306933}"/>
+          <inertia ixx="${wcf*2.2599075E-4}"  ixy="${wcf*-2.6376470E-7}"  ixz="${wcf*-9.8007285E-6}" iyy="${wcf*2.7781302E-4}" iyz="${wcf*-2.0435288E-6}" izz="${wcf*2.1878992E-4}" />
         </inertial>
         <visual>
@@ -89,6 +89,6 @@
     <inertial>
       <origin xyz="0.0099500565 0.038682024 1.6446924E-4" rpy="0 0 0"/>
-      <mass value="0.56782202"/>
-      <inertia ixx="7.8337456E-4"  ixy="-1.9035768E-4"  ixz="-3.0037676E-6" iyy="6.3399921E-4" iyz="-4.3840774E-6" izz="0.001008054" />
+      <mass value="${wcf*0.56782202}"/>
+      <inertia ixx="${wcf*7.8337456E-4}"  ixy="${wcf*-1.9035768E-4}"  ixz="${wcf*-3.0037676E-6}" iyy="${wcf*6.3399921E-4}" iyz="${wcf*-4.3840774E-6}" izz="${wcf*0.001008054}" />
     </inertial>
     <visual>
@@ -109,6 +109,6 @@
     <inertial>
       <origin xyz="-0.0038936743 -2.2022151E-6 -0.0048616005" rpy="0 0 0"/>
-      <mass value="0.77683752"/>
-      <inertia ixx="4.5812904E-4"  ixy="2.4111086E-7"  ixz="9.2521185E-6" iyy="4.3089204E-4" iyz="4.721695E-7" izz="3.4174855E-4" />
+      <mass value="${wcf*0.77683752}"/>
+      <inertia ixx="${wcf*4.5812904E-4}"  ixy="${wcf*2.4111086E-7}"  ixz="${wcf*9.2521185E-6}" iyy="${wcf*4.3089204E-4}" iyz="${wcf*4.721695E-7}" izz="${wcf*3.4174855E-4}" />
     </inertial>
     <visual>
@@ -129,6 +129,6 @@
     <inertial>
       <origin xyz="0.0022714213 0.0071091517 -0.057455221" rpy="0 0 0"/>
-      <mass value="1.0462304"/>
-      <inertia ixx="0.0030934574"  ixy="-6.6702837E-5"  ixz="3.0222291E-4" iyy="0.0029181573" iyz="5.2663661E-4" izz="8.0830389E-4" />
+      <mass value="${wcf*1.0462304}"/>
+      <inertia ixx="${wcf*0.0030934574}"  ixy="${wcf*-6.6702837E-5}"  ixz="${wcf*3.0222291E-4}" iyy="${wcf*0.0029181573}" iyz="${wcf*5.2663661E-4}" izz="${wcf*8.0830389E-4}" />
     </inertial>
     <visual>
@@ -149,6 +149,6 @@
         <inertial>
           <origin xyz="-6.5553403E-4 9.3464748E-4 -9.3101289E-4" rpy="0 0 0"/>
-          <mass value="0.63306933"/>
-          <inertia ixx="2.2599075E-4"  ixy="2.6376470E-7"  ixz="-9.8007285E-6" iyy="2.7781302E-4" iyz="2.0435288E-6" izz="2.1878992E-4" />
+          <mass value="${wcf*0.63306933}"/>
+          <inertia ixx="${wcf*2.2599075E-4}"  ixy="${wcf*2.6376470E-7}"  ixz="${wcf*-9.8007285E-6}" iyy="${wcf*2.7781302E-4}" iyz="${wcf*2.0435288E-6}" izz="${wcf*2.1878992E-4}" />
         </inertial>
         <visual>

Commit message: Added wcf to legs

File: cogimon_urdf/urdf/cogimon.urdf.xacro (robot description, xacro)
@@ -27,4 +27,5 @@
 	</joint>
 </xacro:unless>
+<!-- WEIGHT COEFFICIENT FACTOR is a factor that multiplies weights and inertias -->
 <xacro:property name="wcf" value="1.3" />
 <!-- ************ COGIMON BASE ************** -->

File: cogimon_urdf/urdf/parts/legs.urdf.xacro (robot description, xacro)
@@ -9,6 +9,6 @@
     <inertial>
       <origin xyz="-3.269678E-4 -0.023587321 -2.6496509E-4" rpy="0 0 0"/>
-      <mass value="0.89258227"/>
-      <inertia ixx="4.7672294E-4"  ixy="-3.9936567E-6"  ixz="-2.4802574E-6" iyy="5.458038E-4" iyz="-3.3389575E-6" izz="5.126859E-4" />
+      <mass value="${wcf*0.89258227}"/>
+      <inertia ixx="${wcf*4.7672294E-4}"  ixy="${wcf*-3.9936567E-6}"  ixz="${wcf*-2.4802574E-6}" iyy="${wcf*5.458038E-4}" iyz="${wcf*-3.3389575E-6}" izz="${wcf*5.126859E-4}" />
     </inertial>
     <visual>
@@ -29,6 +29,6 @@
     <inertial>
       <origin xyz="0.0012591632 -0.016896372 -0.058903336" rpy="0 0 0"/>
-      <mass value="1.0246101"/>
-      <inertia ixx="9.165719E-4"  ixy="-1.4449904E-6"  ixz="-1.6685011E-5" iyy="0.00104849584" iyz="2.5492874E-5" izz="6.8637197E-4" />
+      <mass value="${wcf*1.0246101}"/>
+      <inertia ixx="${wcf*9.165719E-4}"  ixy="${wcf*-1.4449904E-6}"  ixz="${wcf*-1.6685011E-5}" iyy="${wcf*0.00104849584}" iyz="${wcf*2.5492874E-5}" izz="${wcf*6.8637197E-4}" />
     </inertial>
     <visual>
@@ -49,6 +49,6 @@
     <inertial>
       <origin xyz="9.8720058E-4 6.7037262E-4 -0.075716843" rpy="0 0 0"/>
-      <mass value="1.7001134"/>
-      <inertia ixx="0.0038979546"  ixy="1.7802399E-6"  ixz="2.6403262E-5" iyy="0.0039360845" iyz="4.522711E-5" izz="9.0218711E-4" />
+      <mass value="${wcf*1.7001134}"/>
+      <inertia ixx="${wcf*0.0038979546}"  ixy="${wcf*1.7802399E-6}"  ixz="${wcf*2.6403262E-5}" iyy="${wcf*0.0039360845}" iyz="${wcf*4.522711E-5}" izz="${wcf*9.0218711E-4}" />
     </inertial>
     <visual>
@@ -69,6 +69,6 @@
     <inertial>
       <origin xyz="0.0024612666 -0.0053099614 -0.08598948" rpy="0 0 0"/>
-      <mass value="1.4098179"/>
-      <inertia ixx="0.0040604004"  ixy="1.1227206E-5"  ixz="1.2260973E-5" iyy="0.004005652855" iyz="5.1899176E-4" izz="0.0012414054" />
+      <mass value="${wcf*1.4098179}"/>
+      <inertia ixx="${wcf*0.0040604004}"  ixy="${wcf*1.1227206E-5}"  ixz="${wcf*1.2260973E-5}" iyy="${wcf*0.004005652855}" iyz="${wcf*5.1899176E-4}" izz="${wcf*0.0012414054}" />
     </inertial>
     <visual>
@@ -89,6 +89,6 @@
     <inertial>
       <origin xyz="8.8067281E-4 -9.2224881E-4 2.3038476E-4" rpy="0 0 0"/>
-      <mass value="0.72992131"/>
-      <inertia ixx="3.2034425E-4"  ixy="7.6346303E-6"  ixz="2.5430158E-7" iyy="3.6584358E-4" iyz="-3.6889276E-6" izz="3.6065156E-4" />
+      <mass value="${wcf*0.72992131}"/>
+      <inertia ixx="${wcf*3.2034425E-4}"  ixy="${wcf*7.6346303E-6}"  ixz="${wcf*2.5430158E-7}" iyy="${wcf*3.6584358E-4}" iyz="${wcf*-3.6889276E-6}" izz="${wcf*3.6065156E-4}" />
     </inertial>
     <visual>
@@ -110,6 +110,6 @@
       <inertial>
         <origin xyz="0.00969210464 -0.0090460227 -0.043062308" rpy="0 0 0"/>
-        <mass value="0.66646684"/>
-        <inertia ixx="0.0012944808"  ixy="-9.2387693E-5"  ixz="2.0080105E-4" iyy="0.0015851846" iyz="2.7599327E-4" izz="0.0013326766" />
+        <mass value="${wcf*0.66646684}"/>
+        <inertia ixx="${wcf*0.0012944808}"  ixy="${wcf*-9.2387693E-5}"  ixz="${wcf*2.0080105E-4}" iyy="${wcf*0.0015851846}" iyz="${wcf*2.7599327E-4}" izz="${wcf*0.0013326766}" />
       </inertial>
       <visual>
@@ -132,6 +132,6 @@
       <inertial>
         <origin xyz="0.00969210464 -0.0090460227 -0.043062308" rpy="0 0 0"/>
-        <mass value="0.66646684"/>
-        <inertia ixx="0.0012944808"  ixy="-9.2387693E-5"  ixz="2.0080105E-4" iyy="0.0015851846" iyz="2.7599327E-4" izz="0.0013326766" />
+        <mass value="${wcf*0.66646684}"/>
+        <inertia ixx="${wcf*0.0012944808}"  ixy="${wcf*-9.2387693E-5}"  ixz="${wcf*2.0080105E-4}" iyy="${wcf*0.0015851846}" iyz="${wcf*2.7599327E-4}" izz="${wcf*0.0013326766}" />
       </inertial>
     <visual>
@@ -154,6 +154,6 @@
     <inertial>
       <origin xyz="-3.269678E-4 0.023587321 -2.6496509E-4" rpy="0 0 0"/>
-      <mass value="0.89258227"/>
-      <inertia ixx="4.7672294E-4"  ixy="3.9936567E-6"  ixz="-2.4802574E-6" iyy="5.458038E-4" iyz="3.3389575E-6" izz="5.126859E-4" />
+      <mass value="${wcf*0.89258227}"/>
+      <inertia ixx="${wcf*4.7672294E-4}"  ixy="${wcf*3.9936567E-6}"  ixz="${wcf*-2.4802574E-6}" iyy="${wcf*5.458038E-4}" iyz="${wcf*3.3389575E-6}" izz="${wcf*5.126859E-4}" />
     </inertial>
     <visual>
@@ -174,6 +174,6 @@
     <inertial>
       <origin xyz="0.0012591632 0.016896372 -0.058903336" rpy="0 0 0"/>
-      <mass value="1.0246101"/>
-      <inertia ixx="9.165719E-4"  ixy="1.4449904E-6"  ixz="-1.6685011E-5" iyy="0.00104849584" iyz="-2.5492874E-5" izz="6.8637197E-4" />
+      <mass value="${wcf*1.0246101}"/>
+      <inertia ixx="${wcf*9.165719E-4}"  ixy="${wcf*1.4449904E-6}"  ixz="${wcf*-1.6685011E-5}" iyy="${wcf*0.00104849584}" iyz="${wcf*-2.5492874E-5}" izz="${wcf*6.8637197E-4}" />
     </inertial>
     <visual>
@@ -194,6 +194,6 @@
     <inertial>
       <origin xyz="9.8720058E-4 -6.7037262E-4 -0.075716843" rpy="0 0 0"/>
-      <mass value="1.7001134"/>
-      <inertia ixx="0.0038979546"  ixy="-1.7802399E-6"  ixz="2.6403262E-5" iyy="0.0039360845" iyz="-4.5227110E-5" izz="9.0218711E-4" />
+      <mass value="${wcf*1.7001134}"/>
+      <inertia ixx="${wcf*0.0038979546}"  ixy="${wcf*-1.7802399E-6}"  ixz="${wcf*2.6403262E-5}" iyy="${wcf*0.0039360845}" iyz="${wcf*-4.5227110E-5}" izz="${wcf*9.0218711E-4}" />
     </inertial>
     <visual>
@@ -214,6 +214,6 @@
     <inertial>
       <origin xyz="0.0024612666 0.0053099614 -0.085989484" rpy="0 0 0"/>
-      <mass value="1.4098179"/>
-      <inertia ixx="0.0040604004"  ixy="-1.1227206E-5"  ixz="1.2260973E-5" iyy="0.004005652855" iyz="-5.1899176E-4" izz="0.0012414054" />
+      <mass value="${wcf*1.4098179}"/>
+      <inertia ixx="${wcf*0.0040604004}"  ixy="${wcf*-1.1227206E-5}"  ixz="${wcf*1.2260973E-5}" iyy="${wcf*0.004005652855}" iyz="${wcf*-5.1899176E-4}" izz="${wcf*0.0012414054}" />
     </inertial>
     <visual>
@@ -234,6 +234,6 @@
     <inertial>
       <origin xyz="8.8067281E-4 9.2224881E-4 2.3038476E-4" rpy="0 0 0"/>
-      <mass value="0.72992131"/>
-      <inertia ixx="3.2034425E-4"  ixy="-7.6346303E-6"  ixz="2.5430158E-7" iyy="3.6584358E-4" iyz="3.6889276E-6" izz="3.6065156E-4" />
+      <mass value="${wcf*0.72992131}"/>
+      <inertia ixx="${wcf*3.2034425E-4}"  ixy="${wcf*-7.6346303E-6}"  ixz="${wcf*2.5430158E-7}" iyy="${wcf*3.6584358E-4}" iyz="${wcf*3.6889276E-6}" izz="${wcf*3.6065156E-4}" />
     </inertial>
     <visual>
@@ -255,6 +255,6 @@
       <inertial>
         <origin xyz="0.0096921046 0.0090460227 -0.043062308" rpy="0 0 0"/>
-        <mass value="0.66646684"/>
-        <inertia ixx="0.0012944808"  ixy="9.2387693E-5"  ixz="2.0080105E-4" iyy="0.0015851846" iyz="-2.7599327E-4" izz="0.0013326766" />
+        <mass value="${wcf*0.66646684}"/>
+        <inertia ixx="${wcf*0.0012944808}"  ixy="${wcf*9.2387693E-5}"  ixz="${wcf*2.0080105E-4}" iyy="${wcf*0.0015851846}" iyz="${wcf*-2.7599327E-4}" izz="${wcf*0.0013326766}" />
       </inertial>
       <visual>
@@ -277,6 +277,6 @@
       <inertial>
         <origin xyz="0.0096921046 0.0090460227 -0.043062308" rpy="0 0 0"/>
-        <mass value="0.66646684"/>
-        <inertia ixx="0.0012944808"  ixy="9.2387693E-5"  ixz="2.0080105E-4" iyy="0.0015851846" iyz="-2.7599327E-4" izz="0.0013326766" />
+        <mass value="${wcf*0.66646684}"/>
+        <inertia ixx="${wcf*0.0012944808}"  ixy="${wcf*9.2387693E-5}"  ixz="${wcf*2.0080105E-4}" iyy="${wcf*0.0015851846}" iyz="${wcf*-2.7599327E-4}" izz="${wcf*0.0013326766}" />
       </inertial>
       <visual>

Commit message: changed wcf to 1.4

File: cogimon_urdf/urdf/cogimon.urdf.xacro (robot description, xacro)
@@ -28,5 +28,5 @@
 </xacro:unless>
 <!-- WEIGHT COEFFICIENT FACTOR is a factor that multiplies weights and inertias -->
-<xacro:property name="wcf" value="1.3" />
+<xacro:property name="wcf" value="1.4" />
 <!-- ************ COGIMON BASE ************** -->
 <xacro:include filename="$(find cogimon_urdf)/urdf/cogimon_base.urdf.xacro"/>
