Commit message: Added link offset. Changed max torque. Added 2 cm to feet.

File: cogimon_urdf/urdf/cogimon.urdf.xacro (robot description, xacro)
@@ -31,4 +31,6 @@
 <!-- WEIGHT COEFFICIENT FACTOR is a factor that multiplies weights and inertias -->
 <xacro:property name="wcf" value="1.4" />
+<!-- HEIGHT COEFFICIENT OFFSET is a factor added to legs and torso links -->
+<xacro:property name="hco" value="0.1" />
 <!-- ************ COGIMON BASE ************** -->
 <xacro:include filename="$(find cogimon_urdf)/urdf/cogimon_base.urdf.xacro"/>

File: cogimon_urdf/urdf/cogimon_robot.urdf.xacro (robot description, xacro)
@@ -16,4 +16,4 @@
   <xacro:include filename="$(find cogimon_urdf)/urdf/gazebo/cogimon_materials.gazebo.xacro" />
   <xacro:include filename="$(find cogimon_urdf)/urdf/gazebo/force_torque.gazebo.xacro" />
-  <origin xyz="0.0 0.0 0.521" rpy="0 0 0" />
+  <origin xyz="0.0 0.0 ${0.521+2.0*hco}" rpy="0 0 0" />
 </robot>

File: cogimon_urdf/urdf/parts/arms.urdf.xacro (robot description, xacro)
@@ -173,5 +173,5 @@
     <origin xyz="-0.014976503999999998 -0.0825 0.15770847" rpy="0 0 0" />
     <axis xyz="0 1 0" />
-    <limit velocity="4.0" effort="50" lower="-3.4034" upper="1.6581" />
+    <limit velocity="4.0" effort="40" lower="-3.4034" upper="1.6581" />
     <dynamics friction="0" damping="3.0"/>
 </joint>
@@ -181,5 +181,5 @@
     <origin xyz="0.0 -0.07329999999999999 0.0" rpy="0 0 0" />
     <axis xyz="1 0 0" />
-    <limit velocity="4.0" effort="50" lower="-2.094" upper="0.31415" />
+    <limit velocity="4.0" effort="40" lower="-2.094" upper="0.31415" />
     <dynamics friction="0" damping="3.0"/>
 </joint>
@@ -189,5 +189,5 @@
     <origin xyz="0.0 0.0 -0.04480846999999999" rpy="0 0 0" />
     <axis xyz="0 0 1" />
-    <limit velocity="4.0" effort="50" lower="-1.5708" upper="1.5708" />
+    <limit velocity="4.0" effort="40" lower="-1.5708" upper="1.5708" />
     <dynamics friction="0" damping="3.0"/>
 </joint>
@@ -197,5 +197,5 @@
     <origin xyz="0.015 0.0 -0.13519152999999998" rpy="0 0 0" />
     <axis xyz="0 1 0" />
-    <limit velocity="4.0" effort="50" lower="-2.3562" upper="0.0" />
+    <limit velocity="4.0" effort="40" lower="-2.3562" upper="0.0" />
     <dynamics friction="0" damping="3.0"/>
   </joint>
@@ -206,5 +206,5 @@
     <origin xyz="-0.014976503999999998 0.0825 0.15770847" rpy="0 0 0" />
     <axis xyz="0 1 0" />
-    <limit velocity="4.0" effort="50" lower="-3.4034" upper="1.6581" />
+    <limit velocity="4.0" effort="40" lower="-3.4034" upper="1.6581" />
     <dynamics friction="0" damping="3.0"/>
 </joint>
@@ -214,5 +214,5 @@
     <origin xyz="0.0 0.07329999999999999 0.0" rpy="0 0 0" />
     <axis xyz="1 0 0" />
-    <limit velocity="4.0" effort="50" lower="-0.31415" upper="2.094" />
+    <limit velocity="4.0" effort="40" lower="-0.31415" upper="2.094" />
     <dynamics friction="0" damping="3.0"/>
 </joint>
@@ -222,5 +222,5 @@
     <origin xyz="0.0 0.0 -0.04480846999999999" rpy="0 0 0" />
     <axis xyz="0 0 1" />
-    <limit velocity="4.0" effort="50" lower="-1.5708" upper="1.5708" />
+    <limit velocity="4.0" effort="40" lower="-1.5708" upper="1.5708" />
     <dynamics friction="0" damping="3.0"/>
 </joint>
@@ -230,5 +230,5 @@
     <origin xyz="0.015 0.0 -0.13519152999999998" rpy="0 0 0" />
     <axis xyz="0 1 0" />
-    <limit velocity="4.0" effort="50" lower="-2.3562" upper="0.0" />
+    <limit velocity="4.0" effort="40" lower="-2.3562" upper="0.0" />
     <dynamics friction="0" damping="3.0"/>
   </joint>

File: cogimon_urdf/urdf/parts/forearms.urdf.xacro (robot description, xacro)
@@ -149,5 +149,5 @@
     <origin xyz="-0.015 0.0 ${-0.051 - Wrj1_to_FT}" rpy="0 0 0"/>
     <axis xyz="0 0 1" />
-    <limit velocity="4.0" effort="5" lower="-1.5708" upper="1.5708" />
+    <limit velocity="4.0" effort="15" lower="-1.5708" upper="1.5708" />
     <dynamics friction="0" damping="0.03"/>
   </joint>
@@ -157,5 +157,5 @@
     <origin xyz="0 0 ${-0.14368 + Wrj1_to_FT}" rpy="0 0 0"/>
     <axis xyz="0 1 0"/>
-    <limit velocity="4.0" effort="5" lower="-0.524" upper="0.524" />
+    <limit velocity="4.0" effort="15" lower="-0.524" upper="0.524" />
     <dynamics friction="0" damping="0.03"/>
   </joint>
@@ -165,5 +165,5 @@
     <origin xyz="0 0 0.0" rpy="0 0 0"/>
     <axis xyz="1 0 0"/>
-    <limit velocity="4.0" effort="5" lower="-0.785375" upper="1.395" />
+    <limit velocity="4.0" effort="15" lower="-0.785375" upper="1.395" />
     <dynamics friction="0" damping="0.03"/>
   </joint>
@@ -179,5 +179,5 @@
     <origin xyz="-0.015 0.0 ${-0.051 - Wrj1_to_FT}" rpy="0 0 0"/>
     <axis xyz="0 0 1" />
-    <limit velocity="4.0" effort="5" lower="-1.5708" upper="1.5708" />
+    <limit velocity="4.0" effort="15" lower="-1.5708" upper="1.5708" />
     <dynamics friction="0" damping="0.03"/>
   </joint>
@@ -187,5 +187,5 @@
     <origin xyz="0 0 ${-0.14368 + Wrj1_to_FT}" rpy="0 0 0"/>
     <axis xyz="0 1 0"/>
-    <limit velocity="4.0" effort="5" lower="-0.524" upper="0.524" />
+    <limit velocity="4.0" effort="15" lower="-0.524" upper="0.524" />
     <dynamics friction="0" damping="0.03"/>
   </joint>
@@ -195,5 +195,5 @@
     <origin xyz="0 0 0.0" rpy="0 0 0"/>
     <axis xyz="1 0 0"/>
-    <limit velocity="4.0" effort="5" lower="-1.395" upper="0.785375" />
+    <limit velocity="4.0" effort="15" lower="-1.395" upper="0.785375" />
     <dynamics friction="0" damping="0.03"/>
   </joint>

File: cogimon_urdf/urdf/parts/legs.urdf.xacro (robot description, xacro)
@@ -138,5 +138,5 @@
      <origin xyz="0.03 0 -0.07" rpy="0 0 0" />
      <geometry>
-       <box size="0.2 0.1 0.04" />
+       <box size="0.2 0.12 0.04" />
      </geometry>
      <material name="dark_gray"/>
@@ -145,5 +145,5 @@
      <origin xyz="0.03 0 -0.07" rpy="0 0 0"/>
      <geometry>
-       <box size="0.2 0.1 0.04" />
+       <box size="0.2 0.12 0.04" />
      </geometry>
    </collision>
@@ -283,5 +283,5 @@
        <origin xyz="0.03 0 -0.07" rpy="0 0 0" />
        <geometry>
-         <box size="0.2 0.1 0.04" />
+         <box size="0.2 0.12 0.04" />
        </geometry>
        <material name="dark_gray"/>
@@ -290,5 +290,5 @@
        <origin xyz="0.03 0 -0.07" rpy="0 0 0"/>
        <geometry>
-         <box size="0.2 0.1 0.04" />
+         <box size="0.2 0.12 0.04" />
        </geometry>
      </collision>
@@ -302,5 +302,5 @@
     <origin xyz="0.0 -0.023 0.0" rpy="0 0 0" />
     <axis xyz="0 1 0" />
-    <limit velocity="4.0" effort="50" lower="-1.9199" upper="0.7854" />
+    <limit velocity="4.0" effort="80" lower="-1.9199" upper="0.7854" />
     <dynamics friction="0" damping="3.0"/>
   </joint>
@@ -310,5 +310,5 @@
     <origin xyz="0.0 -0.0496 0.0" rpy="0 0 0" />
     <axis xyz="1 0 0" />
-    <limit velocity="4.0" effort="50" lower="-1.0472" upper="0.4363" />
+    <limit velocity="4.0" effort="80" lower="-1.0472" upper="0.4363" />
     <dynamics friction="0" damping="3.0"/>
   </joint>
@@ -316,7 +316,7 @@
     <parent link="RThighUpLeg"/>
     <child link="RThighLowLeg"/>
-    <origin xyz="0.0 0.0 -0.1024" rpy="0 0 0" />
+    <origin xyz="0.0 0.0 ${-0.1024-hco}" rpy="0 0 0" />
     <axis xyz="0 0 1" />
-    <limit velocity="4.0" effort="50" lower="-0.8727" upper="0.8727" />
+    <limit velocity="4.0" effort="80" lower="-0.8727" upper="0.8727" />
     <dynamics friction="0" damping="3.0"/>
   </joint>
@@ -326,5 +326,5 @@
     <origin xyz="0.0 0.0 -0.1234" rpy="0 0 0" />
     <axis xyz="0 1 0" />
-    <limit velocity="4.0" effort="50" lower="-0.1745" upper="1.9199" />
+    <limit velocity="4.0" effort="80" lower="-0.1745" upper="1.9199" />
     <dynamics friction="0" damping="3.0"/>
   </joint>
@@ -332,7 +332,7 @@
     <parent link="RLowLeg"/>
     <child link="RFootmot"/>
-    <origin xyz="0.0 0.0 -0.201" rpy="0 0 0" />
+    <origin xyz="0.0 0.0 ${-0.201-hco}" rpy="0 0 0" />
     <axis xyz="1 0 0" />
-    <limit velocity="4.0" effort="50" lower="-0.6109" upper="0.6109" />
+    <limit velocity="4.0" effort="80" lower="-0.6109" upper="0.6109" />
     <dynamics friction="0" damping="3.0"/>
   </joint>
@@ -342,5 +342,5 @@
       <origin xyz="0.0 0.0 0.0" rpy="0 0 0" />
       <axis xyz="0 1 0" />
-      <limit velocity="4.0" effort="50" lower="-1.2217" upper="1.2217" />
+      <limit velocity="4.0" effort="80" lower="-1.2217" upper="1.2217" />
       <dynamics friction="0" damping="3.0"/>
   </joint>
@@ -351,5 +351,5 @@
     <origin xyz="0.0 0.023 0.0" rpy="0 0 0" />
     <axis xyz="0 1 0" />
-    <limit velocity="4.0" effort="50" lower="-1.9199" upper="0.7854" />
+    <limit velocity="4.0" effort="80" lower="-1.9199" upper="0.7854" />
     <dynamics friction="0" damping="3.0"/>
   </joint>
@@ -359,5 +359,5 @@
     <origin xyz="0.0 0.0496 0.0" rpy="0 0 0" />
     <axis xyz="1 0 0" />
-    <limit velocity="4.0" effort="50" lower="-0.4363" upper="1.0472" />
+    <limit velocity="4.0" effort="80" lower="-0.4363" upper="1.0472" />
     <dynamics friction="0" damping="3.0"/>
   </joint>
@@ -365,7 +365,7 @@
     <parent link="LThighUpLeg"/>
     <child link="LThighLowLeg"/>
-    <origin xyz="0.0 0.0 -0.1024" rpy="0 0 0" />
+    <origin xyz="0.0 0.0 ${-0.1024-hco}" rpy="0 0 0" />
     <axis xyz="0 0 1" />
-    <limit velocity="4.0" effort="50" lower="-0.8727" upper="0.8727" />
+    <limit velocity="4.0" effort="80" lower="-0.8727" upper="0.8727" />
     <dynamics friction="0" damping="3.0"/>
   </joint>
@@ -375,5 +375,5 @@
     <origin xyz="0.0 0.0 -0.1234" rpy="0 0 0" />
     <axis xyz="0 1 0" />
-    <limit velocity="4.0" effort="50" lower="-0.1745" upper="1.9199" />
+    <limit velocity="4.0" effort="80" lower="-0.1745" upper="1.9199" />
     <dynamics friction="0" damping="3.0"/>
   </joint>
@@ -381,7 +381,7 @@
     <parent link="LLowLeg"/>
     <child link="LFootmot"/>
-    <origin xyz="0.0 0.0 -0.201" rpy="0 0 0" />
+    <origin xyz="0.0 0.0 ${-0.201-hco}" rpy="0 0 0" />
     <axis xyz="1 0 0" />
-    <limit velocity="4.0" effort="50" lower="-0.6109" upper="0.6109" />
+    <limit velocity="4.0" effort="80" lower="-0.6109" upper="0.6109" />
     <dynamics friction="0" damping="3.0"/>
   </joint>
@@ -391,5 +391,5 @@
       <origin xyz="0.0 0.0 0.0" rpy="0 0 0" />
       <axis xyz="0 1 0" />
-      <limit velocity="4.0" effort="50" lower="-1.2217" upper="1.2217" />
+      <limit velocity="4.0" effort="80" lower="-1.2217" upper="1.2217" />
       <dynamics friction="0" damping="3.0"/>
   </joint>

File: cogimon_urdf/urdf/parts/torso.urdf.xacro (robot description, xacro)
@@ -85,5 +85,5 @@
     <origin xyz="0 0 0" rpy="0 0 0" />
     <axis xyz="0 1 0" />
-    <limit velocity="4.0" effort="50" lower="-0.3491" upper="0.8727" />
+    <limit velocity="4.0" effort="80" lower="-0.3491" upper="0.8727" />
     <dynamics friction="0" damping="3.0"/>
   </joint>
@@ -91,7 +91,7 @@
     <parent link="DWS"/>
     <child link="DWYTorso"/>
-    <origin xyz="0 0 0.04749999" rpy="0 0 0" />
+    <origin xyz="0 0 ${0.04749999+hco}" rpy="0 0 0" />
     <axis xyz="0 0 1" />
-    <limit velocity="4.0" effort="50" lower="-1.3963" upper="1.3962" />
+    <limit velocity="4.0" effort="40" lower="-1.3963" upper="1.3962" />
     <dynamics friction="0" damping="3.0"/>
   </joint>

Commit message: Updated config files for simulation. Changed wcf to have that cogimon weights around 65 kg (it is 64 and something)

File: cogimon_urdf/urdf/cogimon.urdf.xacro (robot description, xacro)
@@ -30,5 +30,5 @@
 </xacro:unless>
 <!-- WEIGHT COEFFICIENT FACTOR is a factor that multiplies weights and inertias -->
-<xacro:property name="wcf" value="1.4" />
+<xacro:property name="wcf" value="2.1" />
 <!-- HEIGHT COEFFICIENT OFFSET is a factor added to legs and torso links -->
 <xacro:property name="hco" value="0.1" />

File: cogimon_urdf/urdf/cogimon_robot.urdf.xacro (robot description, xacro)
@@ -16,4 +16,4 @@
   <xacro:include filename="$(find cogimon_urdf)/urdf/gazebo/cogimon_materials.gazebo.xacro" />
   <xacro:include filename="$(find cogimon_urdf)/urdf/gazebo/force_torque.gazebo.xacro" />
-  <origin xyz="0.0 0.0 ${0.521+2.0*hco}" rpy="0 0 0" />
+  <origin xyz="0.0 0.0 ${0.521+2.0*(hco+0.025)}" rpy="0 0 0" />
 </robot>

Commit message: Updated Waist

File: cogimon_urdf/urdf/cogimon.urdf.xacro (robot description, xacro)
@@ -24,5 +24,5 @@
 	</joint-->
         <!-- NECK -->
-	<!--xacro:include filename="$(find cogimon_urdf)/urdf/parts/neck.urdf.xacro" />
+	<!--xacro:include filename="$(find cogimon_urdf)/urdf/parts/neck.urdf.xacro" /-->
 <!-- ************ COGIMON BASE ************** -->
 <xacro:include filename="$(find cogimon_urdf)/urdf/cogimon_base.urdf.xacro"/>

File: cogimon_urdf/urdf/cogimon_base.urdf.xacro (robot description, xacro)
@@ -14,7 +14,7 @@
 <link name="Waist">
     <inertial>
-      <origin xyz="${-2.9198594E+01*mmTom} ${-1.1793030E-01*mmTom} ${-3.7516729E+01*mmTom}" rpy="0.0 0.0 0.0"/>
+      <origin xyz="${-2.0579946e+01*mmTom} ${-1.0999634e+00*mmTom} ${-3.7500786e+01*mmTom}" rpy="0.0 0.0 0.0"/>
       <mass value="4.2357548"/>
-      <inertia ixx="${4.6492739E+04*mm2Tom2}"  ixy="${3.3912005E+01*mm2Tom2}"  ixz="${3.0361216E+01*mm2Tom2}" iyy="${1.4628117E+04*mm2Tom2}" iyz="${9.6064394E+00*mm2Tom2}" izz="${5.0051187E+04*mm2Tom2}" />
+      <inertia ixx="${4.6492739e+04*mm2Tom2}"  ixy="${3.4766548e+01*mm2Tom2}"  ixz="${3.2487180e+01*mm2Tom2}" iyy="${1.4654103e+04*mm2Tom2}" iyz="${9.3654340e+02*mm2Tom2}" izz="${5.0027621e+04*mm2Tom2}" />
     </inertial>
     <visual>

File: cogimon_urdf/urdf/cogimon_config.urdf.xacro (robot description, xacro)
@@ -3,3 +3,10 @@
 <xacro:property name="model_name" value="IIT COGIMON" />
 <xacro:property name="model_version" value="0.1" />
+<!-- ************SELECT PARTS*************-->
+<!-- *************************************-->
+<xacro:property name="COGIMON_TORSO" value="TRUE" />
+<xacro:property name="COGIMON_LEFT_ARM" value="TRUE" />
+<xacro:property name="COGIMON_RIGH_ARM" value="TRUE" />
+<xacro:property name="COGIMON_LEFT_LEG" value="TRUE" />
+<xacro:property name="COGIMON_RIGH_LEG" value="TRUE" />
 </robot>

Commit message: Added docs and usefull ref frames in the legs

File: cogimon_urdf/urdf/cogimon.urdf.xacro (robot description, xacro)
@@ -27,47 +27,5 @@
 <!-- ************ COGIMON BASE ************** -->
 <xacro:include filename="$(find cogimon_urdf)/urdf/cogimon_base.urdf.xacro"/>
-<!-- ************ FOREARMS ************ -->
-<!-- This links are defined in order to be compliant with http://www.ros.org/reps/rep-0120.html#coordinate-frames
-and to define the end effectors of the robot -->
-<!-- position and orientation of the arm regardless of the tool (grasping device for instance) attached to it -->
-<!--link name="l_wrist"/>
-<link name="r_wrist"/>
-<xacro:if value="${GAZEBO_COGIMON_USES_FOREARMS}">
-    <xacro:include filename="$(find cogimon_urdf)/urdf/parts/forearms.urdf.xacro" />
-    <link name="l_arm_ft"/>
-    <link name="r_arm_ft"/>
-    <joint name="l_arm_ft_joint" type="fixed">
-      <parent link="LForearm"/>
-      <child link="l_arm_ft"/>
-      <origin xyz="0 0 0" rpy="0 0 0" />
-    </joint>
-    <joint name="r_arm_ft_joint" type="fixed">
-      <parent link="RForearm"/>
-      <child link="r_arm_ft"/>
-      <origin xyz="0 0 0" rpy="0 0 0" />
-    </joint>
-</xacro:if>
-<xacro:unless value="${GAZEBO_COGIMON_USES_FOREARMS}">
-    <xacro:include filename="$(find cogimon_urdf)/urdf/parts/no_forearms.urdf.xacro" />
-</xacro:unless>
-    <link name="l_leg_ft"/>
-    <link name="r_leg_ft"/>
-    <joint name="l_leg_ft_joint" type="fixed">
-      <parent link="LFoot"/>
-      <child link="l_leg_ft"/>
-      <origin xyz="0 0 -0.065" rpy="0 0 0" />
-    </joint>
-    <joint name="r_leg_ft_joint" type="fixed">
-      <parent link="RFoot"/>
-      <child link="r_leg_ft"/>
-      <origin xyz="0 0 -0.065" rpy="0 0 0" />
-    </joint-->
-<!-- ************ HANDS ************ -->
-<!--xacro:if value="${GAZEBO_COGIMON_USES_FOREARMS}">
-    <xacro:include filename="$(find cogimon_urdf)/urdf/parts/soft_hand.urdf.xacro" /-->
-    <!-- Reference frames in hands -->
-    <!--xacro:include filename="$(find cogimon_urdf)/urdf/parts/hand_reference_frame.urdf.xacro" />
-</xacro:if-->
-<!-- IMU -->
-<!--xacro:include filename="$(find cogimon_urdf)/urdf/sensors/imu.urdf.xacro"/-->
+<!-- ************ REF FRAMES **************** -->
+<xacro:include filename="$(find cogimon_urdf)/urdf/parts/feet_reference_frames.urdf.xacro"/>
 </robot>

Commit message: Added floating base

File: cogimon_urdf/urdf/cogimon.urdf.xacro (robot description, xacro)
@@ -29,3 +29,17 @@
 <!-- ************ REF FRAMES **************** -->
 <xacro:include filename="$(find cogimon_urdf)/urdf/parts/feet_reference_frames.urdf.xacro"/>
+<xacro:if value="${COGIMON_FLOATING_BASE}" >
+<link name="world"/>
+  <joint name="reference" type="floating">
+    <parent link="world"/>
+    <child link="base_link"/>
+</joint>
+</xacro:if>
+<xacro:if value="${COGIMON_FIXED_BASE}" >
+  <link name="world"/>
+   <joint name="fixed" type="fixed">
+    <parent link="world"/>
+    <child link="base_link"/>
+  </joint>
+</xacro:if>
 </robot>

File: cogimon_urdf/urdf/cogimon_robot.urdf.xacro (robot description, xacro)
@@ -13,11 +13,4 @@
   <xacro:include filename="$(find cogimon_urdf)/urdf/gazebo/xbot_control.gazebo.xacro" />
 </xacro:if>
-<xacro:if value="${COGIMON_FIXED_BASE}" >
-  <link name="world"/>
-   <joint name="fixed" type="fixed">
-    <parent link="world"/>
-    <child link="base_link"/>
-  </joint>
-</xacro:if>
 <origin xyz="0.0 0.0 0.97" rpy="0 0 0" />
 </robot>

File: cogimon_urdf/urdf/gazebo/xbot_control.gazebo.xacro (robot description, xacro)
@@ -3,5 +3,6 @@
 <gazebo>
     <plugin name="xbot_plugin_handler" filename="libGazeboXBotPlugin.so">
-    <path_to_config_file>configs/ADVR_shared/cogimon/configs/config_cogimon.yaml</path_to_config_file>
+       <path_to_config_file>configs/ADVR_shared/cogimon/configs/config_cogimon.yaml</path_to_config_file>
+    </plugin>
 </gazebo>
 </robot>

Commit message: adding missing xacro

File: cogimon_urdf/urdf/cogimon.urdf.xacro (robot description, xacro)
@@ -30,17 +30,20 @@
 <xacro:include filename="$(find cogimon_urdf)/urdf/parts/feet_reference_frames.urdf.xacro"/>
 <xacro:include filename="$(find cogimon_urdf)/urdf/parts/arms_reference_frames.urdf.xacro"/>
-<xacro:if value="${COGIMON_FLOATING_BASE}" >
-<link name="world"/>
-  <joint name="reference" type="floating">
-    <parent link="world"/>
-    <child link="base_link"/>
-</joint>
-</xacro:if>
-<xacro:if value="${COGIMON_FIXED_BASE}" >
-  <link name="world"/>
-   <joint name="fixed" type="fixed">
-    <parent link="world"/>
-    <child link="base_link"/>
-  </joint>
+<xacro:arg name="add_base_joint" default="true"/>
+<xacro:if value="$(arg add_base_joint)">
+  <xacro:if value="${COGIMON_FLOATING_BASE}" >
+    <link name="world"/>
+      <joint name="reference" type="floating">
+        <parent link="world"/>
+        <child link="base_link"/>
+    </joint>
+  </xacro:if>
+  <xacro:if value="${COGIMON_FIXED_BASE}" >
+    <link name="world"/>
+    <joint name="fixed" type="fixed">
+      <parent link="world"/>
+      <child link="base_link"/>
+    </joint>
+  </xacro:if>
 </xacro:if>
 </robot>
