Commit message: Added HipRoll left and right

File: cogimon_urdf/urdf/cogimon_base.urdf.xacro (robot description, xacro)
@@ -52,5 +52,6 @@
   <!--link name="l_toe"/>
   <link name="r_toe"/-->
-<!--xacro:include filename="$(find cogimon_urdf)/urdf/parts/legs.urdf.xacro" />
+<xacro:include filename="$(find cogimon_urdf)/urdf/parts/legs.urdf.xacro" />
+<!--
   <joint name="l_ankle_joint" type="fixed">
      <parent link="LFoot"/>

File: cogimon_urdf/urdf/cogimon_config.urdf.xacro (robot description, xacro)
@@ -5,8 +5,8 @@
 <!-- ************SELECT PARTS*************-->
 <!-- *************************************-->
-<xacro:property name="COGIMON_TORSO" value="TRUE" />
-<xacro:property name="COGIMON_LEFT_ARM" value="TRUE" />
-<xacro:property name="COGIMON_RIGH_ARM" value="TRUE" />
-<xacro:property name="COGIMON_LEFT_LEG" value="TRUE" />
-<xacro:property name="COGIMON_RIGH_LEG" value="TRUE" />
+<xacro:property name="COGIMON_TORSO" value="false" />
+<xacro:property name="COGIMON_LEFT_ARM" value="false" />
+<xacro:property name="COGIMON_RIGHT_ARM" value="false" />
+<xacro:property name="COGIMON_LEFT_LEG" value="true" />
+<xacro:property name="COGIMON_RIGHT_LEG" value="true" />
 </robot>

File: cogimon_urdf/urdf/cogimon_robot.urdf.xacro (robot description, xacro)
@@ -16,4 +16,9 @@
   <xacro:include filename="$(find cogimon_urdf)/urdf/gazebo/cogimon_materials.gazebo.xacro" />
   <xacro:include filename="$(find cogimon_urdf)/urdf/gazebo/force_torque.gazebo.xacro" /-->
+  <link name="world"/>
+   <joint name="fixed" type="fixed">
+    <parent link="world"/>
+    <child link="base_link"/>
+  </joint>
   <origin xyz="0.0 0.0 0.521" rpy="0 0 0" />
 </robot>

File: cogimon_urdf/urdf/parts/legs.urdf.xacro (robot description, xacro)
@@ -1,29 +1,71 @@
 <?xml version="1.0"?>
 <robot xmlns:xacro="http://ros.org/wiki/xacro">
-<xacro:property name="PI" value="3.14159265359" />
-<xacro:property name="PI_2" value="1.57079632679" />
-<xacro:property name="SF" value="0.03937" /> <!-- Scale factor for meshes -->
+<xacro:if value="${COGIMON_RIGHT_LEG}" >
+<!-- LINKS -->
+<link name ="RHipMot">
+    <inertial>
+      <origin xyz="${4.7902756e+00*mmTom} ${1.5595700e+01*mmTom} ${-6.0925801e+01*mmTom}" rpy="0 0 0"/>
+      <mass value="1.6995409"/>
+      <inertia ixx="${7.7713640e+03*mm2Tom2}"  ixy="${2.5414978e+02*mm2Tom2}"  ixz="${-1.1602420e+03*mm2Tom2}" iyy="${8.1906401e+03*mm2Tom2}" iyz="${1.2050460e+03*mm2Tom2}" izz="${3.7083468e+03*mm2Tom2}" />
+    </inertial>
+    <visual>
+      <origin xyz="0.0 0 0" rpy="0 0 0"/>
+      <material name="dark_grey"/>
+      <geometry name="RHipMot_visual">
+        <mesh filename="package://cogimon_urdf/meshes/Leg0.STL" scale="${mmTom} ${-mmTom} ${mmTom}" />
+      </geometry>
+    </visual>
+    <collision>
+      <origin xyz="0.0 0. 0" rpy="0 0 0."/>
+      <geometry name="RHipMot_collision">
+        <mesh filename="package://cogimon_urdf/meshes/simple/Leg0.STL" scale="${mmTom} ${-mmTom} ${mmTom}" />
+      </geometry>
+    </collision>
+</link>
+<!-- JOINTS -->
+<joint name="RHipLat" type="revolute">
+    <parent link="Waist"/>
+    <child link="RHipMot"/>
+    <origin xyz="${12.58*mmTom} ${-110.954508*mmTom} ${-52.922586*mmTom}" rpy="0 0 -0.0262" />
+    <axis xyz="1 0 0" />
+    <limit velocity="3.67" effort="176" lower="${-85.*toRad}" upper="${25.*toRad}" />
+    <dynamics friction="0" damping="3.0"/>
+  </joint>
+</xacro:if>
+<xacro:if value="${COGIMON_LEFT_LEG}" >
+<!-- LINKS -->
+<link name ="LHipMot">
+    <inertial>
+      <origin xyz="${4.7902756e+00*mmTom} ${-1.5595700e+01*mmTom} ${-6.0925801e+01*mmTom}" rpy="0 0 0"/>
+      <mass value="1.6995409"/>
+      <inertia ixx="${7.7713640e+03*mm2Tom2}"  ixy="${-2.5414978e+02*mm2Tom2}"  ixz="${-1.1602420e+03*mm2Tom2}" iyy="${8.1906401e+03*mm2Tom2}" iyz="${-1.2050460e+03*mm2Tom2}" izz="${3.7083468e+03*mm2Tom2}" />
+    </inertial>
+    <visual>
+      <origin xyz="0. 0. 0." rpy="0 0 0."/>
+      <material name="dark_grey"/>
+      <geometry name="RHipMot_visual">
+        <mesh filename="package://cogimon_urdf/meshes/Leg0.STL" scale="${mmTom} ${mmTom} ${mmTom}" />
+      </geometry>
+    </visual>
+    <collision>
+      <origin xyz="0.0 0. 0" rpy="0 0 0."/>
+      <geometry name="RHipMot_collision">
+        <mesh filename="package://cogimon_urdf/meshes/simple/Leg0.STL" scale="${mmTom} ${mmTom} ${mmTom}" />
+      </geometry>
+    </collision>
+  </link>
+<!-- JOINTS -->
+<joint name="LHipLat" type="revolute">
+    <parent link="Waist"/>
+    <child link="LHipMot"/>
+    <origin xyz="${12.58*mmTom} ${110.954508*mmTom} ${-52.922586*mmTom}" rpy="0 0 0.0262" />
+    <axis xyz="1 0 0" />
+    <limit velocity="3.67" effort="176" lower="${-25.*toRad}" upper="${85.*toRad}" />
+    <dynamics friction="0" damping="3.0"/>
+  </joint>
+</xacro:if>
 <!-- LINKS -->
 <!-- ********************RIGHT LEG******************** -->
-<link name ="RHipMot">
-    <inertial>
-      <origin xyz="-3.269678E-4 -0.023587321 -2.6496509E-4" rpy="0 0 0"/>
-      <mass value="${wcf*0.89258227}"/>
-      <inertia ixx="${wcf*4.7672294E-4}"  ixy="${wcf*-3.9936567E-6}"  ixz="${wcf*-2.4802574E-6}" iyy="${wcf*5.458038E-4}" iyz="${wcf*-3.3389575E-6}" izz="${wcf*5.126859E-4}" />
-    </inertial>
-    <visual>
-      <origin xyz="0.0 0.023 -0.52" rpy="0 0 ${PI}"/>
-      <material name="dark_grey"/>
-      <geometry name="RHipMot_visual">
-        <mesh filename="package://cogimon_urdf/meshes/Leg0.STL" scale="${SF} ${SF} ${SF}" />
-      </geometry>
-    </visual>
-    <collision>
-      <origin xyz="0.0 0.023 -0.52" rpy="0 0 ${PI}"/>
-      <geometry name="RHipMot_collision">
-        <mesh filename="package://cogimon_urdf/meshes/simple/Leg0.STL" scale="${SF} ${SF} ${SF}" />
-      </geometry>
-    </collision>
-</link>
+<!--
   <link name ="RThighUpLeg">
     <inertial>
@@ -150,5 +192,7 @@
   </link>
   </xacro:unless>
+-->
 <!-- ********************LEFT LEG******************** -->
+<!--
   <link name ="LHipMot">
     <inertial>
@@ -295,14 +339,8 @@
     </link>
   </xacro:unless>
+  -->
 <!-- JOINTS -->
 <!-- ********************RIGHT LEG******************** -->
-  <joint name="RHipSag" type="revolute">
-    <parent link="Waist"/>
-    <child link="RHipMot"/>
-    <origin xyz="0.0 -0.023 0.0" rpy="0 0 0" />
-    <axis xyz="0 1 0" />
-    <limit velocity="4.0" effort="140" lower="-1.9199" upper="0.7854" />
-    <dynamics friction="0" damping="3.0"/>
-  </joint>
+  <!--
   <joint name="RHipLat" type="revolute">
     <parent link="RHipMot"/>
@@ -345,5 +383,7 @@
       <dynamics friction="0" damping="3.0"/>
   </joint>
+-->
 <!-- ********************LEFT LEG******************** -->
+<!--
   <joint name="LHipSag" type="revolute">
     <parent link="Waist"/>
@@ -394,3 +434,4 @@
       <dynamics friction="0" damping="3.0"/>
   </joint>
+-->
 </robot>

Commit message: added waist

File: cogimon_urdf/urdf/cogimon_base.urdf.xacro (robot description, xacro)
@@ -4,7 +4,6 @@
   ROS urdf definition of the COGIMON humanoid robot by Istituto Italiano di Tecnologia
   DO NOT INCLUDE THIS FILE DIRECTLY! USE cogimon_robot.urdf.xacro INSTEAD!
-  Author: Enrico Mingo & Alessio Rocchi
+  Author: Enrico Mingo Hoffman
   Inertial matrix has to be in CoM frame (URDF specs)
-  Velocity and effort limits are fake!
 -->
 <!-- This links are defined in order to be compliant with http://www.ros.org/reps/rep-0120.html#coordinate-frames
@@ -14,7 +13,7 @@
 <link name="Waist">
     <inertial>
-      <origin xyz="${-2.0579946e+01*mmTom} ${-1.0999634e+00*mmTom} ${-3.7500786e+01*mmTom}" rpy="0.0 0.0 0.0"/>
-      <mass value="4.2357548"/>
-      <inertia ixx="${4.6492739e+04*mm2Tom2}"  ixy="${3.4766548e+01*mm2Tom2}"  ixz="${3.2487180e+01*mm2Tom2}" iyy="${1.4654103e+04*mm2Tom2}" iyz="${9.3654340e+02*mm2Tom2}" izz="${5.0027621e+04*mm2Tom2}" />
+      <origin xyz="${-5.6796324e+01*mmTom} ${4.5196345e-01*mmTom} ${-3.8136153e+01*mmTom}" rpy="0.0 0.0 0.0"/>
+      <mass value="3.4599462"/>
+      <inertia ixx="${3.8130318e+04*mm2Tom2}"  ixy="${9.5451056e+01*mm2Tom2}"  ixz="${-8.2481481e+01*mm2Tom2}" iyy="${8.9760596e+03*mm2Tom2}" iyz="${9.1637353e+00*mm2Tom2}" izz="${3.9650845e+04*mm2Tom2}" />
     </inertial>
     <visual>
@@ -22,5 +21,5 @@
       <material name="dark_grey"/>
       <geometry name="Waist_visual">
-        <mesh filename="package://cogimon_urdf/meshes/Waist.STL" scale="${mmTom} ${mmTom} ${mmTom}"/>
+        <mesh filename="package://cogimon_urdf/meshes/Waist.stl" scale="${mmTom} ${mmTom} ${mmTom}"/>
       </geometry>
     </visual>
@@ -28,5 +27,5 @@
       <origin xyz="0 0 0" rpy="0 0 0"/>
       <geometry name="Waist_collision">
-        <mesh filename="package://cogimon_urdf/meshes/simple/Waist.STL" scale="${mmTom} ${mmTom} ${mmTom}"/>
+        <mesh filename="package://cogimon_urdf/meshes/simple/Waist.stl" scale="${mmTom} ${mmTom} ${mmTom}"/>
       </geometry>
     </collision>
@@ -52,5 +51,5 @@
   <!--link name="l_toe"/>
   <link name="r_toe"/-->
-<xacro:include filename="$(find cogimon_urdf)/urdf/parts/legs.urdf.xacro" />
+<!--xacro:include filename="$(find cogimon_urdf)/urdf/parts/legs.urdf.xacro" /-->
 <!--
   <joint name="l_ankle_joint" type="fixed">

File: cogimon_urdf/urdf/cogimon_config.urdf.xacro (robot description, xacro)
@@ -5,11 +5,15 @@
 <!-- ************SELECT PARTS*************-->
 <!-- *************************************-->
-<xacro:property name="COGIMON_TORSO" value="false" />
-<xacro:property name="COGIMON_LEFT_ARM" value="false" />
-<xacro:property name="COGIMON_RIGHT_ARM" value="false" />
-<xacro:property name="COGIMON_LEFT_LEG" value="false" />
+<xacro:property name="COGIMON_TORSO" value="true" />
+<xacro:property name="COGIMON_LEFT_ARM" value="true" />
+<xacro:property name="COGIMON_RIGHT_ARM" value="true" />
+<xacro:property name="COGIMON_LEFT_LEG" value="true" />
 <xacro:property name="COGIMON_RIGHT_LEG" value="true" />
-<!-- ************SELECT FIXED BASE*************-->
+<!-- ************FLOATING BASE*************-->
 <!-- ******************************************-->
-<xacro:property name="COGIMON_FIXED_BASE" value="false" />
+<xacro:property name="COGIMON_FLOATING_BASE" value="true" />
+<!-- ************XBOT FRAMEWORK*************-->
+<!-- *************************************-->
+-->
+<xacro:property name="COGIMON_XBOT" value="false" />
 </robot>

File: cogimon_urdf/urdf/cogimon_robot.urdf.xacro (robot description, xacro)
@@ -16,5 +16,5 @@
   <xacro:include filename="$(find cogimon_urdf)/urdf/gazebo/cogimon_materials.gazebo.xacro" />
   <xacro:include filename="$(find cogimon_urdf)/urdf/gazebo/force_torque.gazebo.xacro" /-->
-<xacro:if value="${COGIMON_FIXED_BASE}" >
+<!--xacro:if value="${COGIMON_FIXED_BASE}" >
   <link name="world"/>
    <joint name="fixed" type="fixed">
@@ -22,5 +22,5 @@
     <child link="base_link"/>
   </joint>
-</xacro:if>
+</xacro:if-->
 <origin xyz="0.0 0.0 0.8" rpy="0 0 0" />
 </robot>
