Commit message: Added first pair of joints

File: cogimon_urdf/urdf/cogimon_base.urdf.xacro (robot description, xacro)
@@ -51,5 +51,5 @@
   <!--link name="l_toe"/>
   <link name="r_toe"/-->
-<!--xacro:include filename="$(find cogimon_urdf)/urdf/parts/legs.urdf.xacro" /-->
+<xacro:include filename="$(find cogimon_urdf)/urdf/parts/legs.urdf.xacro" />
 <!--
   <joint name="l_ankle_joint" type="fixed">

File: cogimon_urdf/urdf/cogimon_materials.urdf.xacro (robot description, xacro)
@@ -10,3 +10,6 @@
   <color rgba="1.0 0.0 0.0 1"/>
 </material>
+<material name="green">
+  <color rgba="0.0 1.0 0.0 1"/>
+</material>
 </robot>

File: cogimon_urdf/urdf/cogimon_robot.urdf.xacro (robot description, xacro)
@@ -12,9 +12,6 @@
 	<xacro:include filename="$(find cogimon_urdf)/urdf/gazebo/openni_kinect.gazebo.xacro" />
   </xacro:if-->
-<!-- YARP PLUGINS for GAZEBO SIMULATION -->
-  <!--xacro:include filename="$(find cogimon_urdf)/urdf/gazebo/yarp_control.gazebo.xacro" />
   <xacro:include filename="$(find cogimon_urdf)/urdf/gazebo/cogimon_materials.gazebo.xacro" />
-  <xacro:include filename="$(find cogimon_urdf)/urdf/gazebo/force_torque.gazebo.xacro" /-->
-<!--xacro:if value="${COGIMON_FIXED_BASE}" >
+  <!--xacro:include filename="$(find cogimon_urdf)/urdf/gazebo/force_torque.gazebo.xacro" /-->
   <link name="world"/>
    <joint name="fixed" type="fixed">
@@ -22,5 +19,4 @@
     <child link="base_link"/>
   </joint>
-</xacro:if-->
 <origin xyz="0.0 0.0 0.8" rpy="0 0 0" />
 </robot>

File: cogimon_urdf/urdf/gazebo/cogimon_materials.gazebo.xacro (robot description, xacro)
@@ -4,104 +4,13 @@
   <material>Gazebo/DarkGrey</material>
 </gazebo>
-<gazebo reference="DWL">
-  <material>Gazebo/DarkGrey</material>
+<xacro:if value="${COGIMON_RIGHT_LEG}" >
+<gazebo reference="RHipMot">
+  <material>Gazebo/Green</material>
 </gazebo>
-<gazebo reference="DWS">
-  <material>Gazebo/DarkGrey</material>
+</xacro:if>
+<xacro:if value="${COGIMON_LEFT_LEG}" >
+<gazebo reference="LHipMot">
+  <material>Gazebo/Green</material>
 </gazebo>
-<gazebo reference="DWYTorso">
-  <material>Gazebo/Red</material>
-</gazebo>
-<gazebo reference="RShp">
-  <material>Gazebo/DarkGrey</material>
-</gazebo>
-<gazebo reference="RShr">
-  <material>Gazebo/DarkGrey</material>
-</gazebo>
-<gazebo reference="RShy">
-  <material>Gazebo/DarkGrey</material>
-</gazebo>
-<gazebo reference="RElb">
-  <material>Gazebo/DarkGrey</material>
-</gazebo>
-<gazebo reference="RForearm">
-  <material>Gazebo/DarkGrey</material>
-</gazebo>
-<xacro:if value="${GAZEBO_COGIMON_USES_FOREARMS}">
-  <gazebo reference="RWrMot2">
-    <material>Gazebo/Grey</material>
-  </gazebo>
-  <gazebo reference="RWrMot3">
-    <material>Gazebo/Grey</material>
-  </gazebo>
-  <xacro:if value="${GAZEBO_COGIMON_USES_SOFTHANDS}">
-    <gazebo reference="RSoftHand">
-      <material>Gazebo/DarkGrey</material>
-    </gazebo>
-  </xacro:if>
 </xacro:if>
-<gazebo reference="LShp">
-  <material>Gazebo/DarkGrey</material>
-</gazebo>
-<gazebo reference="LShr">
-  <material>Gazebo/DarkGrey</material>
-</gazebo>
-<gazebo reference="LShy">
-  <material>Gazebo/DarkGrey</material>
-</gazebo>
-<gazebo reference="LElb">
-  <material>Gazebo/DarkGrey</material>
-</gazebo>
-<gazebo reference="LForearm">
-  <material>Gazebo/DarkGrey</material>
-</gazebo>
-<xacro:if value="${GAZEBO_COGIMON_USES_FOREARMS}">
-  <gazebo reference="LWrMot2">
-    <material>Gazebo/Grey</material>
-  </gazebo>
-  <gazebo reference="LWrMot3">
-    <material>Gazebo/Grey</material>
-  </gazebo>
-  <xacro:if value="${GAZEBO_COGIMON_USES_SOFTHANDS}">
-    <gazebo reference="LSoftHand">
-      <material>Gazebo/DarkGrey</material>
-    </gazebo>
-  </xacro:if>
-</xacro:if>
-<gazebo reference="RHipMot">
-  <material>Gazebo/DarkGrey</material>
-</gazebo>
-<gazebo reference="RThighUpLeg">
-  <material>Gazebo/DarkGrey</material>
-</gazebo>
-<gazebo reference="RThighLowLeg">
-  <material>Gazebo/DarkGrey</material>
-</gazebo>
-<gazebo reference="RLowLeg">
-  <material>Gazebo/DarkGrey</material>
-</gazebo>
-<gazebo reference="RFootmot">
-  <material>Gazebo/DarkGrey</material>
-</gazebo>
-<gazebo reference="RFoot">
-  <material>Gazebo/DarkGrey</material>
-</gazebo>
-<gazebo reference="LHipMot">
-  <material>Gazebo/DarkGrey</material>
-</gazebo>
-<gazebo reference="LThighUpLeg">
-  <material>Gazebo/DarkGrey</material>
-</gazebo>
-<gazebo reference="LThighLowLeg">
-  <material>Gazebo/DarkGrey</material>
-</gazebo>
-<gazebo reference="LLowLeg">
-  <material>Gazebo/DarkGrey</material>
-</gazebo>
-<gazebo reference="LFootmot">
-  <material>Gazebo/DarkGrey</material>
-</gazebo>
-<gazebo reference="LFoot">
-  <material>Gazebo/DarkGrey</material>
-</gazebo>
 </robot>

File: cogimon_urdf/urdf/parts/legs.urdf.xacro (robot description, xacro)
@@ -1,17 +1,17 @@
 <?xml version="1.0"?>
 <robot xmlns:xacro="http://ros.org/wiki/xacro">
-<xacro:if value="${COGIMON_RIGHT_LEG}" >
+<xacro:if value="${COGIMON_LEFT_LEG}" >
 <!-- LINKS -->
-<link name ="RHipMot">
+<link name ="LHipMot">
     <inertial>
-      <origin xyz="${4.7902756e+00*mmTom} ${1.5595700e+01*mmTom} ${-6.0925801e+01*mmTom}" rpy="0 0 0"/>
-      <mass value="1.6995409"/>
-      <inertia ixx="${2.2053e+06*mm2Tom2}"  ixy="${-0.0066e+06*mm2Tom2}"  ixz="${0.0015e+06*mm2Tom2}" iyy="${2.7733e+06*mm2Tom2}" iyz="${0.0125e+06*mm2Tom2}" izz="${2.7756e+06*mm2Tom2}" />
+      <origin xyz="${-4.1435899e+01*mmTom} ${-2.4099021e-01*mmTom} ${-6.7437774e+01*mmTom}" rpy="0 0 0"/>
+      <mass value="2.0936467"/>
+      <inertia ixx="${2.0328644e+04*mm2Tom2}"  ixy="${1.2836757e+01*mm2Tom2}"  ixz="${-7.1832791e+03*mm2Tom2}" iyy="${2.4404941e+04*mm2Tom2}" iyz="${2.2892687e+01*mm2Tom2}" izz="${8.9864540e+03*mm2Tom2}" />
     </inertial>
     <visual>
-      <origin xyz="0.0 0 0" rpy="0 0 0"/>
-      <material name="dark_grey"/>
+      <origin xyz="0. 0. 0." rpy="0 0 0."/>
+      <material name="green"/>
       <geometry name="RHipMot_visual">
-        <mesh filename="package://cogimon_urdf/meshes/Leg0.STL" scale="${mmTom} ${-mmTom} ${mmTom}" />
+        <mesh filename="package://cogimon_urdf/meshes/HipRoll.stl" scale="${mmTom} ${mmTom} ${mmTom}" />
       </geometry>
     </visual>
@@ -19,137 +19,5 @@
       <origin xyz="0.0 0. 0" rpy="0 0 0."/>
       <geometry name="RHipMot_collision">
-        <mesh filename="package://cogimon_urdf/meshes/simple/Leg0.STL" scale="${mmTom} ${-mmTom} ${mmTom}" />
-      </geometry>
-    </collision>
-</link>
-<!--
-<link name ="RThighUpLeg">
-    <inertial>
-      <origin xyz="${2.9898120e-01*mmTom} ${6.5748642e+01*mmTom} ${-8.8443666e+01*mmTom}" rpy="0 0 0"/>
-      <mass value="1.9691802"/>
-      <inertia ixx="${2.7765e+06*mm2Tom2}"  ixy="${0.0058e+06*mm2Tom2}"  ixz="${-0.0085e+06*mm2Tom2}" iyy="${2.2120e+06*mm2Tom2}" iyz="${0.0082e+06*mm2Tom2}" izz="${2.7816e+06*mm2Tom2}" />
-    </inertial>
-    <visual>
-      <origin xyz="0.0 0 0" rpy="0 0 0"/>
-      <material name="dark_grey"/>
-      <geometry name="RThighUpLeg_visual">
-        <mesh filename="package://cogimon_urdf/meshes/Leg1.STL" scale="${mmTom} ${-mmTom} ${mmTom}" />
-      </geometry>
-    </visual>
-    <collision>
-      <origin xyz="0.0 0. 0." rpy="0 0 0"/>
-      <geometry name="RThighUpLeg_collision">
-        <mesh filename="package://cogimon_urdf/meshes/simple/Leg1.STL" scale="${mmTom} ${-mmTom} ${mmTom}" />
-      </geometry>
-    </collision>
-  </link>
-<link name ="RThighLowLeg">
-    <inertial>
-      <origin xyz="${-2.4777694e+01*mmTom} ${-5.3514533e+00*mmTom} ${-5.1363939e+01*mmTom}" rpy="0 0 0"/>
-      <mass value="2.3534104"/>
-      <inertia ixx="${1.5350e+05*mm2Tom2}"  ixy="${0.0012e+05*mm2Tom2}"  ixz="${-0.0215e+05*mm2Tom2}" iyy="${1.5484e+05*mm2Tom2}" iyz="${-0.0030e+05*mm2Tom2}" izz="${0.9917e+05*mm2Tom2}" />
-    </inertial>
-    <visual>
-      <origin xyz="0.0 0 0." rpy="0 0 0"/>
-      <material name="dark_grey"/>
-      <geometry name="LThighLowLeg_visual">
-        <mesh filename="package://cogimon_urdf/meshes/Leg2.STL" scale="${mmTom} ${-mmTom} ${mmTom}" />
-      </geometry>
-    </visual>
-    <collision>
-      <origin xyz="0.0 0 0" rpy="0 0 0"/>
-      <geometry name="LThighLowLeg_collision">
-        <mesh filename="package://cogimon_urdf/meshes/simple/Leg2.STL" scale="${mmTom} ${-mmTom} ${mmTom}" />
-      </geometry>
-    </collision>
-  </link>
--->
-<!-- JOINTS -->
-<joint name="RHipLat" type="revolute">
-    <parent link="Waist"/>
-    <child link="RHipMot"/>
-    <origin xyz="${12.58*mmTom} ${-110.954508*mmTom} ${-52.922586*mmTom}" rpy="0 0 0" />
-    <axis xyz="1 0 0" />
-    <limit velocity="3.67" effort="176" lower="${-85.*toRad}" upper="${25.*toRad}" />
-    <dynamics friction="0" damping="3.0"/>
-  </joint>
-<!--
-<joint name="RHipSag" type="revolute">
-    <parent link="RHipMot"/>
-    <child link="RThighUpLeg"/>
-    <origin xyz="${-8.5*mmTom} ${-73.9855*mmTom} ${-112.5*mmTom}" rpy="0 0 0" />
-    <axis xyz="0 1 0" />
-    <limit velocity="3.67" effort="176" lower="${-96.*toRad}" upper="${90.*toRad}" />
-    <dynamics friction="0" damping="3.0"/>
-  </joint>
-<joint name="RHipYaw" type="revolute">
-    <parent link="RThighUpLeg"/>
-    <child link="RThighLowLeg"/>
-    <origin xyz="${0.*mmTom} ${92.4945*mmTom} ${-239.0*mmTom}" rpy="0 0 0" />
-    <axis xyz="0 0 1" />
-    <limit velocity="13.6" effort="56" lower="${-75*toRad}" upper="${30*toRad}" />
-    <dynamics friction="0" damping="3.0"/>
-  </joint>
--->
-</xacro:if>
-<xacro:if value="${COGIMON_LEFT_LEG}" >
-<!-- LINKS -->
-<link name ="LHipMot">
-    <inertial>
-      <origin xyz="${4.7902756e+00*mmTom} ${-1.5595700e+01*mmTom} ${-6.0925801e+01*mmTom}" rpy="0 0 0"/>
-      <mass value="1.6995409"/>
-      <inertia ixx="${2.2053e+06*mm2Tom2}"  ixy="${0.0066e+06*mm2Tom2}"  ixz="${0.0015e+06*mm2Tom2}" iyy="${2.7733e+06*mm2Tom2}" iyz="${-0.0125e+06*mm2Tom2}" izz="${2.7756e+06*mm2Tom2}" />
-    </inertial>
-    <visual>
-      <origin xyz="0. 0. 0." rpy="0 0 0."/>
-      <material name="dark_grey"/>
-      <geometry name="RHipMot_visual">
-        <mesh filename="package://cogimon_urdf/meshes/Leg0.STL" scale="${mmTom} ${mmTom} ${mmTom}" />
-      </geometry>
-    </visual>
-    <collision>
-      <origin xyz="0.0 0. 0" rpy="0 0 0."/>
-      <geometry name="RHipMot_collision">
-        <mesh filename="package://cogimon_urdf/meshes/simple/Leg0.STL" scale="${mmTom} ${mmTom} ${mmTom}" />
-      </geometry>
-    </collision>
-  </link>
-  <link name ="LThighUpLeg">
-    <inertial>
-      <origin xyz="${2.9898120e-01*mmTom} ${-6.5748642e+01*mmTom} ${-8.8443666e+01*mmTom}" rpy="0 0 0"/>
-      <mass value="1.9691802"/>
-      <inertia ixx="${2.7765e+06*mm2Tom2}"  ixy="${-0.0058e+06*mm2Tom2}"  ixz="${-0.0085e+06*mm2Tom2}" iyy="${2.2120e+06*mm2Tom2}" iyz="${-0.0082e+06*mm2Tom2}" izz="${2.7816e+06*mm2Tom2}" />
-    </inertial>
-    <visual>
-      <origin xyz="0.0 0 0" rpy="0 0 0"/>
-      <material name="dark_grey"/>
-      <geometry name="LThighUpLeg_visual">
-        <mesh filename="package://cogimon_urdf/meshes/Leg1.STL" scale="${mmTom} ${mmTom} ${mmTom}" />
-      </geometry>
-    </visual>
-    <collision>
-      <origin xyz="0.0 0. 0." rpy="0 0 0"/>
-      <geometry name="LThighUpLeg_collision">
-        <mesh filename="package://cogimon_urdf/meshes/simple/Leg1.STL" scale="${mmTom} ${mmTom} ${mmTom}" />
-      </geometry>
-    </collision>
-  </link>
-<link name ="LThighLowLeg">
-    <inertial>
-      <origin xyz="${-2.4777694e+01*mmTom} ${5.3514533e+00*mmTom} ${-5.1363939e+01*mmTom}" rpy="0 0 0"/>
-      <mass value="2.3534104"/>
-      <inertia ixx="${1.5350e+05*mm2Tom2}"  ixy="${-0.0012e+05*mm2Tom2}"  ixz="${-0.0215e+05*mm2Tom2}" iyy="${1.5484e+05*mm2Tom2}" iyz="${0.0030e+05*mm2Tom2}" izz="${0.9917e+05*mm2Tom2}" />
-    </inertial>
-    <visual>
-      <origin xyz="0.0 0 0." rpy="0 0 0"/>
-      <material name="dark_grey"/>
-      <geometry name="LThighLowLeg_visual">
-        <mesh filename="package://cogimon_urdf/meshes/Leg2.STL" scale="${mmTom} ${mmTom} ${mmTom}" />
-      </geometry>
-    </visual>
-    <collision>
-      <origin xyz="0.0 0 0" rpy="0 0 0"/>
-      <geometry name="LThighLowLeg_collision">
-        <mesh filename="package://cogimon_urdf/meshes/simple/Leg2.STL" scale="${mmTom} ${mmTom} ${mmTom}" />
+        <mesh filename="package://cogimon_urdf/meshes/simple/HipRoll.stl" scale="${mmTom} ${mmTom} ${mmTom}" />
       </geometry>
     </collision>
@@ -159,315 +27,41 @@
     <parent link="Waist"/>
     <child link="LHipMot"/>
-    <origin xyz="${12.58*mmTom} ${110.954508*mmTom} ${-52.922586*mmTom}" rpy="0 0 0" />
+    <origin xyz="${15.45*mmTom} ${112.0*mmTom} ${-50.0*mmTom}" rpy="0 0 0" />
     <axis xyz="1 0 0" />
-    <limit velocity="3.67" effort="176" lower="${-25.*toRad}" upper="${85.*toRad}" />
+    <limit velocity="3.67" effort="176" lower="${-90.*toRad}" upper="${90.*toRad}" />
     <dynamics friction="0" damping="3.0"/>
-  </joint>
-<joint name="LHipSag" type="revolute">
-    <parent link="LHipMot"/>
-    <child link="LThighUpLeg"/>
-    <origin xyz="${-8.5*mmTom} ${73.9855*mmTom} ${-112.5*mmTom}" rpy="0 0 0" />
-    <axis xyz="0 1 0" />
-    <limit velocity="3.67" effort="176" lower="${-96.*toRad}" upper="${90.*toRad}" />
-    <dynamics friction="0" damping="3.0"/>
-  </joint>
-<joint name="LHipYaw" type="revolute">
-    <parent link="LThighUpLeg"/>
-    <child link="LThighLowLeg"/>
-    <origin xyz="${0.*mmTom} ${-92.4945*mmTom} ${-239.0*mmTom}" rpy="0 0 0" />
-    <axis xyz="0 0 1" />
-    <limit velocity="13.6" effort="56" lower="${-30*toRad}" upper="${75*toRad}" />
-    <dynamics friction="0" damping="3.0"/>
-  </joint>
+</joint>
 </xacro:if>
+<xacro:if value="${COGIMON_RIGHT_LEG}" >
 <!-- LINKS -->
-<!-- ********************RIGHT LEG******************** -->
-<!--
-  <link name ="RThighLowLeg">
+<link name ="RHipMot">
     <inertial>
-      <origin xyz="9.8720058E-4 6.7037262E-4 -0.075716843" rpy="0 0 0"/>
-      <mass value="${wcf*1.7001134}"/>
-      <inertia ixx="${wcf*0.0038979546}"  ixy="${wcf*1.7802399E-6}"  ixz="${wcf*2.6403262E-5}" iyy="${wcf*0.0039360845}" iyz="${wcf*4.522711E-5}" izz="${wcf*9.0218711E-4}" />
+      <origin xyz="${-4.1435899e+01*mmTom} ${2.4099021e-01*mmTom} ${-6.7437774e+01*mmTom}" rpy="0 0 0"/>
+      <mass value="2.0936467"/>
+      <inertia ixx="${2.0328644e+04*mm2Tom2}"  ixy="${-1.2836757e+01*mm2Tom2}"  ixz="${-7.1832791e+03*mm2Tom2}" iyy="${2.4404941e+04*mm2Tom2}" iyz="${-2.2892687e+01*mm2Tom2}" izz="${8.9864540e+03*mm2Tom2}" />
     </inertial>
     <visual>
-      <origin xyz="0.0 0.0726 -0.4176" rpy="0 0 ${PI}"/>
-      <material name="dark_grey"/>
-      <geometry name="RThighLowLeg_visual">
-        <mesh filename="package://cogimon_urdf/meshes/Leg2.STL" scale="${SF} ${SF} ${SF}" />
+      <origin xyz="0.0 0 0" rpy="0 0 0"/>
+      <material name="green"/>
+      <geometry name="RHipMot_visual">
+        <mesh filename="package://cogimon_urdf/meshes/HipRoll.stl" scale="${mmTom} ${-mmTom} ${mmTom}" />
       </geometry>
     </visual>
     <collision>
-      <origin xyz="0.0 0.0726 -0.4176" rpy="0 0 ${PI}"/>
-      <geometry name="RThighLowLeg_collision">
-        <mesh filename="package://cogimon_urdf/meshes/simple/Leg2.STL" scale="${SF} ${SF} ${SF}" />
+      <origin xyz="0.0 0. 0" rpy="0 0 0."/>
+      <geometry name="RHipMot_collision">
+        <mesh filename="package://cogimon_urdf/meshes/simple/HipRoll.stl" scale="${mmTom} ${-mmTom} ${mmTom}" />
       </geometry>
     </collision>
-  </link>
-  <link name ="RLowLeg">
-    <inertial>
-      <origin xyz="0.0024612666 -0.0053099614 -0.08598948" rpy="0 0 0"/>
-      <mass value="${wcf*1.4098179}"/>
-      <inertia ixx="${wcf*0.0040604004}"  ixy="${wcf*1.1227206E-5}"  ixz="${wcf*1.2260973E-5}" iyy="${wcf*0.004005652855}" iyz="${wcf*5.1899176E-4}" izz="${wcf*0.0012414054}" />
-    </inertial>
-    <visual>
-      <origin xyz="0.0 0.0726 -0.2942" rpy="0 0 ${PI}"/>
-      <material name="dark_grey"/>
-      <geometry name="RLowLeg_visual">
-        <mesh filename="package://cogimon_urdf/meshes/Leg3.STL" scale="${SF} ${SF} ${SF}" />
-      </geometry>
-    </visual>
-    <collision>
-      <origin xyz="0.0 0.0726 -0.2942" rpy="0 0 ${PI}"/>
-      <geometry name="RLowLeg_collision">
-        <mesh filename="package://cogimon_urdf/meshes/simple/Leg3.STL" scale="${SF} ${SF} ${SF}" />
-      </geometry>
-    </collision>
-  </link>
-  <link name ="RFootmot">
-    <inertial>
-      <origin xyz="8.8067281E-4 -9.2224881E-4 2.3038476E-4" rpy="0 0 0"/>
-      <mass value="${wcf*0.72992131}"/>
-      <inertia ixx="${wcf*3.2034425E-4}"  ixy="${wcf*7.6346303E-6}"  ixz="${wcf*2.5430158E-7}" iyy="${wcf*3.6584358E-4}" iyz="${wcf*-3.6889276E-6}" izz="${wcf*3.6065156E-4}" />
-    </inertial>
-    <visual>
-      <origin xyz="0.0 0.0726 -0.0932" rpy="0 0 ${PI}"/>
-      <material name="dark_grey"/>
-      <geometry name="RFootmot_visual">
-        <mesh filename="package://cogimon_urdf/meshes/Leg4.STL" scale="${SF} ${SF} ${SF}" />
-      </geometry>
-    </visual>
-    <collision>
-      <origin xyz="0.0 0.0726 -0.0932" rpy="0 0 ${PI}"/>
-      <geometry name="RFootmot_collision">
-        <mesh filename="package://cogimon_urdf/meshes/simple/Leg4.STL" scale="${SF} ${SF} ${SF}" />
-      </geometry>
-    </collision>
-  </link>
-  <xacro:if value="${GAZEBO_COGIMON_USES_ROUND_FEET}">
-    <link name ="RFoot">
-      <inertial>
-        <origin xyz="0.00969210464 -0.0090460227 -0.043062308" rpy="0 0 0"/>
-        <mass value="${wcf*0.66646684}"/>
-        <inertia ixx="${wcf*0.0012944808}"  ixy="${wcf*-9.2387693E-5}"  ixz="${wcf*2.0080105E-4}" iyy="${wcf*0.0015851846}" iyz="${wcf*2.7599327E-4}" izz="${wcf*0.0013326766}" />
-      </inertial>
-      <visual>
-        <origin xyz="0.0 0.0726 -0.0932" rpy="0 0 -3.14159265359"/>
-        <material name="dark_grey"/>
-        <geometry name="RFoot_visual">
-          <mesh filename="package://cogimon_urdf/meshes/RoundFoot.STL" scale="0.03937 0.03937 0.03937" />
-        </geometry>
-      </visual>
-      <collision>
-        <origin xyz="0.0 0.0726 -0.0932" rpy="0 0 -3.14159265359"/>
-        <geometry name="RFoot_collision">
-          <mesh filename="package://cogimon_urdf/meshes/simple/RoundFoot.STL" scale="0.03937 0.03937 0.03937" />
-        </geometry>
-      </collision>
-    </link>
-  </xacro:if>
-  <xacro:unless value="${GAZEBO_COGIMON_USES_ROUND_FEET}">
-    <link name ="RFoot">
-      <inertial>
-        <origin xyz="0.00969210464 -0.0090460227 -0.043062308" rpy="0 0 0"/>
-        <mass value="${wcf*0.66646684}"/>
-        <inertia ixx="${wcf*0.0012944808}"  ixy="${wcf*-9.2387693E-5}"  ixz="${wcf*2.0080105E-4}" iyy="${wcf*0.0015851846}" iyz="${wcf*2.7599327E-4}" izz="${wcf*0.0013326766}" />
-      </inertial>
-    <visual>
-     <origin xyz="0.03 0 -0.07" rpy="0 0 0" />
-     <geometry>
-       <box size="0.2 0.12 0.04" />
-     </geometry>
-     <material name="dark_gray"/>
-   </visual>
-   <collision>
-     <origin xyz="0.03 0 -0.07" rpy="0 0 0"/>
-     <geometry>
-       <box size="0.2 0.12 0.04" />
-     </geometry>
-   </collision>
-  </link>
-  </xacro:unless>
--->
-<!-- ********************LEFT LEG******************** -->
-<!--
-  <link name ="LLowLeg">
-    <inertial>
-      <origin xyz="0.0024612666 0.0053099614 -0.085989484" rpy="0 0 0"/>
-      <mass value="${wcf*1.4098179}"/>
-      <inertia ixx="${wcf*0.0040604004}"  ixy="${wcf*-1.1227206E-5}"  ixz="${wcf*1.2260973E-5}" iyy="${wcf*0.004005652855}" iyz="${wcf*-5.1899176E-4}" izz="${wcf*0.0012414054}" />
-    </inertial>
-    <visual>
-      <origin xyz="0.0 -0.0726 -0.2942" rpy="0 0 ${PI}"/>
-      <material name="dark_grey"/>
-      <geometry name="LLowLeg_visual">
-        <mesh filename="package://cogimon_urdf/meshes/Leg3.STL" scale="${SF} -${SF} ${SF}" />
-      </geometry>
-    </visual>
-    <collision>
-      <origin xyz="0.0 -0.0726 -0.2942" rpy="0 0 ${PI}"/>
-      <geometry name="LLowLeg_collision">
-        <mesh filename="package://cogimon_urdf/meshes/simple/Leg3.STL" scale="${SF} -${SF} ${SF}" />
-      </geometry>
-    </collision>
-  </link>
-  <link name ="LFootmot">
-    <inertial>
-      <origin xyz="8.8067281E-4 9.2224881E-4 2.3038476E-4" rpy="0 0 0"/>
-      <mass value="${wcf*0.72992131}"/>
-      <inertia ixx="${wcf*3.2034425E-4}"  ixy="${wcf*-7.6346303E-6}"  ixz="${wcf*2.5430158E-7}" iyy="${wcf*3.6584358E-4}" iyz="${wcf*3.6889276E-6}" izz="${wcf*3.6065156E-4}" />
-    </inertial>
-    <visual>
-      <origin xyz="0.0 -0.0726 -0.0932" rpy="0 0 ${PI}"/>
-      <material name="dark_grey"/>
-      <geometry name="LFootmot_visual">
-        <mesh filename="package://cogimon_urdf/meshes/Leg4.STL" scale="${SF} -${SF} ${SF}" />
-      </geometry>
-    </visual>
-    <collision>
-      <origin xyz="0.0 -0.0726 -0.0932" rpy="0 0 ${PI}"/>
-      <geometry name="LFootmot_collision">
-        <mesh filename="package://cogimon_urdf/meshes/simple/Leg4.STL" scale="${SF} -${SF} ${SF}" />
-      </geometry>
-    </collision>
-  </link>
-  <xacro:if value="${GAZEBO_COGIMON_USES_ROUND_FEET}">
-    <link name ="LFoot">
-      <inertial>
-        <origin xyz="0.0096921046 0.0090460227 -0.043062308" rpy="0 0 0"/>
-        <mass value="${wcf*0.66646684}"/>
-        <inertia ixx="${wcf*0.0012944808}"  ixy="${wcf*9.2387693E-5}"  ixz="${wcf*2.0080105E-4}" iyy="${wcf*0.0015851846}" iyz="${wcf*-2.7599327E-4}" izz="${wcf*0.0013326766}" />
-      </inertial>
-      <visual>
-        <origin xyz="0.0 -0.0726 -0.0932" rpy="0 0 -3.14159265359"/>
-        <material name="dark_grey"/>
-        <geometry name="LFoot_visual">
-          <mesh filename="package://cogimon_urdf/meshes/RoundFoot.STL" scale="0.03937 -0.03937 0.03937" />
-        </geometry>
-      </visual>
-      <collision>
-        <origin xyz="0.0 -0.0726 -0.0932" rpy="0 0 -3.14159265359"/>
-        <geometry name="LFoot_collision">
-          <mesh filename="package://cogimon_urdf/meshes/simple/RoundFoot.STL" scale="0.03937 -0.03937 0.03937" />
-        </geometry>
-      </collision>
-    </link>
-  </xacro:if>
-  <xacro:unless value="${GAZEBO_COGIMON_USES_ROUND_FEET}">
-    <link name ="LFoot">
-      <inertial>
-        <origin xyz="0.0096921046 0.0090460227 -0.043062308" rpy="0 0 0"/>
-        <mass value="${wcf*0.66646684}"/>
-        <inertia ixx="${wcf*0.0012944808}"  ixy="${wcf*9.2387693E-5}"  ixz="${wcf*2.0080105E-4}" iyy="${wcf*0.0015851846}" iyz="${wcf*-2.7599327E-4}" izz="${wcf*0.0013326766}" />
-      </inertial>
-      <visual>
-       <origin xyz="0.03 0 -0.07" rpy="0 0 0" />
-       <geometry>
-         <box size="0.2 0.12 0.04" />
-       </geometry>
-       <material name="dark_gray"/>
-     </visual>
-     <collision>
-       <origin xyz="0.03 0 -0.07" rpy="0 0 0"/>
-       <geometry>
-         <box size="0.2 0.12 0.04" />
-       </geometry>
-     </collision>
-    </link>
-  </xacro:unless>
-  -->
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