Commit message: Added torso roll

File: cogimon_urdf/urdf/cogimon_base.urdf.xacro (robot description, xacro)
@@ -37,3 +37,4 @@
 </joint>
 <xacro:include filename="$(find cogimon_urdf)/urdf/parts/legs.urdf.xacro" />
+<xacro:include filename="$(find cogimon_urdf)/urdf/parts/torso.urdf.xacro" />
 </robot>

File: cogimon_urdf/urdf/cogimon_config.urdf.xacro (robot description, xacro)
@@ -6,6 +6,6 @@
 <!-- *************************************-->
 <xacro:property name="COGIMON_TORSO" value="true" />
-<xacro:property name="COGIMON_LEFT_ARM" value="true" />
-<xacro:property name="COGIMON_RIGHT_ARM" value="true" />
+<xacro:property name="COGIMON_LEFT_ARM" value="false" />
+<xacro:property name="COGIMON_RIGHT_ARM" value="false" />
 <xacro:property name="COGIMON_LEFT_LEG" value="true" />
 <xacro:property name="COGIMON_RIGHT_LEG" value="true" />

File: cogimon_urdf/urdf/gazebo/cogimon.gazebo.xacro (robot description, xacro)
@@ -77,3 +77,9 @@
   </gazebo>
 </xacro:if>
+<xacro:if value="${COGIMON_TORSO}">
+   <gazebo reference="DWL">
+    <implicitSpringDamper>1</implicitSpringDamper>
+    <provideFeedback>true</provideFeedback>
+   </gazebo>
+</xacro:if>
 </robot>

File: cogimon_urdf/urdf/gazebo/cogimon_materials.gazebo.xacro (robot description, xacro)
@@ -44,3 +44,8 @@
 </gazebo>
 </xacro:if>
+<xacro:if value="${COGIMON_TORSO}">
+<gazebo reference="DWL">
+  <material>Gazebo/DarkGrey</material>
+</gazebo>
+</xacro:if>
 </robot>

Commit message: Added imu

File: cogimon_urdf/urdf/cogimon_base.urdf.xacro (robot description, xacro)
@@ -36,4 +36,16 @@
     <origin xyz="0 0 0" rpy="0 0 0" />
 </joint>
+<joint name="imu_joint" type="fixed">
+    <parent link="Waist"/>
+    <child link="imu_link"/>
+    <origin xyz="0 0 0" rpy="0 0 0" />
+</joint>
+<link name="imu_link">
+    <inertial>
+      <origin xyz="0 0 0" rpy="0.0 0.0 0.0"/>
+      <mass value="0"/>
+      <inertia ixx="0"  ixy="0"  ixz="0" iyy="0" iyz="0" izz="0" />
+    </inertial>
+</link>
 <xacro:include filename="$(find cogimon_urdf)/urdf/parts/legs.urdf.xacro" />
 <xacro:include filename="$(find cogimon_urdf)/urdf/parts/torso.urdf.xacro" />

File: cogimon_urdf/urdf/cogimon_robot.urdf.xacro (robot description, xacro)
@@ -10,4 +10,5 @@
   <xacro:include filename="$(find cogimon_urdf)/urdf/gazebo/cogimon_materials.gazebo.xacro" />
   <xacro:include filename="$(find cogimon_urdf)/urdf/gazebo/force_torque.gazebo.xacro" />
+  <xacro:include filename="$(find cogimon_urdf)/urdf/gazebo/imu.gazebo.xacro" />
 <xacro:if value="${COGIMON_XBOT_GAZEBO}" >
   <xacro:include filename="$(find cogimon_urdf)/urdf/gazebo/xbot_control.gazebo.xacro" />

Commit message: Added fixed neck

File: cogimon_urdf/urdf/cogimon_base.urdf.xacro (robot description, xacro)
@@ -52,3 +52,4 @@
 <xacro:include filename="$(find cogimon_urdf)/urdf/parts/torso.urdf.xacro" />
 <xacro:include filename="$(find cogimon_urdf)/urdf/parts/arms.urdf.xacro" />
+<xacro:include filename="$(find cogimon_urdf)/urdf/parts/head.urdf.xacro" />
 </robot>

File: cogimon_urdf/urdf/cogimon_config.urdf.xacro (robot description, xacro)
@@ -5,4 +5,5 @@
 <!-- ************SELECT PARTS*************-->
 <!-- *************************************-->
+<xacro:property name="COGIMON_HEAD" value="true" />
 <xacro:property name="COGIMON_TORSO" value="true" />
 <xacro:property name="COGIMON_LEFT_ARM" value="true" />
@@ -10,4 +11,12 @@
 <xacro:property name="COGIMON_LEFT_LEG" value="true" />
 <xacro:property name="COGIMON_RIGHT_LEG" value="true" />
+<!-- ************COGIMON_LASER_FIXED*******-->
+<!--
+     This will set the laser joint to 'fixed'.
+     Should be used to true for the urdf and srdf which are
+     used in the hardware and visualization, not for IK and ID.
+-->
+<!-- *************************************-->
+<xacro:property name="COGIMON_LASER_FIXED" value="true" />
 <!-- ************COGIMON_PENNACCHIO*******-->
 <!--

File: cogimon_urdf/urdf/config/cogimon.urdf.xacro (robot description, xacro)
@@ -5,5 +5,5 @@
 <!-- ************SELECT PARTS*************-->
 <!-- *************************************-->
-<xacro:property name="COGIMON_HEAD" value="false" />
+<xacro:property name="COGIMON_HEAD" value="true" />
 <xacro:property name="COGIMON_TORSO" value="true" />
 <xacro:property name="COGIMON_LEFT_ARM" value="true" />
@@ -11,4 +11,12 @@
 <xacro:property name="COGIMON_LEFT_LEG" value="true" />
 <xacro:property name="COGIMON_RIGHT_LEG" value="true" />
+<!-- ************COGIMON_LASER_FIXED*******-->
+<!--
+     This will set the laser joint to 'fixed'.
+     Should be used to true for the urdf and srdf which are
+     used in the hardware and visualization, not for IK and ID.
+-->
+<!-- *************************************-->
+<xacro:property name="COGIMON_LASER_FIXED" value="true" />
 <!-- ************COGIMON_PENNACCHIO*******-->
 <!--

File: cogimon_urdf/urdf/config/cogimon_hardware.urdf.xacro (robot description, xacro)
@@ -11,4 +11,12 @@
 <xacro:property name="COGIMON_LEFT_LEG" value="true" />
 <xacro:property name="COGIMON_RIGHT_LEG" value="true" />
+<!-- ************COGIMON_LASER_FIXED*******-->
+<!--
+     This will set the laser joint to 'fixed'.
+     Should be used to true for the urdf and srdf which are
+     used in the hardware and visualization, not for IK and ID.
+-->
+<!-- *************************************-->
+<xacro:property name="COGIMON_LASER_FIXED" value="false" />
 <!-- ************COGIMON_PENNACCHIO*******-->
 <!--

File: cogimon_urdf/urdf/config/cogimon_pennacchio.urdf.xacro (robot description, xacro)
@@ -11,4 +11,12 @@
 <xacro:property name="COGIMON_LEFT_LEG" value="true" />
 <xacro:property name="COGIMON_RIGHT_LEG" value="true" />
+<!-- ************COGIMON_LASER_FIXED*******-->
+<!--
+     This will set the laser joint to 'fixed'.
+     Should be used to true for the urdf and srdf which are
+     used in the hardware and visualization, not for IK and ID.
+-->
+<!-- *************************************-->
+<xacro:property name="COGIMON_LASER_FIXED" value="true" />
 <!-- ************COGIMON_PENNACCHIO*******-->
 <!--

File: cogimon_urdf/urdf/gazebo/cogimon.gazebo.xacro (robot description, xacro)
@@ -90,5 +90,5 @@
 </xacro:if>
 <xacro:if value="${COGIMON_LEFT_ARM}">
-<gazebo reference="LShSag">
+   <gazebo reference="LShSag">
     <implicitSpringDamper>1</implicitSpringDamper>
     <provideFeedback>true</provideFeedback>
@@ -120,5 +120,5 @@
 </xacro:if>
 <xacro:if value="${COGIMON_RIGHT_ARM}">
-<gazebo reference="RShSag">
+   <gazebo reference="RShSag">
     <implicitSpringDamper>1</implicitSpringDamper>
     <provideFeedback>true</provideFeedback>
@@ -149,3 +149,5 @@
   </gazebo>
 </xacro:if>
+<xacro:if value="${COGIMON_HEAD}">
+</xacro:if>
 </robot>

Commit message: Added soft hands

File: cogimon_urdf/urdf/cogimon_base.urdf.xacro (robot description, xacro)
@@ -52,3 +52,4 @@
 <xacro:include filename="$(find cogimon_urdf)/urdf/parts/torso.urdf.xacro" />
 <xacro:include filename="$(find cogimon_urdf)/urdf/parts/arms.urdf.xacro" />
+<xacro:include filename="$(find cogimon_urdf)/urdf/parts/soft_hands.urdf.xacro" />
 </robot>

File: cogimon_urdf/urdf/parts/arms.urdf.xacro (robot description, xacro)
@@ -147,4 +147,24 @@
  </collision>
 </link>
+<link name="r_wrist">
+    <inertial>
+      <origin xyz="${8.2161929e-02*mmTom} ${-2.6334189*mmTom} ${-1.6465877e+01*mmTom}" rpy="0 0 0"/>
+      <mass value="3.7827821e-01"/>
+      <inertia ixx="${2.3321716e+02*mm2Tom2}"  ixy="${-2.3681435*mm2Tom2}"  ixz="${-1.8039102*mm2Tom2}" iyy="${2.0626291e+02*mm2Tom2}" iyz="${-3.1588290e+01*mm2Tom2}" izz="${2.7399881e+02*mm2Tom2}" />
+    </inertial>
+    <visual>
+      <origin xyz="0 0 0" rpy="${PI} 0 0"/>
+      <geometry name="RShp_visual">
+        <mesh filename="package://cogimon_urdf/meshes/Wrist.STL" scale="0.001 0.001 0.001" />
+      </geometry>
+      <material name="dark_grey"/>
+    </visual>
+    <collision>
+      <origin xyz="0 0 0" rpy="${PI} 0 0"/>
+      <geometry name="RShp_collision">
+        <mesh filename="package://cogimon_urdf/meshes/simple/Wrist.STL" scale="0.001 0.001 0.001" />
+      </geometry>
+    </collision>
+</link>
 <joint name="RShSag" type="revolute">
     <parent link="DWYTorso"/>
@@ -203,4 +223,9 @@
        <dynamics friction="0" damping="0.03"/>
 </joint>
+<joint name="r_wrist_joint" type="fixed">
+       <parent link="RWrMot3"/>
+       <child link="r_wrist"/>
+       <origin xyz="0 0 0" rpy="0 0 0" />
+</joint>
 </xacro:if>
 <xacro:if value="${COGIMON_LEFT_ARM}">
@@ -345,4 +370,24 @@
    </geometry>
  </collision>
+</link>
+<link name="l_wrist">
+    <inertial>
+      <origin xyz="${8.2161929e-02*mmTom} ${2.6334189*mmTom} ${-1.6465877e+01*mmTom}" rpy="0 0 0"/>
+      <mass value="3.7827821e-01"/>
+      <inertia ixx="${2.3321716e+02*mm2Tom2}"  ixy="${2.3681435*mm2Tom2}"  ixz="${-1.8039102*mm2Tom2}" iyy="${2.0626291e+02*mm2Tom2}" iyz="${3.1588290e+01*mm2Tom2}" izz="${2.7399881e+02*mm2Tom2}" />
+    </inertial>
+    <visual>
+      <origin xyz="0 0 0" rpy="${PI} 0 0"/>
+      <geometry name="LShp_visual">
+        <mesh filename="package://cogimon_urdf/meshes/Wrist.STL" scale="0.001 -0.001 0.001" />
+      </geometry>
+      <material name="dark_grey"/>
+    </visual>
+    <collision>
+      <origin xyz="0 0 0" rpy="${PI} 0 0"/>
+      <geometry name="LShp_collision">
+        <mesh filename="package://cogimon_urdf/meshes/simple/Wrist.STL" scale="0.001 -0.001 0.001" />
+      </geometry>
+    </collision>
 </link>
 <joint name="LShSag" type="revolute">
@@ -402,4 +447,9 @@
        <dynamics friction="0" damping="0.03"/>
 </joint>
+<joint name="l_wrist_joint" type="fixed">
+       <parent link="LWrMot3"/>
+       <child link="l_wrist"/>
+       <origin xyz="0 0 0" rpy="0 0 0" />
+</joint>
 </xacro:if>
 </robot>

Commit message: Fixed imu position

File: cogimon_urdf/urdf/cogimon_base.urdf.xacro (robot description, xacro)
@@ -39,5 +39,5 @@
     <parent link="Waist"/>
     <child link="imu_link"/>
-    <origin xyz="0 0 0" rpy="0 0 0" />
+    <origin xyz="${-146.332*mmTom} 0 ${-38.75*mmTom}" rpy="0 0 0" />
 </joint>
 <link name="imu_link">

Commit message: Added balls end-effectors

File: cogimon_urdf/urdf/cogimon_base.urdf.xacro (robot description, xacro)
@@ -59,4 +59,5 @@
 <xacro:include filename="$(find cogimon_urdf)/urdf/parts/arms.urdf.xacro" />
 <xacro:include filename="$(find cogimon_urdf)/urdf/parts/head.urdf.xacro" />
-<xacro:include filename="$(find cogimon_urdf)/urdf/parts/soft_hands.urdf.xacro" />
+<!-- xacro:include filename="$(find cogimon_urdf)/urdf/parts/soft_hands.urdf.xacro" / -->
+<xacro:include filename="$(find cogimon_urdf)/urdf/parts/ball_endeff.urdf.xacro" />
 </robot>

File: cogimon_urdf/urdf/parts/arms_macro.urdf.xacro (robot description, xacro)
@@ -142,24 +142,4 @@
    </geometry>
  </collision>
-</link>
-<link name="r_wrist">
-    <inertial>
-      <origin xyz="${8.2161929e-02*mmTom} ${-2.6334189*mmTom} ${-1.6465877e+01*mmTom}" rpy="0 0 0"/>
-      <mass value="3.7827821e-01"/>
-      <inertia ixx="${2.3321716e+02*mm2Tom2}"  ixy="${-2.3681435*mm2Tom2}"  ixz="${-1.8039102*mm2Tom2}" iyy="${2.0626291e+02*mm2Tom2}" iyz="${-3.1588290e+01*mm2Tom2}" izz="${2.7399881e+02*mm2Tom2}" />
-    </inertial>
-    <visual>
-      <origin xyz="0 0 0" rpy="${PI} 0 0"/>
-      <geometry name="RShp_visual">
-        <mesh filename="package://cogimon_urdf/meshes/Wrist.STL" scale="0.001 0.001 0.001" />
-      </geometry>
-      <material name="dark_grey"/>
-    </visual>
-    <collision>
-      <origin xyz="0 0 0" rpy="${PI} 0 0"/>
-      <geometry name="RShp_collision">
-        <mesh filename="package://cogimon_urdf/meshes/simple/Wrist.STL" scale="0.001 0.001 0.001" />
-      </geometry>
-    </collision>
 </link>
 <joint name="${joint1_name}" type="revolute">
@@ -219,9 +199,4 @@
        <dynamics friction="0" damping="0.03"/>
 </joint>
-<joint name="r_wrist_joint" type="fixed">
-       <parent link="RWrMot3"/>
-       <child link="r_wrist"/>
-       <origin xyz="0 0 0" rpy="0 0 0" />
-</joint>
 </xacro:macro>
 <xacro:macro name="left_arm" params="joint1_name joint2_name joint3_name joint4_name joint5_name joint6_name joint7_name">
@@ -366,24 +341,4 @@
    </geometry>
  </collision>
-</link>
-<link name="l_wrist">
-    <inertial>
-      <origin xyz="${8.2161929e-02*mmTom} ${2.6334189*mmTom} ${-1.6465877e+01*mmTom}" rpy="0 0 0"/>
-      <mass value="3.7827821e-01"/>
-      <inertia ixx="${2.3321716e+02*mm2Tom2}"  ixy="${2.3681435*mm2Tom2}"  ixz="${-1.8039102*mm2Tom2}" iyy="${2.0626291e+02*mm2Tom2}" iyz="${3.1588290e+01*mm2Tom2}" izz="${2.7399881e+02*mm2Tom2}" />
-    </inertial>
-    <visual>
-      <origin xyz="0 0 0" rpy="${PI} 0 0"/>
-      <geometry name="LShp_visual">
-        <mesh filename="package://cogimon_urdf/meshes/Wrist.STL" scale="0.001 -0.001 0.001" />
-      </geometry>
-      <material name="dark_grey"/>
-    </visual>
-    <collision>
-      <origin xyz="0 0 0" rpy="${PI} 0 0"/>
-      <geometry name="LShp_collision">
-        <mesh filename="package://cogimon_urdf/meshes/simple/Wrist.STL" scale="0.001 -0.001 0.001" />
-      </geometry>
-    </collision>
 </link>
 <joint name="${joint1_name}" type="revolute">
@@ -443,9 +398,4 @@
        <dynamics friction="0" damping="0.03"/>
 </joint>
-<joint name="l_wrist_joint" type="fixed">
-       <parent link="LWrMot3"/>
-       <child link="l_wrist"/>
-       <origin xyz="0 0 0" rpy="0 0 0" />
-</joint>
 </xacro:macro>
 </robot>

File: cogimon_urdf/urdf/parts/soft_hands.urdf.xacro (robot description, xacro)
@@ -7,4 +7,24 @@
 <link name="RSoftHand"/>
 <link name="TCP_R"/>
+<link name="r_wrist">
+    <inertial>
+      <origin xyz="${8.2161929e-02*mmTom} ${-2.6334189*mmTom} ${-1.6465877e+01*mmTom}" rpy="0 0 0"/>
+      <mass value="3.7827821e-01"/>
+      <inertia ixx="${2.3321716e+02*mm2Tom2}"  ixy="${-2.3681435*mm2Tom2}"  ixz="${-1.8039102*mm2Tom2}" iyy="${2.0626291e+02*mm2Tom2}" iyz="${-3.1588290e+01*mm2Tom2}" izz="${2.7399881e+02*mm2Tom2}" />
+    </inertial>
+    <visual>
+      <origin xyz="0 0 0" rpy="${PI} 0 0"/>
+      <geometry name="RShp_visual">
+        <mesh filename="package://cogimon_urdf/meshes/Wrist.STL" scale="0.001 0.001 0.001" />
+      </geometry>
+      <material name="dark_grey"/>
+    </visual>
+    <collision>
+      <origin xyz="0 0 0" rpy="${PI} 0 0"/>
+      <geometry name="RShp_collision">
+        <mesh filename="package://cogimon_urdf/meshes/simple/Wrist.STL" scale="0.001 0.001 0.001" />
+      </geometry>
+    </collision>
+</link>
 <link name="RSoftHandLink">
     <inertial>
@@ -27,4 +47,9 @@
    </collision>
 </link>
+<joint name="r_wrist_joint" type="fixed">
+       <parent link="RWrMot3"/>
+       <child link="r_wrist"/>
+       <origin xyz="0 0 0" rpy="0 0 0" />
+</joint>
 <joint name="r_handj" type="fixed">
         <parent link="r_wrist"/>
@@ -46,4 +71,24 @@
 <link name="LSoftHand"/>
 <link name="TCP_L"/>
+<link name="l_wrist">
+    <inertial>
+      <origin xyz="${8.2161929e-02*mmTom} ${2.6334189*mmTom} ${-1.6465877e+01*mmTom}" rpy="0 0 0"/>
+      <mass value="3.7827821e-01"/>
+      <inertia ixx="${2.3321716e+02*mm2Tom2}"  ixy="${2.3681435*mm2Tom2}"  ixz="${-1.8039102*mm2Tom2}" iyy="${2.0626291e+02*mm2Tom2}" iyz="${3.1588290e+01*mm2Tom2}" izz="${2.7399881e+02*mm2Tom2}" />
+    </inertial>
+    <visual>
+      <origin xyz="0 0 0" rpy="${PI} 0 0"/>
+      <geometry name="LShp_visual">
+        <mesh filename="package://cogimon_urdf/meshes/Wrist.STL" scale="0.001 -0.001 0.001" />
+      </geometry>
+      <material name="dark_grey"/>
+    </visual>
+    <collision>
+      <origin xyz="0 0 0" rpy="${PI} 0 0"/>
+      <geometry name="LShp_collision">
+        <mesh filename="package://cogimon_urdf/meshes/simple/Wrist.STL" scale="0.001 -0.001 0.001" />
+      </geometry>
+    </collision>
+</link>
 <link name="LSoftHandLink">
     <inertial>
@@ -67,4 +112,9 @@
 </link>
 <!-- JOINTS -->
+<joint name="l_wrist_joint" type="fixed">
+       <parent link="LWrMot3"/>
+       <child link="l_wrist"/>
+       <origin xyz="0 0 0" rpy="0 0 0" />
+</joint>
   <joint name="l_handj" type="fixed">
         <parent link="l_wrist"/>

Commit message: modified imu_link w.r.t. Waist

File: cogimon_urdf/urdf/cogimon_base.urdf.xacro (robot description, xacro)
@@ -39,5 +39,6 @@
     <parent link="Waist"/>
     <child link="imu_link"/>
-    <origin xyz="${-146.332*mmTom} 0 ${-38.75*mmTom}" rpy="0 0 0" />
+    <!--origin xyz="${-146.332*mmTom} 0 ${-38.75*mmTom}" rpy="0 0 0" /-->
+    <origin xyz="${-78.5400*mmTom} 0 ${-59.100*mmTom}" rpy="0 0 0" />
 </joint>
 <link name="imu_link">
