Commit message: Added capsules files

File: cogimon_urdf/urdf/cogimon_config.urdf.xacro (robot description, xacro)
@@ -1,5 +1,5 @@
 <?xml version="1.0"?>
 <robot xmlns:xacro="http://ros.org/wiki/xacro" name="COGIMON">
-<xacro:property name="model_name" value="IIT Coman w/ Softhand" />
+<xacro:property name="model_name" value="IIT COGIMON w/ Softhand" />
 <xacro:property name="model_version" value="0.1" />
 <!--

Commit message: Added left/right yaw hip

File: cogimon_urdf/urdf/cogimon_config.urdf.xacro (robot description, xacro)
@@ -10,3 +10,6 @@
 <xacro:property name="COGIMON_LEFT_LEG" value="true" />
 <xacro:property name="COGIMON_RIGHT_LEG" value="true" />
+<!-- ************SELECT FIXED BASE*************-->
+<!-- ******************************************-->
+<xacro:property name="COGIMON_FIXED_BASE" value="true" />
 </robot>

File: cogimon_urdf/urdf/cogimon_robot.urdf.xacro (robot description, xacro)
@@ -16,4 +16,5 @@
   <xacro:include filename="$(find cogimon_urdf)/urdf/gazebo/cogimon_materials.gazebo.xacro" />
   <xacro:include filename="$(find cogimon_urdf)/urdf/gazebo/force_torque.gazebo.xacro" /-->
+<xacro:if value="${COGIMON_FIXED_BASE}" >
   <link name="world"/>
    <joint name="fixed" type="fixed">
@@ -21,4 +22,5 @@
     <child link="base_link"/>
   </joint>
-  <origin xyz="0.0 0.0 0.521" rpy="0 0 0" />
+</xacro:if>
+<origin xyz="0.0 0.0 0.8" rpy="0 0 0" />
 </robot>

File: cogimon_urdf/urdf/parts/legs.urdf.xacro (robot description, xacro)
@@ -43,9 +43,29 @@
     </collision>
   </link>
+<link name ="RThighLowLeg">
+    <inertial>
+      <origin xyz="${-2.4777694e+01*mmTom} ${-5.3514533e+00*mmTom} ${-5.1363939e+01*mmTom}" rpy="0 0 0"/>
+      <mass value="2.3534104"/>
+      <inertia ixx="${1.0437839e+04*mm2Tom2}"  ixy="${1.2143782e+02*mm2Tom2}"  ixz="${-2.1459939e+03*mm2Tom2}" iyy="${1.1776825e+04*mm2Tom2}" iyz="${-3.0212597e+02*mm2Tom2}" izz="${7.4250380e+03*mm2Tom2}" />
+    </inertial>
+    <visual>
+      <origin xyz="0.0 0 0." rpy="0 0 0"/>
+      <material name="dark_grey"/>
+      <geometry name="LThighLowLeg_visual">
+        <mesh filename="package://cogimon_urdf/meshes/Leg2.STL" scale="${mmTom} ${-mmTom} ${mmTom}" />
+      </geometry>
+    </visual>
+    <collision>
+      <origin xyz="0.0 0 0" rpy="0 0 0"/>
+      <geometry name="LThighLowLeg_collision">
+        <mesh filename="package://cogimon_urdf/meshes/simple/Leg2.STL" scale="${mmTom} ${-mmTom} ${mmTom}" />
+      </geometry>
+    </collision>
+  </link>
 <!-- JOINTS -->
 <joint name="RHipLat" type="revolute">
     <parent link="Waist"/>
     <child link="RHipMot"/>
-    <origin xyz="${12.58*mmTom} ${-110.954508*mmTom} ${-52.922586*mmTom}" rpy="0 0 -0.0262" />
+    <origin xyz="${12.58*mmTom} ${-110.954508*mmTom} ${-52.922586*mmTom}" rpy="0 0 0" />
     <axis xyz="1 0 0" />
     <limit velocity="3.67" effort="176" lower="${-85.*toRad}" upper="${25.*toRad}" />
@@ -60,4 +80,12 @@
     <dynamics friction="0" damping="3.0"/>
   </joint>
+<joint name="RHipYaw" type="revolute">
+    <parent link="RThighUpLeg"/>
+    <child link="RThighLowLeg"/>
+    <origin xyz="${0.*mmTom} ${92.4945*mmTom} ${-239.0*mmTom}" rpy="0 0 0" />
+    <axis xyz="0 0 1" />
+    <limit velocity="13.6" effort="56" lower="${-75*toRad}" upper="${30*toRad}" />
+    <dynamics friction="0" damping="3.0"/>
+  </joint>
 </xacro:if>
 <xacro:if value="${COGIMON_LEFT_LEG}" >
@@ -103,9 +131,29 @@
     </collision>
   </link>
+<link name ="LThighLowLeg">
+    <inertial>
+      <origin xyz="${-2.4777694e+01*mmTom} ${5.3514533e+00*mmTom} ${-5.1363939e+01*mmTom}" rpy="0 0 0"/>
+      <mass value="2.3534104"/>
+      <inertia ixx="${1.0437839e+04*mm2Tom2}"  ixy="${-1.2143782e+02*mm2Tom2}"  ixz="${-2.1459939e+03*mm2Tom2}" iyy="${1.1776825e+04*mm2Tom2}" iyz="${3.0212597e+02*mm2Tom2}" izz="${7.4250380e+03*mm2Tom2}" />
+    </inertial>
+    <visual>
+      <origin xyz="0.0 0 0." rpy="0 0 0"/>
+      <material name="dark_grey"/>
+      <geometry name="LThighLowLeg_visual">
+        <mesh filename="package://cogimon_urdf/meshes/Leg2.STL" scale="${mmTom} ${mmTom} ${mmTom}" />
+      </geometry>
+    </visual>
+    <collision>
+      <origin xyz="0.0 0 0" rpy="0 0 0"/>
+      <geometry name="LThighLowLeg_collision">
+        <mesh filename="package://cogimon_urdf/meshes/simple/Leg2.STL" scale="${mmTom} ${mmTom} ${mmTom}" />
+      </geometry>
+    </collision>
+  </link>
 <!-- JOINTS -->
 <joint name="LHipLat" type="revolute">
     <parent link="Waist"/>
     <child link="LHipMot"/>
-    <origin xyz="${12.58*mmTom} ${110.954508*mmTom} ${-52.922586*mmTom}" rpy="0 0 0.0262" />
+    <origin xyz="${12.58*mmTom} ${110.954508*mmTom} ${-52.922586*mmTom}" rpy="0 0 0" />
     <axis xyz="1 0 0" />
     <limit velocity="3.67" effort="176" lower="${-25.*toRad}" upper="${85.*toRad}" />
@@ -120,28 +168,16 @@
     <dynamics friction="0" damping="3.0"/>
   </joint>
+<joint name="LHipYaw" type="revolute">
+    <parent link="LThighUpLeg"/>
+    <child link="LThighLowLeg"/>
+    <origin xyz="${0.*mmTom} ${-92.4945*mmTom} ${-239.0*mmTom}" rpy="0 0 0" />
+    <axis xyz="0 0 1" />
+    <limit velocity="13.6" effort="56" lower="${-30*toRad}" upper="${75*toRad}" />
+    <dynamics friction="0" damping="3.0"/>
+  </joint>
 </xacro:if>
 <!-- LINKS -->
 <!-- ********************RIGHT LEG******************** -->
 <!--
-  <link name ="RThighUpLeg">
-    <inertial>
-      <origin xyz="0.0012591632 -0.016896372 -0.058903336" rpy="0 0 0"/>
-      <mass value="${wcf*1.0246101}"/>
-      <inertia ixx="${wcf*9.165719E-4}"  ixy="${wcf*-1.4449904E-6}"  ixz="${wcf*-1.6685011E-5}" iyy="${wcf*0.00104849584}" iyz="${wcf*2.5492874E-5}" izz="${wcf*6.8637197E-4}" />
-    </inertial>
-    <visual>
-      <origin xyz="0.0 0.0726 -0.52" rpy="0 0 ${PI}"/>
-      <material name="dark_grey"/>
-      <geometry name="RThighUpLeg_visual">
-        <mesh filename="package://cogimon_urdf/meshes/Leg1.STL" scale="${SF} ${SF} ${SF}" />
-      </geometry>
-    </visual>
-    <collision>
-      <origin xyz="0.0 0.0726 -0.52" rpy="0 0 ${PI}"/>
-      <geometry name="RThighUpLeg_collision">
-        <mesh filename="package://cogimon_urdf/meshes/simple/Leg1.STL" scale="${SF} ${SF} ${SF}" />
-      </geometry>
-    </collision>
-  </link>
   <link name ="RThighLowLeg">
     <inertial>
@@ -251,24 +287,4 @@
 <!-- ********************LEFT LEG******************** -->
 <!--
-  <link name ="LThighLowLeg">
-    <inertial>
-      <origin xyz="9.8720058E-4 -6.7037262E-4 -0.075716843" rpy="0 0 0"/>
-      <mass value="${wcf*1.7001134}"/>
-      <inertia ixx="${wcf*0.0038979546}"  ixy="${wcf*-1.7802399E-6}"  ixz="${wcf*2.6403262E-5}" iyy="${wcf*0.0039360845}" iyz="${wcf*-4.5227110E-5}" izz="${wcf*9.0218711E-4}" />
-    </inertial>
-    <visual>
-      <origin xyz="0.0 -0.0726 -0.4176" rpy="0 0 ${PI}"/>
-      <material name="dark_grey"/>
-      <geometry name="LThighLowLeg_visual">
-        <mesh filename="package://cogimon_urdf/meshes/Leg2.STL" scale="${SF} -${SF} ${SF}" />
-      </geometry>
-    </visual>
-    <collision>
-      <origin xyz="0.0 -0.0726 -0.4176" rpy="0 0 ${PI}"/>
-      <geometry name="LThighLowLeg_collision">
-        <mesh filename="package://cogimon_urdf/meshes/simple/Leg2.STL" scale="${SF} -${SF} ${SF}" />
-      </geometry>
-    </collision>
-  </link>
   <link name ="LLowLeg">
     <inertial>

Commit message: Fixed inertias in leg links. The previous inertias were wrong since we were considering directly the rotor inertia together with the (next) link without considering the transmission. To compute the new inertias we first subtracted rotor inertia and then we added the rotor inertia times reduction squared: I_new = (I_old - I_rotor)+I_rotor*N^2

File: cogimon_urdf/urdf/cogimon_config.urdf.xacro (robot description, xacro)
@@ -12,4 +12,4 @@
 <!-- ************SELECT FIXED BASE*************-->
 <!-- ******************************************-->
-<xacro:property name="COGIMON_FIXED_BASE" value="true" />
+<xacro:property name="COGIMON_FIXED_BASE" value="false" />
 </robot>

File: cogimon_urdf/urdf/parts/legs.urdf.xacro (robot description, xacro)
@@ -7,5 +7,5 @@
       <origin xyz="${4.7902756e+00*mmTom} ${1.5595700e+01*mmTom} ${-6.0925801e+01*mmTom}" rpy="0 0 0"/>
       <mass value="1.6995409"/>
-      <inertia ixx="${7.7713640e+03*mm2Tom2}"  ixy="${2.5414978e+02*mm2Tom2}"  ixz="${-1.1602420e+03*mm2Tom2}" iyy="${8.1906401e+03*mm2Tom2}" iyz="${1.2050460e+03*mm2Tom2}" izz="${3.7083468e+03*mm2Tom2}" />
+      <inertia ixx="${2.2053e+06*mm2Tom2}"  ixy="${-0.0066e+06*mm2Tom2}"  ixz="${0.0015e+06*mm2Tom2}" iyy="${2.7733e+06*mm2Tom2}" iyz="${0.0125e+06*mm2Tom2}" izz="${2.7756e+06*mm2Tom2}" />
     </inertial>
     <visual>
@@ -27,5 +27,5 @@
       <origin xyz="${2.9898120e-01*mmTom} ${6.5748642e+01*mmTom} ${-8.8443666e+01*mmTom}" rpy="0 0 0"/>
       <mass value="1.9691802"/>
-      <inertia ixx="${1.6200713e+04*mm2Tom2}"  ixy="${1.9336329e+01*mm2Tom2}"  ixz="${-3.8620029e+01*mm2Tom2}" iyy="${1.4426424e+04*mm2Tom2}" iyz="${3.5985350e+03*mm2Tom2}" izz="${4.8264937e+03*mm2Tom2}" />
+      <inertia ixx="${2.7765e+06*mm2Tom2}"  ixy="${0.0058e+06*mm2Tom2}"  ixz="${-0.0085e+06*mm2Tom2}" iyy="${2.2120e+06*mm2Tom2}" iyz="${0.0082e+06*mm2Tom2}" izz="${2.7816e+06*mm2Tom2}" />
     </inertial>
     <visual>
@@ -47,5 +47,5 @@
       <origin xyz="${-2.4777694e+01*mmTom} ${-5.3514533e+00*mmTom} ${-5.1363939e+01*mmTom}" rpy="0 0 0"/>
       <mass value="2.3534104"/>
-      <inertia ixx="${1.0437839e+04*mm2Tom2}"  ixy="${1.2143782e+02*mm2Tom2}"  ixz="${-2.1459939e+03*mm2Tom2}" iyy="${1.1776825e+04*mm2Tom2}" iyz="${-3.0212597e+02*mm2Tom2}" izz="${7.4250380e+03*mm2Tom2}" />
+      <inertia ixx="${1.5350e+05*mm2Tom2}"  ixy="${0.0012e+05*mm2Tom2}"  ixz="${-0.0215e+05*mm2Tom2}" iyy="${1.5484e+05*mm2Tom2}" iyz="${-0.0030e+05*mm2Tom2}" izz="${0.9917e+05*mm2Tom2}" />
     </inertial>
     <visual>
@@ -95,5 +95,5 @@
       <origin xyz="${4.7902756e+00*mmTom} ${-1.5595700e+01*mmTom} ${-6.0925801e+01*mmTom}" rpy="0 0 0"/>
       <mass value="1.6995409"/>
-      <inertia ixx="${7.7713640e+03*mm2Tom2}"  ixy="${-2.5414978e+02*mm2Tom2}"  ixz="${-1.1602420e+03*mm2Tom2}" iyy="${8.1906401e+03*mm2Tom2}" iyz="${-1.2050460e+03*mm2Tom2}" izz="${3.7083468e+03*mm2Tom2}" />
+      <inertia ixx="${2.2053e+06*mm2Tom2}"  ixy="${0.0066e+06*mm2Tom2}"  ixz="${0.0015e+06*mm2Tom2}" iyy="${2.7733e+06*mm2Tom2}" iyz="${-0.0125e+06*mm2Tom2}" izz="${2.7756e+06*mm2Tom2}" />
     </inertial>
     <visual>
@@ -115,5 +115,5 @@
       <origin xyz="${2.9898120e-01*mmTom} ${-6.5748642e+01*mmTom} ${-8.8443666e+01*mmTom}" rpy="0 0 0"/>
       <mass value="1.9691802"/>
-      <inertia ixx="${1.6200713e+04*mm2Tom2}"  ixy="${-1.9336329e+01*mm2Tom2}"  ixz="${-3.8620029e+01*mm2Tom2}" iyy="${1.4426424e+04*mm2Tom2}" iyz="${-3.5985350e+03*mm2Tom2}" izz="${4.8264937e+03*mm2Tom2}" />
+      <inertia ixx="${2.7765e+06*mm2Tom2}"  ixy="${-0.0058e+06*mm2Tom2}"  ixz="${-0.0085e+06*mm2Tom2}" iyy="${2.2120e+06*mm2Tom2}" iyz="${-0.0082e+06*mm2Tom2}" izz="${2.7816e+06*mm2Tom2}" />
     </inertial>
     <visual>
@@ -135,5 +135,5 @@
       <origin xyz="${-2.4777694e+01*mmTom} ${5.3514533e+00*mmTom} ${-5.1363939e+01*mmTom}" rpy="0 0 0"/>
       <mass value="2.3534104"/>
-      <inertia ixx="${1.0437839e+04*mm2Tom2}"  ixy="${-1.2143782e+02*mm2Tom2}"  ixz="${-2.1459939e+03*mm2Tom2}" iyy="${1.1776825e+04*mm2Tom2}" iyz="${3.0212597e+02*mm2Tom2}" izz="${7.4250380e+03*mm2Tom2}" />
+      <inertia ixx="${1.5350e+05*mm2Tom2}"  ixy="${-0.0012e+05*mm2Tom2}"  ixz="${-0.0215e+05*mm2Tom2}" iyy="${1.5484e+05*mm2Tom2}" iyz="${0.0030e+05*mm2Tom2}" izz="${0.9917e+05*mm2Tom2}" />
     </inertial>
     <visual>

Commit message: update

File: cogimon_urdf/urdf/cogimon_config.urdf.xacro (robot description, xacro)
@@ -8,5 +8,5 @@
 <xacro:property name="COGIMON_LEFT_ARM" value="false" />
 <xacro:property name="COGIMON_RIGHT_ARM" value="false" />
-<xacro:property name="COGIMON_LEFT_LEG" value="true" />
+<xacro:property name="COGIMON_LEFT_LEG" value="false" />
 <xacro:property name="COGIMON_RIGHT_LEG" value="true" />
 <!-- ************SELECT FIXED BASE*************-->

File: cogimon_urdf/urdf/parts/legs.urdf.xacro (robot description, xacro)
@@ -23,4 +23,5 @@
     </collision>
 </link>
+<!--
 <link name ="RThighUpLeg">
     <inertial>
@@ -63,4 +64,5 @@
     </collision>
   </link>
+-->
 <!-- JOINTS -->
 <joint name="RHipLat" type="revolute">
@@ -72,4 +74,5 @@
     <dynamics friction="0" damping="3.0"/>
   </joint>
+<!--
 <joint name="RHipSag" type="revolute">
     <parent link="RHipMot"/>
@@ -88,4 +91,5 @@
     <dynamics friction="0" damping="3.0"/>
   </joint>
+-->
 </xacro:if>
 <xacro:if value="${COGIMON_LEFT_LEG}" >

Commit message: Added last joint and link. FInished leg

File: cogimon_urdf/urdf/cogimon_config.urdf.xacro (robot description, xacro)
@@ -13,7 +13,9 @@
 <!-- ******************************************-->
 <xacro:property name="COGIMON_FLOATING_BASE" value="true" />
+<!-- ************FIXED BASE*************-->
+<!-- ******************************************-->
+<xacro:property name="COGIMON_FIXED_BASE" value="false" />
 <!-- ************XBOT FRAMEWORK*************-->
 <!-- *************************************-->
--->
 <xacro:property name="COGIMON_XBOT" value="false" />
 </robot>

File: cogimon_urdf/urdf/cogimon_robot.urdf.xacro (robot description, xacro)
@@ -14,4 +14,5 @@
   <xacro:include filename="$(find cogimon_urdf)/urdf/gazebo/cogimon_materials.gazebo.xacro" />
   <!--xacro:include filename="$(find cogimon_urdf)/urdf/gazebo/force_torque.gazebo.xacro" /-->
+<xacro:if value="${COGIMON_FIXED_BASE}" >
   <link name="world"/>
    <joint name="fixed" type="fixed">
@@ -19,4 +20,5 @@
     <child link="base_link"/>
   </joint>
-<origin xyz="0.0 0.0 1.0" rpy="0 0 0" />
+</xacro:if>
+<origin xyz="0.0 0.0 0.97" rpy="0 0 0" />
 </robot>

File: cogimon_urdf/urdf/gazebo/cogimon_materials.gazebo.xacro (robot description, xacro)
@@ -20,4 +20,7 @@
   <material>Gazebo/DarkGrey</material>
 </gazebo>
+<gazebo reference="RFoot">
+  <material>Gazebo/DarkGrey</material>
+</gazebo>
 </xacro:if>
 <xacro:if value="${COGIMON_LEFT_LEG}" >
@@ -37,4 +40,7 @@
   <material>Gazebo/DarkGrey</material>
 </gazebo>
+<gazebo reference="LFoot">
+  <material>Gazebo/DarkGrey</material>
+</gazebo>
 </xacro:if>
 </robot>

File: cogimon_urdf/urdf/parts/legs.urdf.xacro (robot description, xacro)
@@ -101,4 +101,24 @@
         <mesh filename="package://cogimon_urdf/meshes/simple/AnklePitch.stl" scale="${mmTom} ${mmTom} ${mmTom}" />
       </geometry>
+    </collision>
+</link>
+<link name ="LFoot">
+    <inertial>
+      <origin xyz="${-8.6960323e+00*mmTom} ${-6.6741928e-02*mmTom} ${-4.1675435e+01*mmTom}" rpy="0 0 0"/>
+      <mass value="1.7819594e+00"/>
+      <inertia ixx="${1.9182691e+03*mm2Tom2}"  ixy="${5.7926583e+00*mm2Tom2}"  ixz="${3.2836542e+02*mm2Tom2}" iyy="${5.3518735e+03*mm2Tom2}" iyz="${-3.0518008e+00*mm2Tom2}" izz="${ 6.4063918e+03*mm2Tom2}" />
+    </inertial>
+    <visual>
+      <origin xyz="0 0 0" rpy="0 0 0"/>
+      <geometry name="LFoot_visual">
+        <mesh filename="package://cogimon_urdf/meshes/Foot.stl" scale="${mmTom} ${mmTom} ${mmTom}" />
+      </geometry>
+      <material name="dark_grey"/>
+    </visual>
+    <collision>
+      <origin xyz="0.0 0.0 -0.046" rpy="0 0 0"/>
+       <geometry>
+        <box size="0.21 0.11 0.015" />
+       </geometry>
     </collision>
 </link>
@@ -144,4 +164,12 @@
     <dynamics friction="0" damping="0.1"/>
 </joint>
+<joint name="LAnkleRoll" type="revolute">
+    <parent link="LFootmot"/>
+    <child link="LFoot"/>
+    <origin xyz="0 0 0" rpy="0 0 0" />
+    <axis xyz="1 0 0" />
+    <limit velocity="3.67" effort="176" lower="${-90.*toRad}" upper="${90.*toRad}" />
+    <dynamics friction="0" damping="3.0"/>
+</joint>
 </xacro:if>
 <xacro:if value="${COGIMON_RIGHT_LEG}" >
@@ -245,4 +273,24 @@
         <mesh filename="package://cogimon_urdf/meshes/simple/AnklePitch.stl" scale="${mmTom} ${mmTom} ${mmTom}" />
       </geometry>
+    </collision>
+</link>
+<link name ="RFoot">
+    <inertial>
+      <origin xyz="${-8.6960323e+00*mmTom} ${-6.6741928e-02*mmTom} ${-4.1675435e+01*mmTom}" rpy="0 0 0"/>
+      <mass value="1.7819594e+00"/>
+      <inertia ixx="${1.9182691e+03*mm2Tom2}"  ixy="${5.7926583e+00*mm2Tom2}"  ixz="${3.2836542e+02*mm2Tom2}" iyy="${5.3518735e+03*mm2Tom2}" iyz="${-3.0518008e+00*mm2Tom2}" izz="${ 6.4063918e+03*mm2Tom2}" />
+    </inertial>
+    <visual>
+      <origin xyz="0 0 0" rpy="0 0 0"/>
+      <geometry name="RFoot_visual">
+        <mesh filename="package://cogimon_urdf/meshes/Foot.stl" scale="${mmTom} ${mmTom} ${mmTom}" />
+      </geometry>
+      <material name="dark_grey"/>
+    </visual>
+    <collision>
+      <origin xyz="0.0 0.0 -0.046" rpy="0 0 0"/>
+       <geometry>
+        <box size="0.21 0.11 0.015" />
+       </geometry>
     </collision>
 </link>
@@ -288,4 +336,12 @@
     <dynamics friction="0" damping="0.1"/>
 </joint>
+<joint name="RAnkleRoll" type="revolute">
+    <parent link="RFootmot"/>
+    <child link="RFoot"/>
+    <origin xyz="0 0 0" rpy="0 0 0" />
+    <axis xyz="1 0 0" />
+    <limit velocity="3.67" effort="176" lower="${-90.*toRad}" upper="${90.*toRad}" />
+    <dynamics friction="0" damping="3.0"/>
+</joint>
 </xacro:if>
 </robot>

Commit message: Added "Pennacchio"

File: cogimon_urdf/urdf/cogimon_config.urdf.xacro (robot description, xacro)
@@ -10,4 +10,12 @@
 <xacro:property name="COGIMON_LEFT_LEG" value="true" />
 <xacro:property name="COGIMON_RIGHT_LEG" value="true" />
+<!-- ************COGIMON_PENNACCHIO*******-->
+<!--
+     This will add a fake torso link after the first
+     torso joint (roll). If this is true, arms has
+     to be false and torso has to be true.
+-->
+<!-- *************************************-->
+<xacro:property name="COGIMON_PENNACCHIO" value="true" />
 <!-- ************FLOATING BASE*************-->
 <!-- ******************************************-->

File: cogimon_urdf/urdf/gazebo/cogimon.gazebo.xacro (robot description, xacro)
@@ -78,5 +78,5 @@
 </xacro:if>
 <xacro:if value="${COGIMON_TORSO}">
-   <gazebo reference="DWL">
+   <gazebo reference="WaistLat">
     <implicitSpringDamper>1</implicitSpringDamper>
     <provideFeedback>true</provideFeedback>

File: cogimon_urdf/urdf/gazebo/cogimon_materials.gazebo.xacro (robot description, xacro)
@@ -48,4 +48,9 @@
   <material>Gazebo/DarkGrey</material>
 </gazebo>
+<xacro:if value="${COGIMON_TORSO}">
+<gazebo reference="pennacchio">
+  <material>Gazebo/DarkGrey</material>
+</gazebo>
+</xacro:if>
 </xacro:if>
 </robot>

File: cogimon_urdf/urdf/parts/torso.urdf.xacro (robot description, xacro)
@@ -23,4 +23,26 @@
     </collision>
 </link>
+<xacro:if value="${COGIMON_PENNACCHIO}" >
+<link name ="pennacchio">
+    <inertial>
+      <origin xyz="${-3.4081174e-03*mmTom} ${-3.4081174e-03*mmTom} ${1.7247336e+02*mmTom} " rpy="0 0 0"/>
+      <mass value="2.1651618"/>
+      <inertia ixx="${4.5713534e+04*mm2Tom2}"  ixy="${1.9747985e-02*mm2Tom2}"  ixz="${5.9794097e-01*mm2Tom2}" iyy="${4.5712755e+04*mm2Tom2}" iyz="${-2.6722676e-01*mm2Tom2}" izz="${6.0311791e+02*mm2Tom2}" />
+    </inertial>
+    <visual>
+      <origin xyz="0.0 0.0 0.0" rpy="0 0 0"/>
+      <geometry name="pennacchio_visual">
+        <mesh filename="package://cogimon_urdf/meshes/Pennacchio.stl" scale="${mmTom} ${mmTom} ${mmTom}" />
+      </geometry>
+      <material name="dark_grey"/>
+    </visual>
+    <collision>
+      <origin xyz="0.0 0.0 0.0" rpy="0 0 0"/>
+      <geometry name="pennacchio_collision">
+        <mesh filename="package://cogimon_urdf/meshes/simple/Pennacchio.stl" scale="${mmTom} ${mmTom} ${mmTom}" />
+      </geometry>
+    </collision>
+</link>
+</xacro:if>
 <!-- JOINTS -->
 <joint name="WaistLat" type="revolute">
@@ -32,4 +54,11 @@
     <dynamics friction="0" damping="3.0"/>
 </joint>
+<xacro:if value="${COGIMON_PENNACCHIO}" >
+<joint name="pennacchio_frame" type="fixed">
+    <parent link="DWL"/>
+    <child link="pennacchio"/>
+    <origin xyz="${-54.0957*mmTom} 0.0 ${66.5*mmTom}" rpy="0 0 0" />
+</joint>
+</xacro:if>
 </xacro:if>
 </robot>
