Commit message: Added possibility to select new or old feet. Still WIP

File: cogimon_urdf/urdf/cogimon_config.urdf.xacro (robot description, xacro)
@@ -11,4 +11,7 @@
 <xacro:property name="COGIMON_LEFT_LEG" value="true" />
 <xacro:property name="COGIMON_RIGHT_LEG" value="true" />
+<!-- ************NEW FEET*************-->
+<!-- *************************************-->
+<xacro:property name="COGIMON_FEET_2" value="false" />
 <!-- ************COGIMON_LASER_FIXED*******-->
 <!--

File: cogimon_urdf/urdf/config/cogimon_hardware.urdf.xacro (robot description, xacro)
@@ -11,4 +11,7 @@
 <xacro:property name="COGIMON_LEFT_LEG" value="true" />
 <xacro:property name="COGIMON_RIGHT_LEG" value="true" />
+<!-- ************NEW FEET*************-->
+<!-- *************************************-->
+<xacro:property name="COGIMON_FEET_2" value="false" />
 <!-- ************COGIMON_LASER_FIXED*******-->
 <!--

File: cogimon_urdf/urdf/config/cogimon_pennacchio.urdf.xacro (robot description, xacro)
@@ -11,4 +11,7 @@
 <xacro:property name="COGIMON_LEFT_LEG" value="true" />
 <xacro:property name="COGIMON_RIGHT_LEG" value="true" />
+<!-- ************NEW FEET*************-->
+<!-- *************************************-->
+<xacro:property name="COGIMON_FEET_2" value="false" />
 <!-- ************COGIMON_LASER_FIXED*******-->
 <!--

File: cogimon_urdf/urdf/parts/legs.urdf.xacro (robot description, xacro)
@@ -103,14 +103,15 @@
     </collision>
 </link>
+<xacro:if value="${COGIMON_FEET_2}" >
 <link name ="LFoot">
     <inertial>
-      <origin xyz="${-8.6960323e+00*mmTom} ${-6.6741928e-02*mmTom} ${-4.1675435e+01*mmTom}" rpy="0 0 0"/>
-      <mass value="1.7819594e+00"/>
-      <inertia ixx="${1.9182691e+03*mm2Tom2}"  ixy="${5.7926583e+00*mm2Tom2}"  ixz="${3.2836542e+02*mm2Tom2}" iyy="${5.3518735e+03*mm2Tom2}" iyz="${-3.0518008e+00*mm2Tom2}" izz="${ 6.4063918e+03*mm2Tom2}" />
+      <origin xyz="${-7.7094563*mmTom} ${-6.5520742e-02*mmTom} ${-4.3453782e+01*mmTom}" rpy="0 0 0"/>
+      <mass value="2.0663292"/>
+      <inertia ixx="${2.6932116e+03*mm2Tom2}"  ixy="${4.2852647e+00*mm2Tom2}"  ixz="${3.7001167e+02*mm2Tom2}" iyy="${7.1293752e+03*mm2Tom2}" iyz="${-2.5956611*mm2Tom2}" izz="${8.6807822e+03*mm2Tom2}" />
     </inertial>
     <visual>
       <origin xyz="0 0 0" rpy="0 0 0"/>
       <geometry name="LFoot_visual">
-        <mesh filename="package://cogimon_urdf/meshes/Foot.stl" scale="${mmTom} ${mmTom} ${mmTom}" />
+        <mesh filename="package://cogimon_urdf/meshes/Foot2.stl" scale="${mmTom} ${mmTom} ${mmTom}" />
       </geometry>
       <material name="dark_grey"/>
@@ -123,4 +124,27 @@
     </collision>
 </link>
+</xacro:if>
+<xacro:unless value="${COGIMON_FEET_2}" >
+<link name ="LFoot">
+    <inertial>
+      <origin xyz="${-8.6960323e+00*mmTom} ${-6.6741928e-02*mmTom} ${-4.1675435e+01*mmTom}" rpy="0 0 0"/>
+      <mass value="1.7819594e+00"/>
+      <inertia ixx="${1.9182691e+03*mm2Tom2}"  ixy="${5.7926583e+00*mm2Tom2}"  ixz="${3.2836542e+02*mm2Tom2}" iyy="${5.3518735e+03*mm2Tom2}" iyz="${-3.0518008e+00*mm2Tom2}" izz="${ 6.4063918e+03*mm2Tom2}" />
+    </inertial>
+    <visual>
+      <origin xyz="0 0 0" rpy="0 0 0"/>
+      <geometry name="LFoot_visual">
+        <mesh filename="package://cogimon_urdf/meshes/Foot.stl" scale="${mmTom} ${mmTom} ${mmTom}" />
+      </geometry>
+      <material name="dark_grey"/>
+    </visual>
+    <collision>
+      <origin xyz="0.0 0.0 -0.046" rpy="0 0 0"/>
+       <geometry>
+        <box size="0.21 0.11 0.015" />
+       </geometry>
+    </collision>
+</link>
+</xacro:unless>
 <!-- JOINTS -->
 <joint name="LHipLat" type="revolute">
@@ -276,14 +300,15 @@
     </collision>
 </link>
+<xacro:if value="${COGIMON_FEET_2}" >
 <link name ="RFoot">
     <inertial>
-      <origin xyz="${-8.6960323e+00*mmTom} ${-6.6741928e-02*mmTom} ${-4.1675435e+01*mmTom}" rpy="0 0 0"/>
-      <mass value="1.7819594e+00"/>
-      <inertia ixx="${1.9182691e+03*mm2Tom2}"  ixy="${5.7926583e+00*mm2Tom2}"  ixz="${3.2836542e+02*mm2Tom2}" iyy="${5.3518735e+03*mm2Tom2}" iyz="${-3.0518008e+00*mm2Tom2}" izz="${ 6.4063918e+03*mm2Tom2}" />
-    </inertial>
-    <visual>
-      <origin xyz="0 0 0" rpy="0 0 0"/>
-      <geometry name="RFoot_visual">
-        <mesh filename="package://cogimon_urdf/meshes/Foot.stl" scale="${mmTom} ${mmTom} ${mmTom}" />
+      <origin xyz="${-7.7094563*mmTom} ${-6.5520742e-02*mmTom} ${-4.3453782e+01*mmTom}" rpy="0 0 0"/>
+      <mass value="2.0663292"/>
+      <inertia ixx="${2.6932116e+03*mm2Tom2}"  ixy="${4.2852647e+00*mm2Tom2}"  ixz="${3.7001167e+02*mm2Tom2}" iyy="${7.1293752e+03*mm2Tom2}" iyz="${-2.5956611*mm2Tom2}" izz="${8.6807822e+03*mm2Tom2}" />
+    </inertial>
+    <visual>
+      <origin xyz="0 0 0" rpy="0 0 0"/>
+      <geometry name="LFoot_visual">
+        <mesh filename="package://cogimon_urdf/meshes/Foot2.stl" scale="${mmTom} ${mmTom} ${mmTom}" />
       </geometry>
       <material name="dark_grey"/>
@@ -296,4 +321,27 @@
     </collision>
 </link>
+</xacro:if>
+<xacro:unless value="${COGIMON_FEET_2}" >
+<link name ="RFoot">
+    <inertial>
+      <origin xyz="${-8.6960323e+00*mmTom} ${-6.6741928e-02*mmTom} ${-4.1675435e+01*mmTom}" rpy="0 0 0"/>
+      <mass value="1.7819594e+00"/>
+      <inertia ixx="${1.9182691e+03*mm2Tom2}"  ixy="${5.7926583e+00*mm2Tom2}"  ixz="${3.2836542e+02*mm2Tom2}" iyy="${5.3518735e+03*mm2Tom2}" iyz="${-3.0518008e+00*mm2Tom2}" izz="${ 6.4063918e+03*mm2Tom2}" />
+    </inertial>
+    <visual>
+      <origin xyz="0 0 0" rpy="0 0 0"/>
+      <geometry name="RFoot_visual">
+        <mesh filename="package://cogimon_urdf/meshes/Foot.stl" scale="${mmTom} ${mmTom} ${mmTom}" />
+      </geometry>
+      <material name="dark_grey"/>
+    </visual>
+    <collision>
+      <origin xyz="0.0 0.0 -0.046" rpy="0 0 0"/>
+       <geometry>
+        <box size="0.21 0.11 0.015" />
+       </geometry>
+    </collision>
+</link>
+</xacro:unless>
 <!-- JOINTS -->
 <joint name="RHipLat" type="revolute">

Commit message: Added new feet

File: cogimon_urdf/urdf/cogimon_config.urdf.xacro (robot description, xacro)
@@ -13,5 +13,5 @@
 <!-- ************NEW FEET*************-->
 <!-- *************************************-->
-<xacro:property name="COGIMON_FEET_2" value="false" />
+<xacro:property name="COGIMON_FEET_2" value="true" />
 <!-- ************COGIMON_LASER_FIXED*******-->
 <!--

File: cogimon_urdf/urdf/config/cogimon_hardware.urdf.xacro (robot description, xacro)
@@ -13,5 +13,5 @@
 <!-- ************NEW FEET*************-->
 <!-- *************************************-->
-<xacro:property name="COGIMON_FEET_2" value="false" />
+<xacro:property name="COGIMON_FEET_2" value="true" />
 <!-- ************COGIMON_LASER_FIXED*******-->
 <!--

File: cogimon_urdf/urdf/config/cogimon_pennacchio.urdf.xacro (robot description, xacro)
@@ -13,5 +13,5 @@
 <!-- ************NEW FEET*************-->
 <!-- *************************************-->
-<xacro:property name="COGIMON_FEET_2" value="false" />
+<xacro:property name="COGIMON_FEET_2" value="true" />
 <!-- ************COGIMON_LASER_FIXED*******-->
 <!--

File: cogimon_urdf/urdf/parts/feet_reference_frames.urdf.xacro (robot description, xacro)
@@ -32,5 +32,10 @@
 </joint>
 <joint name="l_sole_joint" type="fixed">
-       <origin xyz="0 0 ${-54.*mmTom}" rpy="0 0 0" />
+        <xacro:if value="${COGIMON_FEET_2}">
+          <origin xyz="0 0 ${-69.*mmTom}" rpy="0 0 0" />
+        </xacro:if>
+        <xacro:unless value="${COGIMON_FEET_2}">
+          <origin xyz="0 0 ${-54.*mmTom}" rpy="0 0 0" />
+        </xacro:unless>
 	<parent link="l_ankle"/>
 	<child link="l_sole"/>
@@ -65,5 +70,10 @@
 </joint>
 <joint name="r_sole_joint" type="fixed">
-       <origin xyz="0 0 ${-54.*mmTom}" rpy="0 0 0" />
+        <xacro:if value="${COGIMON_FEET_2}">
+          <origin xyz="0 0 ${-69.*mmTom}" rpy="0 0 0" />
+        </xacro:if>
+        <xacro:unless value="${COGIMON_FEET_2}">
+          <origin xyz="0 0 ${-54.*mmTom}" rpy="0 0 0" />
+        </xacro:unless>
 	<parent link="r_ankle"/>
 	<child link="r_sole"/>

Commit message: default is xbotcore in config

File: cogimon_urdf/urdf/cogimon_config.urdf.xacro (robot description, xacro)
@@ -38,7 +38,7 @@
 <!-- ************XBOT-GAZEBO FRAMEWORK*************-->
 <!-- *************************************-->
-<xacro:property name="COGIMON_XBOT_GAZEBO" value="false" />
+<xacro:property name="COGIMON_XBOT_GAZEBO" value="true" />
 <!-- ************OROCOS-GAZEBO FRAMEWORK*************-->
 <!-- *************************************-->
-<xacro:property name="COGIMON_OROCOS_GAZEBO" value="true" />
+<xacro:property name="COGIMON_OROCOS_GAZEBO" value="false" />
 </robot>

Commit message: added arms

File: cogimon_urdf/urdf/cogimon_config.urdf.xacro (robot description, xacro)
@@ -8,6 +8,6 @@
 <xacro:property name="COGIMON_HEAD" value="true" />
 <xacro:property name="COGIMON_TORSO" value="true" />
-<xacro:property name="COGIMON_LEFT_ARM" value="false" />
-<xacro:property name="COGIMON_RIGHT_ARM" value="false" />
+<xacro:property name="COGIMON_LEFT_ARM" value="true" />
+<xacro:property name="COGIMON_RIGHT_ARM" value="true" />
 <xacro:property name="COGIMON_LEFT_LEG" value="true" />
 <xacro:property name="COGIMON_RIGHT_LEG" value="true" />
