Commit message: Added meshes for the neck. Added possibility to add head.

File: cogimon_urdf/urdf/config/cogimon.urdf.xacro (robot description, xacro)
@@ -5,4 +5,5 @@
 <!-- ************SELECT PARTS*************-->
 <!-- *************************************-->
+<xacro:property name="COGIMON_HEAD" value="false" />
 <xacro:property name="COGIMON_TORSO" value="true" />
 <xacro:property name="COGIMON_LEFT_ARM" value="true" />

File: cogimon_urdf/urdf/config/cogimon_hardware.urdf.xacro (robot description, xacro)
@@ -1,12 +1,12 @@
 <?xml version="1.0"?>
 <robot xmlns:xacro="http://ros.org/wiki/xacro" name="COGIMON">
-<xacro:property name="model_name" value="IIT COGIMON PENNACCHIO" />
+<xacro:property name="model_name" value="IIT COGIMON" />
 <xacro:property name="model_version" value="0.1" />
 <!-- ************SELECT PARTS*************-->
 <!-- *************************************-->
-<xacro:property name="COGIMON_HEAD" value="false" />
+<xacro:property name="COGIMON_HEAD" value="true" />
 <xacro:property name="COGIMON_TORSO" value="true" />
-<xacro:property name="COGIMON_LEFT_ARM" value="false" />
-<xacro:property name="COGIMON_RIGHT_ARM" value="false" />
+<xacro:property name="COGIMON_LEFT_ARM" value="true" />
+<xacro:property name="COGIMON_RIGHT_ARM" value="true" />
 <xacro:property name="COGIMON_LEFT_LEG" value="true" />
 <xacro:property name="COGIMON_RIGHT_LEG" value="true" />
@@ -18,5 +18,5 @@
 -->
 <!-- *************************************-->
-<xacro:property name="COGIMON_PENNACCHIO" value="true" />
+<xacro:property name="COGIMON_PENNACCHIO" value="false" />
 <!-- ************FLOATING BASE*************-->
 <!-- ******************************************-->
