Commit message: switched to false values for COGIMON_OROCOS_GAZEBO

File: cogimon_urdf/urdf/config/cogimon_hardware.urdf.xacro (robot description, xacro)
@@ -38,7 +38,7 @@
 <!-- ************XBOT-GAZEBO FRAMEWORK*************-->
 <!-- *************************************-->
-<xacro:property name="COGIMON_XBOT_GAZEBO" value="false" />
+<xacro:property name="COGIMON_XBOT_GAZEBO" value="true" />
 <!-- ************OROCOS-GAZEBO FRAMEWORK*************-->
 <!-- *************************************-->
-<xacro:property name="COGIMON_OROCOS_GAZEBO" value="true" />
+<xacro:property name="COGIMON_OROCOS_GAZEBO" value="false" />
 </robot>

File: cogimon_urdf/urdf/config/cogimon_pennacchio.urdf.xacro (robot description, xacro)
@@ -38,7 +38,7 @@
 <!-- ************XBOT-GAZEBO FRAMEWORK*************-->
 <!-- *************************************-->
-<xacro:property name="COGIMON_XBOT_GAZEBO" value="false" />
+<xacro:property name="COGIMON_XBOT_GAZEBO" value="true" />
 <!-- ************OROCOS-GAZEBO FRAMEWORK*************-->
 <!-- *************************************-->
-<xacro:property name="COGIMON_OROCOS_GAZEBO" value="true" />
+<xacro:property name="COGIMON_OROCOS_GAZEBO" value="false" />
 </robot>
