Commit message: Changed orientation of imu link to be compatible with the one of the simulator. Changed srdf

File: cogimon_srdf/srdf/cogimon.srdf.xacro (robot description, xacro)
@@ -15,6 +15,5 @@
     </group>
     <group name="imu_sensors">
-    <!-- NEAREST JOINT TO IMU -->
-        <joint name="WaistSag"/>
+        <link name="imu_link"/>
     </group>
     <xacro:if value="${GAZEBO_COGIMON_USES_FOREARMS}">

File: cogimon_urdf/urdf/sensors/imu.urdf.xacro (robot description, xacro)
@@ -18,5 +18,6 @@
     <parent link="Waist"/>
     <child link="imu_link"/>
-    <origin xyz="-0.072 -0.0068 0.044" rpy="0 ${PI} 0"/>
+    <!--origin xyz="-0.072 -0.0068 0.044" rpy="0 ${PI} 0"/-->
+    <origin xyz="-0.072 -0.0068 0.044" rpy="0 0 0"/>
 </joint>
 </robot>

Commit message: Started working on real cogimon. Added Waist

File: cogimon_srdf/srdf/cogimon.srdf.xacro (robot description, xacro)
@@ -18,33 +18,16 @@
         <link name="imu_link"/>
     </group>
-    <xacro:if value="${GAZEBO_COGIMON_USES_FOREARMS}">
-        <group name="left_arm">
-            <chain base_link="DWYTorso" tip_link="l_wrist"/>
-        </group>
-        <group name="right_arm">
-            <chain base_link="DWYTorso" tip_link="r_wrist"/>
-        </group>
-        <group name="force_torque_sensors">
-            <joint name="l_leg_ft_joint"/>
-    	    <joint name="r_leg_ft_joint"/>
-    	    <joint name="l_arm_ft_joint"/>
-    	    <joint name="r_arm_ft_joint"/>
-        </group>
-    </xacro:if>
-    <xacro:unless value="${GAZEBO_COGIMON_USES_FOREARMS}">
-        <group name="left_arm">
-            <chain base_link="DWYTorso" tip_link="l_wrist"/>
-        </group>
-        <group name="right_arm">
-            <chain base_link="DWYTorso" tip_link="r_wrist"/>
-        </group>
-        <group name="force_torque_sensors">
-        <!-- NEAREST JOINT TO FORCE_TORQUE SENSOR -->
-            <!--<joint name="LAnkSag"/>
-            <joint name="RAnkSag"/>-->
-            <joint name="l_ankle_joint"/>
-            <joint name="r_ankle_joint"/>
-        </group>
-    </xacro:unless>
+    <group name="left_arm">
+     <chain base_link="DWYTorso" tip_link="l_wrist"/>
+    </group>
+    <group name="right_arm">
+     <chain base_link="DWYTorso" tip_link="r_wrist"/>
+    </group>
+    <group name="force_torque_sensors">
+      <joint name="l_leg_ft_joint"/>
+      <joint name="r_leg_ft_joint"/>
+      <joint name="l_arm_ft_joint"/>
+      <joint name="r_arm_ft_joint"/>
+    </group>
     <group name="left_leg">
         <chain base_link="Waist" tip_link="l_sole"/>

File: cogimon_urdf/urdf/cogimon.urdf.xacro (robot description, xacro)
@@ -4,8 +4,9 @@
   ROS urdf definition of the COGIMON humanoid robot by Istituto Italiano di Tecnologia
   DO NOT INCLUDE THIS FILE DIRECTLY! USE cogimon_robot.urdf.xacro INSTEAD!
-  Author: Enrico Mingo & Alessio Rocchi
+  Author: Enrico Mingo
   Inertial matrix has to be in CoM frame (URDF specs)
-  Velocity and effort limits are fake!
 -->
+<!-- ************ SOME DEFS ********************** -->
+<xacro:include filename="$(find cogimon_urdf)/urdf/conversions.urdf.xacro" />
 <!-- ************ MODEL CONFIGURATION ************ -->
 <xacro:include filename="$(find cogimon_urdf)/urdf/cogimon_config.urdf.xacro" />
@@ -16,21 +17,12 @@
 and to define the end effectors of the robot.
 The coordinate frame called gaze defines the head position and orientation. The orientation indicates in which direction the head appears to be looking regardless of any sensors (camera for instance). -->
-<link name="gaze"/>
-<xacro:if value="${GAZEBO_COGIMON_USES_XTION}">
-	<xacro:include filename="$(find cogimon_urdf)/urdf/sensors/xtion.urdf.xacro" />
-</xacro:if>
-<xacro:unless value="${GAZEBO_COGIMON_USES_XTION}">
+<!--link name="gaze"/>
 	<joint name="gaze_joint" type="fixed">
 		<parent link="torso"/>
 		<child link="gaze"/>
 		<origin xyz="0 0 0.1" rpy="0 0 0" />
-	</joint>
+	</joint-->
         <!-- NECK -->
-	<xacro:include filename="$(find cogimon_urdf)/urdf/parts/neck.urdf.xacro" />
-</xacro:unless>
-<!-- WEIGHT COEFFICIENT FACTOR is a factor that multiplies weights and inertias -->
-<xacro:property name="wcf" value="2.1" />
-<!-- HEIGHT COEFFICIENT OFFSET is a factor added to legs and torso links -->
-<xacro:property name="hco" value="0.1" />
+	<!--xacro:include filename="$(find cogimon_urdf)/urdf/parts/neck.urdf.xacro" />
 <!-- ************ COGIMON BASE ************** -->
 <xacro:include filename="$(find cogimon_urdf)/urdf/cogimon_base.urdf.xacro"/>
@@ -39,5 +31,5 @@
 and to define the end effectors of the robot -->
 <!-- position and orientation of the arm regardless of the tool (grasping device for instance) attached to it -->
-<link name="l_wrist"/>
+<!--link name="l_wrist"/>
 <link name="r_wrist"/>
 <xacro:if value="${GAZEBO_COGIMON_USES_FOREARMS}">
@@ -70,12 +62,12 @@
       <child link="r_leg_ft"/>
       <origin xyz="0 0 -0.065" rpy="0 0 0" />
-    </joint>
+    </joint-->
 <!-- ************ HANDS ************ -->
-<xacro:if value="${GAZEBO_COGIMON_USES_FOREARMS}">
-    <xacro:include filename="$(find cogimon_urdf)/urdf/parts/soft_hand.urdf.xacro" />
+<!--xacro:if value="${GAZEBO_COGIMON_USES_FOREARMS}">
+    <xacro:include filename="$(find cogimon_urdf)/urdf/parts/soft_hand.urdf.xacro" /-->
     <!-- Reference frames in hands -->
-    <xacro:include filename="$(find cogimon_urdf)/urdf/parts/hand_reference_frame.urdf.xacro" />
-</xacro:if>
+    <!--xacro:include filename="$(find cogimon_urdf)/urdf/parts/hand_reference_frame.urdf.xacro" />
+</xacro:if-->
 <!-- IMU -->
-<xacro:include filename="$(find cogimon_urdf)/urdf/sensors/imu.urdf.xacro"/>
+<!--xacro:include filename="$(find cogimon_urdf)/urdf/sensors/imu.urdf.xacro"/-->
 </robot>

File: cogimon_urdf/urdf/cogimon_base.urdf.xacro (robot description, xacro)
@@ -8,5 +8,4 @@
   Velocity and effort limits are fake!
 -->
-<xacro:property name="PI" value="3.14159265359" />
 <!-- This links are defined in order to be compliant with http://www.ros.org/reps/rep-0120.html#coordinate-frames
 and to define the end effectors of the robot
@@ -15,19 +14,19 @@
 <link name="Waist">
     <inertial>
-      <origin xyz="-0.026391145 -5.8216364E-4 0.052632312" rpy="0.0 0.0 0.0"/>
-      <mass value="${wcf*1.8008695}"/>
-      <inertia ixx="${wcf*0.0051032982}"  ixy="${wcf*-5.7170981E-5}"  ixz="${wcf*0.0016920543}" iyy="${wcf*0.006241636}" iyz="${wcf*1.7225949E-5}" izz="${wcf*0.0024517762}" />
+      <origin xyz="${-2.9198594E+01*mmTom} ${-1.1793030E-01*mmTom} ${-3.7516729E+01*mmTom}" rpy="0.0 0.0 0.0"/>
+      <mass value="4.2357548"/>
+      <inertia ixx="${4.6492739E+04*mm2Tom2}"  ixy="${3.3912005E+01*mm2Tom2}"  ixz="${3.0361216E+01*mm2Tom2}" iyy="${1.4628117E+04*mm2Tom2}" iyz="${9.6064394E+00*mm2Tom2}" izz="${5.0051187E+04*mm2Tom2}" />
     </inertial>
     <visual>
-      <origin xyz="0 0 -0.52" rpy="0 0 ${PI}"/>
+      <origin xyz="0 0 0" rpy="0 0 0"/>
       <material name="dark_grey"/>
       <geometry name="Waist_visual">
-        <mesh filename="package://cogimon_urdf/meshes/Waist.STL" scale="0.03937 0.03937 0.03937"/>
+        <mesh filename="package://cogimon_urdf/meshes/Waist.STL" scale="${mmTom} ${mmTom} ${mmTom}"/>
       </geometry>
     </visual>
     <collision>
-      <origin xyz="0 0 -0.52" rpy="0 0 ${PI}"/>
+      <origin xyz="0 0 0" rpy="0 0 0"/>
       <geometry name="Waist_collision">
-        <mesh filename="package://cogimon_urdf/meshes/simple/Waist.STL" scale="0.03937 0.03937 0.03937"/>
+        <mesh filename="package://cogimon_urdf/meshes/simple/Waist.STL" scale="${mmTom} ${mmTom} ${mmTom}"/>
       </geometry>
     </collision>
@@ -40,18 +39,18 @@
 <!-- ********************TORSO******************** -->
 <!-- first real link of the robot, inertial reference frame -->
-<xacro:include filename="$(find cogimon_urdf)/urdf/parts/torso.urdf.xacro" />
+<!--xacro:include filename="$(find cogimon_urdf)/urdf/parts/torso.urdf.xacro" /-->
 <!-- ********************LEGS******************** -->
 <!-- This links are defined in order to be compliant with http://www.ros.org/reps/rep-0120.html#coordinate-frames
 and to define the end effectors of the robot -->
 <!--  position and orientation of the leg regardless of the support body geometry -->
-  <link name="l_ankle"/>
-  <link name="r_ankle"/>
+  <!--link name="l_ankle"/>
+  <link name="r_ankle"/-->
 <!-- position and orientation of the left leg support body. The (X,Y) plane of this frame must be coplanar with the support body contact surface. It is recommended to choose the origin as the projection of the support body origin on the contact surface. The Z coordinate of this frame should be on the ground level when standing. -->
-  <link name="l_sole"/>
-  <link name="r_sole"/>
+  <!--link name="l_sole"/>
+  <link name="r_sole"/-->
 <!--  position and orientation of the leg toe body. The (X,Y) plan of this frame must be coplanar with the toe body contact surface. It is recommended to choose the origin as the projection of the body center on the contact surface. -->
-  <link name="l_toe"/>
-  <link name="r_toe"/>
-<xacro:include filename="$(find cogimon_urdf)/urdf/parts/legs.urdf.xacro" />
+  <!--link name="l_toe"/>
+  <link name="r_toe"/-->
+<!--xacro:include filename="$(find cogimon_urdf)/urdf/parts/legs.urdf.xacro" />
   <joint name="l_ankle_joint" type="fixed">
      <parent link="LFoot"/>
@@ -83,8 +82,8 @@
     <child link="r_toe"/>
     <origin xyz="0.13 0 0" rpy="0 0 0" />
-  </joint>
+  </joint-->
 <!-- Reference frames in feet -->
-<xacro:include filename="$(find cogimon_urdf)/urdf/parts/foot_reference_frame.urdf.xacro" />
+<!--xacro:include filename="$(find cogimon_urdf)/urdf/parts/foot_reference_frame.urdf.xacro" /-->
 <!-- ********************ARMS******************** -->
-<xacro:include filename="$(find cogimon_urdf)/urdf/parts/arms.urdf.xacro" />
+<!--xacro:include filename="$(find cogimon_urdf)/urdf/parts/arms.urdf.xacro" /-->
 </robot>

File: cogimon_urdf/urdf/cogimon_config.urdf.xacro (robot description, xacro)
@@ -1,44 +1,5 @@
 <?xml version="1.0"?>
 <robot xmlns:xacro="http://ros.org/wiki/xacro" name="COGIMON">
-<xacro:property name="model_name" value="IIT COGIMON w/ Softhand" />
+<xacro:property name="model_name" value="IIT COGIMON" />
 <xacro:property name="model_version" value="0.1" />
-<!--
-####################################################
-##
-##  FEET SELECTION
-##
-##
-##
-####################################################
--->
-<xacro:property name="GAZEBO_COGIMON_USES_ROUND_FEET" value="false" />
-<!--
-####################################################
-##
-##  FOREARMS & HANDS SELECTION
-##
-##
-##
-####################################################
--->
-<xacro:property name="GAZEBO_COGIMON_USES_FOREARMS" value="true" />
-<xacro:property name="GAZEBO_COGIMON_USES_SOFTHANDS" value="true" />
-<!--
-####################################################
-##
-##  Xtion SELECTION
-##
-##
-## options:
-## 1) COGIMON classic without the staff to carry the sensor.
-##      Torso frame is connected to gaze link through a gaze_joint "fixed"
-## 2) COGIMON with staff and xtion sensor. Torso frame is connected to a xtion_staff_link through
-##      a xtion_staff_joint "fixed". Xtion_staff_link is then connected to gaze_link through gaze_joint "fixed".
-##
-####################################################
-#
-# 1/2 (true/false)
-#
--->
-<xacro:property name="GAZEBO_COGIMON_USES_XTION" value="false" />
 </robot>

File: cogimon_urdf/urdf/cogimon_robot.urdf.xacro (robot description, xacro)
@@ -7,13 +7,13 @@
   -->
   <xacro:include filename="$(find cogimon_urdf)/urdf/cogimon.urdf.xacro" />
-  <xacro:include filename="$(find cogimon_urdf)/urdf/gazebo/microstrain_3dmgx2_imu.gazebo.xacro" />
+  <!--xacro:include filename="$(find cogimon_urdf)/urdf/gazebo/microstrain_3dmgx2_imu.gazebo.xacro" />
   <xacro:include filename="$(find cogimon_urdf)/urdf/gazebo/cogimon.gazebo.xacro" />
   <xacro:if value="${GAZEBO_COGIMON_USES_XTION}">
 	<xacro:include filename="$(find cogimon_urdf)/urdf/gazebo/openni_kinect.gazebo.xacro" />
-  </xacro:if>
+  </xacro:if-->
 <!-- YARP PLUGINS for GAZEBO SIMULATION -->
-  <xacro:include filename="$(find cogimon_urdf)/urdf/gazebo/yarp_control.gazebo.xacro" />
+  <!--xacro:include filename="$(find cogimon_urdf)/urdf/gazebo/yarp_control.gazebo.xacro" />
   <xacro:include filename="$(find cogimon_urdf)/urdf/gazebo/cogimon_materials.gazebo.xacro" />
-  <xacro:include filename="$(find cogimon_urdf)/urdf/gazebo/force_torque.gazebo.xacro" />
-  <origin xyz="0.0 0.0 ${0.521+2.0*(hco+0.025)}" rpy="0 0 0" />
+  <xacro:include filename="$(find cogimon_urdf)/urdf/gazebo/force_torque.gazebo.xacro" /-->
+  <origin xyz="0.0 0.0 0.521" rpy="0 0 0" />
 </robot>

File: cogimon_urdf/urdf/config/cogimon.urdf.xacro (robot description, xacro)
@@ -1,44 +1,12 @@
 <?xml version="1.0"?>
 <robot xmlns:xacro="http://ros.org/wiki/xacro" name="COGIMON">
-<xacro:property name="model_name" value="IIT COGIMON w/ Softhand" />
+<xacro:property name="model_name" value="IIT COGIMON" />
 <xacro:property name="model_version" value="0.1" />
-<!--
-####################################################
-##
-##  FEET SELECTION
-##
-##
-##
-####################################################
--->
-<xacro:property name="GAZEBO_COGIMON_USES_ROUND_FEET" value="false" />
-<!--
-####################################################
-##
-##  FOREARMS & HANDS SELECTION
-##
-##
-##
-####################################################
--->
-<xacro:property name="GAZEBO_COGIMON_USES_FOREARMS" value="true" />
-<xacro:property name="GAZEBO_COGIMON_USES_SOFTHANDS" value="true" />
-<!--
-####################################################
-##
-##  Xtion SELECTION
-##
-##
-## options:
-## 1) COGIMON classic without the staff to carry the sensor.
-##      Torso frame is connected to gaze link through a gaze_joint "fixed"
-## 2) COGIMON with staff and xtion sensor. Torso frame is connected to a xtion_staff_link through
-##      a xtion_staff_joint "fixed". Xtion_staff_link is then connected to gaze_link through gaze_joint "fixed".
-##
-####################################################
-#
-# 1/2 (true/false)
-#
--->
-<xacro:property name="GAZEBO_COGIMON_USES_XTION" value="false" />
+<!-- ************SELECT PARTS*************-->
+<!-- *************************************-->
+<xacro:property name="COGIMON_TORSO" value="TRUE" />
+<xacro:property name="COGIMON_LEFT_ARM" value="TRUE" />
+<xacro:property name="COGIMON_RIGH_ARM" value="TRUE" />
+<xacro:property name="COGIMON_LEFT_LEG" value="TRUE" />
+<xacro:property name="COGIMON_RIGH_LEG" value="TRUE" />
 </robot>
