Commit message: Added files for simulation with orocos

File: cogimon_srdf/srdf/cogimon.srdf.xacro (robot description, xacro)
@@ -6,43 +6,35 @@
 <robot xmlns:xacro="http://ros.org/wiki/xacro" name="cogimon">
     <xacro:include filename="$(find cogimon_urdf)/urdf/cogimon_config.urdf.xacro" />
-    <virtual_joint name="virtual_joint" parent_frame="world" child_link="base_link" type="floating" />
-    <!--GROUPS: Representation of a set of joints and links. This can be useful for specifying DOF to plan for, defining arms, end effectors, etc-->
-    <!--LINKS: When a link is specified, the parent joint of that link (if it exists) is automatically included-->
-    <!--JOINTS: When a joint is specified, the child link of that joint (which will always exist) is automatically included-->
-    <!--CHAINS: When a chain is specified, all the links along the chain (including endpoints) are included in the group. Additionally, all the joints that are parents to included links are also included. This means that joints along the chain and the parent joint of the base link are included in the group-->
-    <!--SUBGROUPS: Groups can also be formed by referencing to already defined group names-->
     <group name="base">
         <link name="Waist"/>
     </group>
-    <group name="imu_sensors">
-        <link name="imu_link"/>
+<xacro:if value="${COGIMON_LEFT_LEG}">
+    <group name="left_leg">
+        <chain base_link="Waist" tip_link="LFoot"/>
     </group>
-    <group name="left_arm">
-     <chain base_link="DWYTorso" tip_link="l_wrist"/>
+</xacro:if>
+<xacro:if value="${COGIMON_RIGHT_LEG}">
+    <group name="right_leg">
+        <chain base_link="Waist" tip_link="RFoot"/>
     </group>
-    <group name="right_arm">
-     <chain base_link="DWYTorso" tip_link="r_wrist"/>
+</xacro:if>
+  <group name="legs">
+<xacro:if value="${COGIMON_LEFT_LEG}">
+    <group name="left_leg"/>
+</xacro:if>
+<xacro:if value="${COGIMON_RIGHT_LEG}">
+    <group name="right_leg"/>
+</xacro:if>
+  </group>
+    <group name="chains"> <!--THIS HAS TO BE THE LAST GROUP IN THE FILE -->
+<xacro:if value="${COGIMON_LEFT_LEG}">
+        <group name="left_leg"/>
+</xacro:if>
+<xacro:if value="${COGIMON_RIGHT_LEG}">
+        <group name="right_leg"/>
+</xacro:if>
     </group>
-    <group name="force_torque_sensors">
-      <joint name="l_leg_ft_joint"/>
-      <joint name="r_leg_ft_joint"/>
-      <joint name="l_arm_ft_joint"/>
-      <joint name="r_arm_ft_joint"/>
-    </group>
-    <group name="left_leg">
-        <chain base_link="Waist" tip_link="l_sole"/>
-    </group>
-    <group name="right_leg">
-        <chain base_link="Waist" tip_link="r_sole"/>
-    </group>
-    <group name="torso">
-        <chain base_link="Waist" tip_link="DWYTorso"/>
-    </group>
-    <group name="chains"> <!--THIS HAS TO BE THE LAST GROUP IN THE FILE -->
-        <group name="left_arm"/>
-        <group name="right_arm"/>
-        <group name="left_leg"/>
-        <group name="right_leg"/>
-        <group name="torso"/>
-    </group>
+<xacro:if value="${COGIMON_OROCOS_GAZEBO}">
+   <xacro:include filename="$(find cogimon_urdf)/urdf/gazebo/rtt_gazebo.gazebo.xacro" />
+</xacro:if>
 </robot>

File: cogimon_urdf/urdf/cogimon_config.urdf.xacro (robot description, xacro)
@@ -16,6 +16,9 @@
 <!-- ******************************************-->
 <xacro:property name="COGIMON_FIXED_BASE" value="false" />
-<!-- ************XBOT FRAMEWORK*************-->
+<!-- ************XBOT-GAZEBO FRAMEWORK*************-->
 <!-- *************************************-->
-<xacro:property name="COGIMON_XBOT" value="false" />
+<xacro:property name="COGIMON_XBOT_GAZEBO" value="false" />
+<!-- ************OROCOS-GAZEBO FRAMEWORK*************-->
+<!-- *************************************-->
+<xacro:property name="COGIMON_OROCOS_GAZEBO" value="true" />
 </robot>

File: cogimon_urdf/urdf/cogimon_robot.urdf.xacro (robot description, xacro)
@@ -7,9 +7,5 @@
   -->
   <xacro:include filename="$(find cogimon_urdf)/urdf/cogimon.urdf.xacro" />
-  <!--xacro:include filename="$(find cogimon_urdf)/urdf/gazebo/microstrain_3dmgx2_imu.gazebo.xacro" />
   <xacro:include filename="$(find cogimon_urdf)/urdf/gazebo/cogimon.gazebo.xacro" />
-  <xacro:if value="${GAZEBO_COGIMON_USES_XTION}">
-	<xacro:include filename="$(find cogimon_urdf)/urdf/gazebo/openni_kinect.gazebo.xacro" />
-  </xacro:if-->
   <xacro:include filename="$(find cogimon_urdf)/urdf/gazebo/cogimon_materials.gazebo.xacro" />
   <!--xacro:include filename="$(find cogimon_urdf)/urdf/gazebo/force_torque.gazebo.xacro" /-->

File: cogimon_urdf/urdf/gazebo/cogimon.gazebo.xacro (robot description, xacro)
@@ -2,4 +2,5 @@
 <robot xmlns:xacro="http://ros.org/wiki/xacro">
 <!-- contact model for foot surface -->
+<xacro:if value="${COGIMON_LEFT_LEG}">
    <gazebo reference="LFoot">
      <kp>1000000.0</kp>
@@ -11,4 +12,6 @@
      <minDepth>0.0</minDepth>
    </gazebo>
+</xacro:if>
+<xacro:if value="${COGIMON_RIGHT_LEG}">
    <gazebo reference="RFoot">
      <kp>1000000.0</kp>
@@ -20,13 +23,7 @@
      <minDepth>0.00</minDepth>
    </gazebo>
+</xacro:if>
 <!-- Other parameters... -->
-   <gazebo reference="WaistSag">
-    <implicitSpringDamper>1</implicitSpringDamper>
-    <provideFeedback>true</provideFeedback>
-   </gazebo>
-   <gazebo reference="WaistYaw">
-    <implicitSpringDamper>1</implicitSpringDamper>
-    <provideFeedback>true</provideFeedback>
-   </gazebo>
+<xacro:if value="${COGIMON_RIGHT_LEG}">
    <gazebo reference="RHipSag">
     <implicitSpringDamper>1</implicitSpringDamper>
@@ -41,16 +38,18 @@
     <provideFeedback>true</provideFeedback>
    </gazebo>
-   <gazebo reference="RKneeSag">
+   <gazebo reference="RKneePitch">
     <implicitSpringDamper>1</implicitSpringDamper>
     <provideFeedback>true</provideFeedback>
    </gazebo>
-   <gazebo reference="RAnkLat">
+   <gazebo reference="RAnkleRoll">
     <implicitSpringDamper>1</implicitSpringDamper>
     <provideFeedback>true</provideFeedback>
    </gazebo>
-   <gazebo reference="RAnkSag">
+   <gazebo reference="RAnklePitch">
     <implicitSpringDamper>1</implicitSpringDamper>
     <provideFeedback>true</provideFeedback>
   </gazebo>
+</xacro:if>
+<xacro:if value="${COGIMON_LEFT_LEG}">
    <gazebo reference="LHipSag">
     <implicitSpringDamper>1</implicitSpringDamper>
@@ -65,87 +64,16 @@
     <provideFeedback>true</provideFeedback>
    </gazebo>
-   <gazebo reference="LKneeSag">
+   <gazebo reference="LKneePitch">
     <implicitSpringDamper>1</implicitSpringDamper>
     <provideFeedback>true</provideFeedback>
    </gazebo>
-   <gazebo reference="LAnkLat">
+   <gazebo reference="LAnkleRoll">
     <implicitSpringDamper>1</implicitSpringDamper>
     <provideFeedback>true</provideFeedback>
    </gazebo>
-   <gazebo reference="LAnkSag">
+   <gazebo reference="LAnklePitch">
     <implicitSpringDamper>1</implicitSpringDamper>
     <provideFeedback>true</provideFeedback>
-   </gazebo>
-   <gazebo reference="RShSag">
-    <implicitSpringDamper>1</implicitSpringDamper>
-    <provideFeedback>true</provideFeedback>
-   </gazebo>
-   <gazebo reference="RShLat">
-    <implicitSpringDamper>1</implicitSpringDamper>
-    <provideFeedback>true</provideFeedback>
-   </gazebo>
-   <gazebo reference="RShYaw">
-    <implicitSpringDamper>1</implicitSpringDamper>
-    <provideFeedback>true</provideFeedback>
-   </gazebo>
-   <gazebo reference="RElbj">
-    <implicitSpringDamper>1</implicitSpringDamper>
-    <provideFeedback>true</provideFeedback>
-   </gazebo>
-<xacro:if value="${GAZEBO_COGIMON_USES_FOREARMS}">
-   <gazebo reference="RForearmPlate">
-    <implicitSpringDamper>1</implicitSpringDamper>
-    <provideFeedback>true</provideFeedback>
-   </gazebo>
-   <gazebo reference="RWrj1">
-    <implicitSpringDamper>1</implicitSpringDamper>
-    <provideFeedback>true</provideFeedback>
-   </gazebo>
-   <gazebo reference="RWrj2">
-    <implicitSpringDamper>1</implicitSpringDamper>
-    <provideFeedback>true</provideFeedback>
-   </gazebo>
-    <xacro:unless value="${GAZEBO_COGIMON_USES_SOFTHANDS}">
-      <gazebo reference="r_handj">
-        <implicitSpringDamper>1</implicitSpringDamper>
-        <provideFeedback>true</provideFeedback>
-      </gazebo>
-    </xacro:unless>
-</xacro:if>
-   <gazebo reference="LShSag">
-    <implicitSpringDamper>1</implicitSpringDamper>
-    <provideFeedback>true</provideFeedback>
-   </gazebo>
-   <gazebo reference="LShLat">
-    <implicitSpringDamper>1</implicitSpringDamper>
-    <provideFeedback>true</provideFeedback>
-   </gazebo>
-   <gazebo reference="LShYaw">
-    <implicitSpringDamper>1</implicitSpringDamper>
-    <provideFeedback>true</provideFeedback>
-   </gazebo>
-   <gazebo reference="LElbj">
-    <implicitSpringDamper>1</implicitSpringDamper>
-    <provideFeedback>true</provideFeedback>
-   </gazebo>
-<xacro:if value="${GAZEBO_COGIMON_USES_FOREARMS}">
-   <gazebo reference="LForearmPlate">
-    <implicitSpringDamper>1</implicitSpringDamper>
-    <provideFeedback>true</provideFeedback>
-   </gazebo>
-   <gazebo reference="LWrj1">
-    <implicitSpringDamper>1</implicitSpringDamper>
-    <provideFeedback>true</provideFeedback>
-   </gazebo>
-   <gazebo reference="LWrj2">
-    <implicitSpringDamper>1</implicitSpringDamper>
-    <provideFeedback>true</provideFeedback>
-   </gazebo>
-    <xacro:unless value="${GAZEBO_COGIMON_USES_SOFTHANDS}">
-      <gazebo reference="l_handj">
-        <implicitSpringDamper>1</implicitSpringDamper>
-        <provideFeedback>true</provideFeedback>
-      </gazebo>
-    </xacro:unless>
+  </gazebo>
 </xacro:if>
 </robot>

Commit message: Added xbot related stuffs

File: cogimon_srdf/srdf/cogimon.srdf.xacro (robot description, xacro)
@@ -38,3 +38,17 @@
    <xacro:include filename="$(find cogimon_urdf)/urdf/gazebo/rtt_gazebo.gazebo.xacro" />
 </xacro:if>
+<group_state name="home" group="chains">
+        <joint name="LHipLat" value="0.0"/>
+        <joint name="LHipSag" value="0.0"/>
+        <joint name="LHipYaw" value="0.0"/>
+        <joint name="LKneePitch" value="0.0"/>
+        <joint name="LAnklePitch" value="0.0"/>
+        <joint name="LAnkleRoll" value="0.0"/>
+        <joint name="RHipLat" value="0.0"/>
+        <joint name="RHipSag" value="0.0"/>
+        <joint name="RHipYaw" value="0.0"/>
+        <joint name="RKneePitch" value="0.0"/>
+        <joint name="RAnklePitch" value="0.0"/>
+        <joint name="RAnkleRoll" value="0.0"/>
+</group_state>
 </robot>

File: cogimon_urdf/urdf/cogimon_config.urdf.xacro (robot description, xacro)
@@ -18,7 +18,7 @@
 <!-- ************XBOT-GAZEBO FRAMEWORK*************-->
 <!-- *************************************-->
-<xacro:property name="COGIMON_XBOT_GAZEBO" value="false" />
+<xacro:property name="COGIMON_XBOT_GAZEBO" value="true" />
 <!-- ************OROCOS-GAZEBO FRAMEWORK*************-->
 <!-- *************************************-->
-<xacro:property name="COGIMON_OROCOS_GAZEBO" value="true" />
+<xacro:property name="COGIMON_OROCOS_GAZEBO" value="false" />
 </robot>

Commit message: Updated model. Added ft sensors. Removed cloned folder

File: cogimon_srdf/srdf/cogimon.srdf.xacro (robot description, xacro)
@@ -9,4 +9,12 @@
         <link name="Waist"/>
     </group>
+<group name="force_torque_sensors">
+<xacro:if value="${COGIMON_LEFT_LEG}">
+    <joint name="l_leg_ft_joint"/>
+</xacro:if>
+<xacro:if value="${COGIMON_RIGHT_LEG}">
+    <joint name="r_leg_ft_joint"/>
+</xacro:if>
+</group>
 <xacro:if value="${COGIMON_LEFT_LEG}">
     <group name="left_leg">

File: cogimon_urdf/urdf/cogimon_base.urdf.xacro (robot description, xacro)
@@ -36,54 +36,4 @@
     <origin xyz="0 0 0" rpy="0 0 0" />
 </joint>
-<!-- ********************TORSO******************** -->
-<!-- first real link of the robot, inertial reference frame -->
-<!--xacro:include filename="$(find cogimon_urdf)/urdf/parts/torso.urdf.xacro" /-->
-<!-- ********************LEGS******************** -->
-<!-- This links are defined in order to be compliant with http://www.ros.org/reps/rep-0120.html#coordinate-frames
-and to define the end effectors of the robot -->
-<!--  position and orientation of the leg regardless of the support body geometry -->
-  <!--link name="l_ankle"/>
-  <link name="r_ankle"/-->
-<!-- position and orientation of the left leg support body. The (X,Y) plane of this frame must be coplanar with the support body contact surface. It is recommended to choose the origin as the projection of the support body origin on the contact surface. The Z coordinate of this frame should be on the ground level when standing. -->
-  <!--link name="l_sole"/>
-  <link name="r_sole"/-->
-<!--  position and orientation of the leg toe body. The (X,Y) plan of this frame must be coplanar with the toe body contact surface. It is recommended to choose the origin as the projection of the body center on the contact surface. -->
-  <!--link name="l_toe"/>
-  <link name="r_toe"/-->
 <xacro:include filename="$(find cogimon_urdf)/urdf/parts/legs.urdf.xacro" />
-<!--
-  <joint name="l_ankle_joint" type="fixed">
-     <parent link="LFoot"/>
-     <child link="l_ankle"/>
-     <origin xyz="0 0 0" rpy="0 0 0" />
-  </joint>
-  <joint name="r_ankle_joint" type="fixed">
-    <parent link="RFoot"/>
-    <child link="r_ankle"/>
-    <origin xyz="0 0 0" rpy="0 0 0" />
-  </joint>
-  <joint name="l_sole_joint" type="fixed">
-    <parent link="LFoot"/>
-    <child link="l_sole"/>
-    <origin xyz="0 0 -0.09" rpy="0 0 0" />
-  </joint>
-  <joint name="r_sole_joint" type="fixed">
-    <parent link="RFoot"/>
-    <child link="r_sole"/>
-    <origin xyz="0 0 -0.09" rpy="0 0 0" />
-  </joint>
-  <joint name="l_toe_joint" type="fixed">
-    <parent link="l_sole"/>
-    <child link="l_toe"/>
-    <origin xyz="0.13 0 0" rpy="0 0 0" />
-  </joint>
-  <joint name="r_toe_joint" type="fixed">
-    <parent link="r_sole"/>
-    <child link="r_toe"/>
-    <origin xyz="0.13 0 0" rpy="0 0 0" />
-  </joint-->
-<!-- Reference frames in feet -->
-<!--xacro:include filename="$(find cogimon_urdf)/urdf/parts/foot_reference_frame.urdf.xacro" /-->
-<!-- ********************ARMS******************** -->
-<!--xacro:include filename="$(find cogimon_urdf)/urdf/parts/arms.urdf.xacro" /-->
 </robot>

File: cogimon_urdf/urdf/cogimon_config.urdf.xacro (robot description, xacro)
@@ -18,7 +18,7 @@
 <!-- ************XBOT-GAZEBO FRAMEWORK*************-->
 <!-- *************************************-->
-<xacro:property name="COGIMON_XBOT_GAZEBO" value="true" />
+<xacro:property name="COGIMON_XBOT_GAZEBO" value="false" />
 <!-- ************OROCOS-GAZEBO FRAMEWORK*************-->
 <!-- *************************************-->
-<xacro:property name="COGIMON_OROCOS_GAZEBO" value="false" />
+<xacro:property name="COGIMON_OROCOS_GAZEBO" value="true" />
 </robot>

File: cogimon_urdf/urdf/cogimon_robot.urdf.xacro (robot description, xacro)
@@ -9,5 +9,5 @@
   <xacro:include filename="$(find cogimon_urdf)/urdf/gazebo/cogimon.gazebo.xacro" />
   <xacro:include filename="$(find cogimon_urdf)/urdf/gazebo/cogimon_materials.gazebo.xacro" />
-  <!--xacro:include filename="$(find cogimon_urdf)/urdf/gazebo/force_torque.gazebo.xacro" /-->
+  <xacro:include filename="$(find cogimon_urdf)/urdf/gazebo/force_torque.gazebo.xacro" />
 <xacro:if value="${COGIMON_XBOT_GAZEBO}" >
   <xacro:include filename="$(find cogimon_urdf)/urdf/gazebo/xbot_control.gazebo.xacro" />

File: cogimon_urdf/urdf/gazebo/rtt_gazebo.gazebo.xacro (robot description, xacro)
@@ -4,10 +4,10 @@
 <rtt-gazebo reference="right_leg">
        <controller type="JointPositionCtrl">
-              <gains reference="RHipSag" P="1000." D="1.0" I="0."/>
-              <gains reference="RHipLat" P="1000." D="1.0" I="0."/>
-              <gains reference="RHipYaw" P="1000." D="1.0" I="0."/>
-              <gains reference="RKneePitch" P="1000." D="1.0" I="0."/>
-              <gains reference="RAnklePitch" P="1000." D="1.0" I="0."/>
-              <gains reference="RAnkleRoll" P="1000." D="1.0" I="0."/>
+              <gains D="12.0" I="2." P="7500." reference="RHipSag"/>
+              <gains D="10.0" I="0." P="4500." reference="RHipLat"/>
+              <gains D="10." I="0." P="4000." reference="RHipYaw"/>
+              <gains D="5.0" I="0." P="3500." reference="RKneePitch"/>
+              <gains D="7.0" I="0." P="5500." reference="RAnklePitch"/>
+              <gains D="5.0" I="0." P="2500." reference="RAnkleRoll"/>
        </controller>
        <controller type="JointImpedanceCtrl">
@@ -25,10 +25,10 @@
 <rtt-gazebo reference="left_leg">
        <controller type="JointPositionCtrl">
-              <gains reference="LHipSag" P="1000." D="1.0" I="0."/>
-              <gains reference="LHipLat" P="1000." D="1.0" I="0."/>
-              <gains reference="LHipYaw" P="1000." D="1.0" I="0."/>
-              <gains reference="LKneePitch" P="1000." D="1.0" I="0."/>
-              <gains reference="LAnklePitch" P="1000." D="1.0" I="0."/>
-              <gains reference="LAnkleRoll" P="1000." D="1.0" I="0."/>
+              <gains D="12.0" I="2." P="7500." reference="LHipSag"/>
+              <gains D="10.0" I="0." P="4500." reference="LHipLat"/>
+              <gains D="10." I="0." P="4000." reference="LHipYaw"/>
+              <gains D="5.0" I="0." P="3500." reference="LKneePitch"/>
+              <gains D="7.0" I="0." P="5500." reference="LAnklePitch"/>
+              <gains D="5.0" I="0." P="2500." reference="LAnkleRoll"/>
        </controller>
        <controller type="JointImpedanceCtrl">

File: cogimon_urdf/urdf/parts/feet_reference_frames.urdf.xacro (robot description, xacro)
@@ -20,4 +20,10 @@
 <link name="l_toe"/>
 <link name="l_heel"/>
+<link name="l_leg_ft"/>
+<joint name="l_leg_ft_joint" type="fixed">
+       <origin xyz="0 0 -0.035" rpy="0 0 0" />
+	<parent link="LFoot"/>
+	<child link="l_leg_ft"/>
+</joint>
 <joint name="l_ankle_joint" type="fixed">
        <origin xyz="0 0 0" rpy="0 0 0" />
@@ -47,4 +53,10 @@
 <link name="r_toe"/>
 <link name="r_heel"/>
+<link name="r_leg_ft"/>
+<joint name="r_leg_ft_joint" type="fixed">
+       <origin xyz="0 0 -0.035" rpy="0 0 0" />
+	<parent link="RFoot"/>
+	<child link="r_leg_ft"/>
+</joint>
 <joint name="r_ankle_joint" type="fixed">
        <origin xyz="0 0 0" rpy="0 0 0" />

Commit message: Added torso chain and gains for rtt_gazebo

File: cogimon_srdf/srdf/cogimon.srdf.xacro (robot description, xacro)
@@ -27,4 +27,9 @@
     </group>
 </xacro:if>
+<xacro:if value="${COGIMON_TORSO}">
+    <group name="torso">
+        <chain base_link="Waist" tip_link="DWL"/>
+    </group>
+</xacro:if>
   <group name="legs">
 <xacro:if value="${COGIMON_LEFT_LEG}">
@@ -33,4 +38,7 @@
 <xacro:if value="${COGIMON_RIGHT_LEG}">
     <group name="right_leg"/>
+</xacro:if>
+<xacro:if value="${COGIMON_TORSO}">
+    <group name="torso"/>
 </xacro:if>
   </group>
@@ -41,4 +49,7 @@
 <xacro:if value="${COGIMON_RIGHT_LEG}">
         <group name="right_leg"/>
+</xacro:if>
+<xacro:if value="${COGIMON_TORSO}">
+        <group name="torso"/>
 </xacro:if>
     </group>
@@ -59,4 +70,5 @@
         <joint name="RAnklePitch" value="0.0"/>
         <joint name="RAnkleRoll" value="0.0"/>
+        <joint name="WaistLat" value="0.0"/>
 </group_state>
 </robot>

File: cogimon_urdf/urdf/gazebo/rtt_gazebo.gazebo.xacro (robot description, xacro)
@@ -43,3 +43,14 @@
 </rtt-gazebo>
 </xacro:if>
+<xacro:if value="${COGIMON_TORSO}">
+<rtt-gazebo reference="torso">
+       <controller type="JointPositionCtrl">
+              <gains D="12.0" I="2." P="7500." reference="WaistLat"/>
+       </controller>
+       <controller type="JointImpedanceCtrl">
+              <gains reference="WaistLat" stiffness="300." damping="30."/>
+       </controller>
+       <controller type="JointTorqueCtrl"/>
+</rtt-gazebo>
+</xacro:if>
 </robot>
