Commit message: Added torso

File: cogimon_srdf/srdf/cogimon.srdf.xacro (robot description, xacro)
@@ -29,5 +29,10 @@
 <xacro:if value="${COGIMON_TORSO}">
     <group name="torso">
-        <chain base_link="Waist" tip_link="DWL"/>
+	<xacro:if value="${COGIMON_PENNACCHIO}">
+        	<chain base_link="Waist" tip_link="DWL"/>
+	</xacro:if>
+        <xacro:unless value="${COGIMON_PENNACCHIO}">
+        	<chain base_link="Waist" tip_link="DWYTorso"/>
+	</xacro:unless>
     </group>
 </xacro:if>

File: cogimon_urdf/urdf/config/cogimon.urdf.xacro (robot description, xacro)
@@ -17,5 +17,5 @@
 -->
 <!-- *************************************-->
-<xacro:property name="COGIMON_PENNACCHIO" value="true" />
+<xacro:property name="COGIMON_PENNACCHIO" value="false" />
 <!-- ************FLOATING BASE*************-->
 <!-- ******************************************-->

File: cogimon_urdf/urdf/config/cogimon_pennacchio.urdf.xacro (robot description, xacro)
@@ -1,5 +1,5 @@
 <?xml version="1.0"?>
 <robot xmlns:xacro="http://ros.org/wiki/xacro" name="COGIMON">
-<xacro:property name="model_name" value="IIT COGIMON" />
+<xacro:property name="model_name" value="IIT COGIMON PENNACCHIO" />
 <xacro:property name="model_version" value="0.1" />
 <!-- ************SELECT PARTS*************-->
@@ -17,5 +17,5 @@
 -->
 <!-- *************************************-->
-<xacro:property name="COGIMON_PENNACCHIO" value="false" />
+<xacro:property name="COGIMON_PENNACCHIO" value="true" />
 <!-- ************FLOATING BASE*************-->
 <!-- ******************************************-->

File: cogimon_urdf/urdf/gazebo/cogimon_materials.gazebo.xacro (robot description, xacro)
@@ -48,9 +48,17 @@
   <material>Gazebo/DarkGrey</material>
 </gazebo>
-<xacro:if value="${COGIMON_TORSO}">
+<xacro:if value="${COGIMON_PENNACCHIO}">
 <gazebo reference="pennacchio">
   <material>Gazebo/DarkGrey</material>
 </gazebo>
 </xacro:if>
+<xacro:unless value="${COGIMON_PENNACCHIO}">
+<gazebo reference="DWLExt">
+  <material>Gazebo/Green</material>
+</gazebo>
+<gazebo reference="DWYTorso">
+  <material>Gazebo/DarkGrey</material>
+</gazebo>
+</xacro:unless>
 </xacro:if>
 </robot>

File: cogimon_urdf/urdf/gazebo/rtt_gazebo.gazebo.xacro (robot description, xacro)
@@ -47,7 +47,13 @@
        <controller type="JointPositionCtrl">
               <gains D="12.0" I="2." P="7500." reference="WaistLat"/>
+	      <xacro:unless value="${COGIMON_PENNACCHIO}">
+			<gains D="10.0" I="2." P="5000." reference="WaistYaw"/>
+	      </xacro:unless>
        </controller>
        <controller type="JointImpedanceCtrl">
               <gains reference="WaistLat" stiffness="300." damping="30."/>
+              <xacro:unless value="${COGIMON_PENNACCHIO}">
+			<gains reference="WaistYaw" stiffness="300." damping="30."/>
+	      </xacro:unless>
        </controller>
        <controller type="JointTorqueCtrl"/>

File: cogimon_urdf/urdf/parts/torso.urdf.xacro (robot description, xacro)
@@ -69,4 +69,46 @@
 </link>
 </xacro:if>
+<xacro:unless value="${COGIMON_PENNACCHIO}">
+<link name ="DWLExt">
+    <inertial>
+      <origin xyz="${1.5386429e-03*mmTom} ${5.1668430e-02*mmTom} ${9.5210134e+01 *mmTom} " rpy="0 0 0"/>
+      <mass value="9.6910635e-01"/>
+      <inertia ixx="${3.0414870e+03*mm2Tom2}"  ixy="${-2.8413688*mm2Tom2}"  ixz="${9.6851038e+01*mm2Tom2}" iyy="${3.0465319e+03*mm2Tom2}" iyz="${-8.8025302*mm2Tom2}" izz="${1.5978729e+03*mm2Tom2}" />
+    </inertial>
+    <visual>
+      <origin xyz="0.0 0.0 0.0" rpy="0 0 0"/>
+      <geometry name="DWLExt_visual">
+        <mesh filename="package://cogimon_urdf/meshes/TorsoRollExt.stl" scale="${mmTom} ${mmTom} ${mmTom}" />
+      </geometry>
+      <material name="green"/>
+    </visual>
+    <collision>
+      <origin xyz="0.0 0.0 0.0" rpy="0 0 0"/>
+      <geometry name="DWLExt_collision">
+        <mesh filename="package://cogimon_urdf/meshes/simple/TorsoRollExt.stl" scale="${mmTom} ${mmTom} ${mmTom}" />
+      </geometry>
+    </collision>
+</link>
+<link name ="DWYTorso">
+    <inertial>
+        <origin xyz="${-5.9646212e+01*mmTom} ${1.4305062*mmTom} ${4.2741527e+01*mmTom}" rpy="0 0 0"/>
+        <mass value="1.2512295e+01"/>
+      <inertia ixx="${2.1021617e+05*mm2Tom2}"  ixy="${-1.5527214e+02*mm2Tom2}"  ixz="${-5.0216602e+04*mm2Tom2}" iyy="${1.9982996e+05*mm2Tom2}" iyz="${-2.9204792e+02*mm2Tom2}" izz="${1.4025094e+05*mm2Tom2}" />
+    </inertial>
+    <visual>
+      <origin xyz="0.0 0.0 0.0" rpy="0 0 0"/>
+      <geometry name="DWYTorso_visual">
+        <mesh filename="package://cogimon_urdf/meshes/Chest.stl" scale="${mmTom} ${mmTom} ${mmTom}" />
+      </geometry>
+      <material name="dark_grey"/>
+    </visual>
+    <collision>
+      <origin xyz="0.0 0.0 0.0" rpy="0 0 0"/>
+      <geometry name="DWYTorso_collision">
+        <mesh filename="package://cogimon_urdf/meshes/simple/Chest.stl" scale="${mmTom} ${mmTom} ${mmTom}" />
+      </geometry>
+    </collision>
+</link>
+</xacro:unless>
 <!-- JOINTS -->
 <joint name="WaistLat" type="revolute">
@@ -90,4 +132,19 @@
 </joint>
 </xacro:if>
+<xacro:unless value="${COGIMON_PENNACCHIO}">
+<joint name="WaistFixed" type="fixed">
+    <parent link="DWL"/>
+    <child link="DWLExt"/>
+    <origin xyz="${-54.0957*mmTom} 0.0 ${63.5*mmTom}" rpy="0 0 0" />
+</joint>
+<joint name="WaistYaw" type="revolute">
+    <parent link="DWLExt"/>
+    <child link="DWYTorso"/>
+    <origin xyz="0 0 ${168.15*mmTom}" rpy="0 0 0" />
+    <axis xyz="0 0 1" />
+    <limit velocity="6.283" effort="120" lower="${-100.0*toRad}" upper="${100.0*toRad}" />
+    <dynamics friction="0" damping="3.0"/>
+</joint>
+</xacro:unless>
 </xacro:if>
 </robot>

Commit message: Added upper body

File: cogimon_srdf/srdf/cogimon.srdf.xacro (robot description, xacro)
@@ -37,16 +37,15 @@
     </group>
 </xacro:if>
-  <group name="legs">
-<xacro:if value="${COGIMON_LEFT_LEG}">
-    <group name="left_leg"/>
+<xacro:if value="${COGIMON_LEFT_ARM}">
+    <group name="left_arm">
+        <chain base_link="DWYTorso" tip_link="LWrMot3"/>
+    </group>
 </xacro:if>
-<xacro:if value="${COGIMON_RIGHT_LEG}">
-    <group name="right_leg"/>
+<xacro:if value="${COGIMON_RIGHT_ARM}">
+    <group name="right_arm">
+        <chain base_link="DWYTorso" tip_link="RWrMot3"/>
+    </group>
 </xacro:if>
-<xacro:if value="${COGIMON_TORSO}">
-    <group name="torso"/>
-</xacro:if>
-  </group>
-    <group name="chains"> <!--THIS HAS TO BE THE LAST GROUP IN THE FILE -->
+<group name="chains"> <!--THIS HAS TO BE THE LAST GROUP IN THE FILE -->
 <xacro:if value="${COGIMON_LEFT_LEG}">
         <group name="left_leg"/>
@@ -58,8 +57,15 @@
         <group name="torso"/>
 </xacro:if>
-    </group>
+<xacro:if value="${COGIMON_LEFT_ARM}">
+        <group name="left_arm"/>
+</xacro:if>
+<xacro:if value="${COGIMON_RIGHT_ARM}">
+        <group name="right_arm"/>
+</xacro:if>
+</group>
 <xacro:if value="${COGIMON_OROCOS_GAZEBO}">
    <xacro:include filename="$(find cogimon_urdf)/urdf/gazebo/rtt_gazebo.gazebo.xacro" />
 </xacro:if>
+<xacro:if value="${COGIMON_XBOT_GAZEBO}">
 <group_state name="home" group="chains">
         <joint name="LHipLat" value="0.0"/>
@@ -76,4 +82,20 @@
         <joint name="RAnkleRoll" value="0.0"/>
         <joint name="WaistLat" value="0.0"/>
+	<joint name="Waistyaw" value="0.0"/>
+        <joint name="RShSag" value="0.0"/>
+        <joint name="RShLat" value="0.0"/>
+        <joint name="RShYaw" value="0.0"/>
+        <joint name="RElbj" value="0.0"/>
+        <joint name="RForearmPlate" value="0.0"/>
+        <joint name="RWrj1" value="0.0"/>
+        <joint name="RWrj2" value="0.0"/>
+        <joint name="LShSag" value="0.0"/>
+        <joint name="LShLat" value="0.0"/>
+        <joint name="LShYaw" value="0.0"/>
+        <joint name="LElbj" value="0.0"/>
+        <joint name="LForearmPlate" value="0.0"/>
+        <joint name="LWrj1" value="0.0"/>
+        <joint name="LWrj2" value="0.0"/>
 </group_state>
+</xacro:if>
 </robot>

File: cogimon_urdf/urdf/cogimon_base.urdf.xacro (robot description, xacro)
@@ -48,5 +48,7 @@
     </inertial>
 </link>
+<!-- SELECTION OF KINEMATICS CHAINS IS HANDLED INSIDE THE FILES -->
 <xacro:include filename="$(find cogimon_urdf)/urdf/parts/legs.urdf.xacro" />
 <xacro:include filename="$(find cogimon_urdf)/urdf/parts/torso.urdf.xacro" />
+<xacro:include filename="$(find cogimon_urdf)/urdf/parts/arms.urdf.xacro" />
 </robot>

File: cogimon_urdf/urdf/cogimon_config.urdf.xacro (robot description, xacro)
@@ -6,6 +6,6 @@
 <!-- *************************************-->
 <xacro:property name="COGIMON_TORSO" value="true" />
-<xacro:property name="COGIMON_LEFT_ARM" value="false" />
-<xacro:property name="COGIMON_RIGHT_ARM" value="false" />
+<xacro:property name="COGIMON_LEFT_ARM" value="true" />
+<xacro:property name="COGIMON_RIGHT_ARM" value="true" />
 <xacro:property name="COGIMON_LEFT_LEG" value="true" />
 <xacro:property name="COGIMON_RIGHT_LEG" value="true" />

File: cogimon_urdf/urdf/gazebo/cogimon.gazebo.xacro (robot description, xacro)
@@ -82,4 +82,70 @@
     <provideFeedback>true</provideFeedback>
    </gazebo>
+   <xacro:unless value="${COGIMON_PENNACCHIO}">
+     <gazebo reference="WaistYaw">
+    <implicitSpringDamper>1</implicitSpringDamper>
+    <provideFeedback>true</provideFeedback>
+   </gazebo>
+   </xacro:unless>
+</xacro:if>
+<xacro:if value="${COGIMON_LEFT_ARM}">
+<gazebo reference="LShSag">
+    <implicitSpringDamper>1</implicitSpringDamper>
+    <provideFeedback>true</provideFeedback>
+   </gazebo>
+   <gazebo reference="LShLat">
+    <implicitSpringDamper>1</implicitSpringDamper>
+    <provideFeedback>true</provideFeedback>
+   </gazebo>
+   <gazebo reference="LShYaw">
+    <implicitSpringDamper>1</implicitSpringDamper>
+    <provideFeedback>true</provideFeedback>
+   </gazebo>
+   <gazebo reference="LElbj">
+    <implicitSpringDamper>1</implicitSpringDamper>
+    <provideFeedback>true</provideFeedback>
+   </gazebo>
+   <gazebo reference="LForearmPlate">
+    <implicitSpringDamper>1</implicitSpringDamper>
+    <provideFeedback>true</provideFeedback>
+   </gazebo>
+   <gazebo reference="LWrj1">
+    <implicitSpringDamper>1</implicitSpringDamper>
+    <provideFeedback>true</provideFeedback>
+  </gazebo>
+   <gazebo reference="LWrj2">
+    <implicitSpringDamper>1</implicitSpringDamper>
+    <provideFeedback>true</provideFeedback>
+  </gazebo>
+</xacro:if>
+<xacro:if value="${COGIMON_RIGHT_ARM}">
+<gazebo reference="RShSag">
+    <implicitSpringDamper>1</implicitSpringDamper>
+    <provideFeedback>true</provideFeedback>
+   </gazebo>
+   <gazebo reference="RShLat">
+    <implicitSpringDamper>1</implicitSpringDamper>
+    <provideFeedback>true</provideFeedback>
+   </gazebo>
+   <gazebo reference="RShYaw">
+    <implicitSpringDamper>1</implicitSpringDamper>
+    <provideFeedback>true</provideFeedback>
+   </gazebo>
+   <gazebo reference="RElbj">
+    <implicitSpringDamper>1</implicitSpringDamper>
+    <provideFeedback>true</provideFeedback>
+   </gazebo>
+   <gazebo reference="RForearmPlate">
+    <implicitSpringDamper>1</implicitSpringDamper>
+    <provideFeedback>true</provideFeedback>
+   </gazebo>
+   <gazebo reference="RWrj1">
+    <implicitSpringDamper>1</implicitSpringDamper>
+    <provideFeedback>true</provideFeedback>
+  </gazebo>
+   <gazebo reference="RWrj2">
+    <implicitSpringDamper>1</implicitSpringDamper>
+    <provideFeedback>true</provideFeedback>
+  </gazebo>
 </xacro:if>
 </robot>

File: cogimon_urdf/urdf/gazebo/cogimon_materials.gazebo.xacro (robot description, xacro)
@@ -62,3 +62,49 @@
 </xacro:unless>
 </xacro:if>
+<xacro:if value="${COGIMON_LEFT_ARM}">
+<gazebo reference="LShp">
+  <material>Gazebo/Green</material>
+</gazebo>
+<gazebo reference="LShr">
+  <material>Gazebo/DarkGrey</material>
+</gazebo>
+<gazebo reference="LShy">
+  <material>Gazebo/Green</material>
+</gazebo>
+<gazebo reference="LElb">
+  <material>Gazebo/DarkGrey</material>
+</gazebo>
+<gazebo reference="LForearm">
+  <material>Gazebo/Green</material>
+</gazebo>
+<gazebo reference="LWrMot2">
+  <material>Gazebo/DarkGrey</material>
+</gazebo>
+<gazebo reference="LWrMot2">
+  <material>Gazebo/Green</material>
+</gazebo>
+</xacro:if>
+<xacro:if value="${COGIMON_RIGHT_ARM}">
+<gazebo reference="RShp">
+  <material>Gazebo/Green</material>
+</gazebo>
+<gazebo reference="RShr">
+  <material>Gazebo/DarkGrey</material>
+</gazebo>
+<gazebo reference="RShy">
+  <material>Gazebo/Green</material>
+</gazebo>
+<gazebo reference="RElb">
+  <material>Gazebo/DarkGrey</material>
+</gazebo>
+<gazebo reference="RForearm">
+  <material>Gazebo/Green</material>
+</gazebo>
+<gazebo reference="RWrMot2">
+  <material>Gazebo/DarkGrey</material>
+</gazebo>
+<gazebo reference="RWrMot2">
+  <material>Gazebo/Green</material>
+</gazebo>
+</xacro:if>
 </robot>

File: cogimon_urdf/urdf/gazebo/rtt_gazebo.gazebo.xacro (robot description, xacro)
@@ -60,3 +60,49 @@
 </rtt-gazebo>
 </xacro:if>
+<xacro:if value="${COGIMON_LEFT_ARM}">
+<rtt-gazebo reference="left_arm">
+       <controller type="JointPositionCtrl">
+              <gains D="10.0" I="2." P="7500." reference="LShSag"/>
+	      <gains D="10.0" I="0." P="4500." reference="LShLat"/>
+	      <gains D="10." I="0." P="4000." reference="LShYaw"/>
+	      <gains D="5.0" I="0." P="3500." reference="LElbj"/>
+	      <gains D="2.0" I="0." P="2000." reference="LForearmPlate"/>
+	      <gains D="2.0" I="0." P="2000." reference="LWrj1"/>
+              <gains D="2.0" I="0." P="2000." reference="LWrj2"/>
+       </controller>
+       <controller type="JointImpedanceCtrl">
+              <gains reference="LShSag" stiffness="300." damping="30."/>
+              <gains reference="LShLat" stiffness="300." damping="30."/>
+              <gains reference="LShYaw" stiffness="300." damping="30."/>
+              <gains reference="LElbj" stiffness="300." damping="30."/>
+              <gains reference="LForearmPlate" stiffness="300." damping="30."/>
+              <gains reference="LWrj1" stiffness="300." damping="30."/>
+              <gains reference="LWrj2" stiffness="300." damping="30."/>
+       </controller>
+       <controller type="JointTorqueCtrl"/>
+</rtt-gazebo>
+</xacro:if>
+<xacro:if value="${COGIMON_RIGHT_ARM}">
+<rtt-gazebo reference="right_arm">
+       <controller type="JointPositionCtrl">
+              <gains D="10.0" I="2." P="7500." reference="RShSag"/>
+	      <gains D="10.0" I="0." P="4500." reference="RShLat"/>
+	      <gains D="10." I="0." P="4000." reference="RShYaw"/>
+	      <gains D="5.0" I="0." P="3500." reference="RElbj"/>
+	      <gains D="2.0" I="0." P="2000." reference="RForearmPlate"/>
+	      <gains D="2.0" I="0." P="2000." reference="RWrj1"/>
+              <gains D="2.0" I="0." P="2000." reference="RWrj2"/>
+       </controller>
+       <controller type="JointImpedanceCtrl">
+              <gains reference="RShSag" stiffness="300." damping="30."/>
+              <gains reference="RShLat" stiffness="300." damping="30."/>
+              <gains reference="RShYaw" stiffness="300." damping="30."/>
+              <gains reference="RElbj" stiffness="300." damping="30."/>
+              <gains reference="RForearmPlate" stiffness="300." damping="30."/>
+              <gains reference="RWrj1" stiffness="300." damping="30."/>
+              <gains reference="RWrj2" stiffness="300." damping="30."/>
+       </controller>
+       <controller type="JointTorqueCtrl"/>
+</rtt-gazebo>
+</xacro:if>
 </robot>

Commit message: Added head joint and possibility to select if fixed or revolute. Updated srdf with new kinematic chains accordingly to the given configs

File: cogimon_srdf/srdf/cogimon.srdf.xacro (robot description, xacro)
@@ -47,4 +47,11 @@
     </group>
 </xacro:if>
+<xacro:unless value="${COGIMON_LASER_FIXED}">
+    <xacro:if value="${COGIMON_HEAD}">
+        <group name="head">
+            <chain base_link="Neck" tip_link="HeadHokuyo"/>
+        </group>
+    </xacro:if>
+</xacro:unless>
 <group name="chains"> <!--THIS HAS TO BE THE LAST GROUP IN THE FILE -->
 <xacro:if value="${COGIMON_LEFT_LEG}">
@@ -63,4 +70,9 @@
         <group name="right_arm"/>
 </xacro:if>
+<xacro:unless value="${COGIMON_LASER_FIXED}">
+    <xacro:if value="${COGIMON_HEAD}">
+        <group name="head"/>
+    </xacro:if>
+</xacro:unless>
 </group>
 <xacro:if value="${COGIMON_OROCOS_GAZEBO}">
@@ -97,4 +109,9 @@
         <joint name="LWrj1" value="0.0"/>
         <joint name="LWrj2" value="0.0"/>
+	<xacro:unless value="${COGIMON_LASER_FIXED}">
+    	<xacro:if value="${COGIMON_HEAD}">
+        	<joint name="head_roll" value="0.0"/>
+    	</xacro:if>
+	</xacro:unless>
 </group_state>
 </xacro:if>

File: cogimon_urdf/urdf/gazebo/cogimon.gazebo.xacro (robot description, xacro)
@@ -144,5 +144,5 @@
     <provideFeedback>true</provideFeedback>
   </gazebo>
-   <gazebo reference="RWrj2">
+  <gazebo reference="RWrj2">
     <implicitSpringDamper>1</implicitSpringDamper>
     <provideFeedback>true</provideFeedback>
@@ -150,4 +150,8 @@
 </xacro:if>
 <xacro:if value="${COGIMON_HEAD}">
+  <gazebo reference="head_roll">
+    <implicitSpringDamper>1</implicitSpringDamper>
+    <provideFeedback>true</provideFeedback>
+  </gazebo>
 </xacro:if>
 </robot>

File: cogimon_urdf/urdf/gazebo/rtt_gazebo.gazebo.xacro (robot description, xacro)
@@ -106,3 +106,10 @@
 </rtt-gazebo>
 </xacro:if>
+<xacro:unless value="${COGIMON_LASER_FIXED}">
+  <xacro:if value="${COGIMON_HEAD}">
+    <controller type="JointPositionCtrl">
+      <gains D="5.0" I="0." P="1000." reference="head_roll"/>
+    </controller>
+  </xacro:if>
+</xacro:unless>
 </robot>

Commit message: Added imu in srdf and small real link in model

File: cogimon_srdf/srdf/cogimon.srdf.xacro (robot description, xacro)
@@ -16,4 +16,7 @@
     <joint name="r_leg_ft_joint"/>
 </xacro:if>
+</group>
+<group name="imu_sensors">
+     <link name="imu_link"/>
 </group>
 <xacro:if value="${COGIMON_LEFT_LEG}">

File: cogimon_urdf/urdf/cogimon_base.urdf.xacro (robot description, xacro)
@@ -43,8 +43,14 @@
 <link name="imu_link">
     <inertial>
-      <origin xyz="0 0 0" rpy="0.0 0.0 0.0"/>
-      <mass value="0"/>
-      <inertia ixx="0"  ixy="0"  ixz="0" iyy="0" iyz="0" izz="0" />
+      <mass value="0.01"/>
+      <origin xyz="0 0 0"/>
+      <inertia ixx="1.0E-6" ixy="0" ixz="0" iyy="1.0E-6" iyz="0" izz="1.0E-6"/>
     </inertial>
+    <visual>
+      <origin rpy="0 0 0" xyz="0 0 0"/>
+      <geometry>
+        <box size="0.01 0.01 0.01"/>
+      </geometry>
+    </visual>
 </link>
 <!-- SELECTION OF KINEMATICS CHAINS IS HANDLED INSIDE THE FILES -->

Commit message: Added hands in srdf

File: cogimon_srdf/srdf/cogimon.srdf.xacro (robot description, xacro)
@@ -9,4 +9,12 @@
         <link name="Waist"/>
     </group>
+<group name="hands">
+<xacro:if value="${COGIMON_RIGHT_ARM}">
+      <joint name="r_wrist_joint"/>
+</xacro:if>
+<xacro:if value="${COGIMON_LEFT_ARM}">
+      <joint name="l_wrist_joint"/>
+</xacro:if>
+</group>
 <group name="force_torque_sensors">
 <xacro:if value="${COGIMON_LEFT_LEG}">

Commit message: Added ref frame for ft sensors. Added ft_sensors in simulation. Added ft sesnors in srdf

File: cogimon_srdf/srdf/cogimon.srdf.xacro (robot description, xacro)
@@ -18,4 +18,10 @@
 </group>
 <group name="force_torque_sensors">
+<xacro:if value="${COGIMON_LEFT_ARM}">
+    <joint name="l_arm_ft_joint"/>
+</xacro:if>
+<xacro:if value="${COGIMON_RIGHT_ARM}">
+    <joint name="r_arm_ft_joint"/>
+</xacro:if>
 <xacro:if value="${COGIMON_LEFT_LEG}">
     <joint name="l_leg_ft_joint"/>

File: cogimon_urdf/urdf/cogimon.urdf.xacro (robot description, xacro)
@@ -29,4 +29,5 @@
 <!-- ************ REF FRAMES **************** -->
 <xacro:include filename="$(find cogimon_urdf)/urdf/parts/feet_reference_frames.urdf.xacro"/>
+<xacro:include filename="$(find cogimon_urdf)/urdf/parts/arms_reference_frames.urdf.xacro"/>
 <xacro:if value="${COGIMON_FLOATING_BASE}" >
 <link name="world"/>

File: cogimon_urdf/urdf/gazebo/force_torque.gazebo.xacro (robot description, xacro)
@@ -7,4 +7,32 @@
 -->
 <robot xmlns:xacro="http:/ros.org/wiki/xacro">
+<xacro:if value="${COGIMON_LEFT_ARM}" >
+       <gazebo reference="LWrMot3">
+              <sensor type="force_torque" name="l_arm_ft">
+                     <force_torque>
+                       <frame>sensor</frame>
+                       <measure_direction>child_to_parent</measure_direction>
+                     </force_torque>
+		       <always_on>true</always_on>
+		       <visualize>true</visualize>
+		       <update_rate>1000</update_rate>
+		       <pose>0 0 -0.02 0 0 0</pose> <!-- check! -->
+	       </sensor>
+       </gazebo>
+</xacro:if>
+<xacro:if value="${COGIMON_RIGHT_ARM}" >
+       <gazebo reference="RWrMot3">
+	       <sensor type="force_torque" name="r_arm_ft">
+                     <force_torque>
+                       <frame>sensor</frame>
+                       <measure_direction>child_to_parent</measure_direction>
+                     </force_torque>
+		       <always_on>true</always_on>
+		       <visualize>true</visualize>
+		       <update_rate>1000</update_rate>
+		       <pose>0 0 -0.02 0 0 0</pose> <!-- check! -->
+              </sensor>
+       </gazebo>
+</xacro:if>
 <xacro:if value="${COGIMON_LEFT_LEG}" >
        <gazebo reference="LAnkleRoll">

Commit message: fixed name

File: cogimon_srdf/srdf/cogimon.srdf.xacro (robot description, xacro)
@@ -111,5 +111,5 @@
         <joint name="RAnkleRoll" value="0.0"/>
         <joint name="WaistLat" value="0.0"/>
-	<joint name="Waistyaw" value="0.0"/>
+	<joint name="WaistYaw" value="0.0"/>
         <joint name="RShSag" value="0.0"/>
         <joint name="RShLat" value="0.0"/>
