Commit message: changed homing in srdf

File: cogimon_srdf/srdf/cogimon.srdf.xacro (robot description, xacro)
@@ -98,32 +98,32 @@
 <xacro:if value="${COGIMON_XBOT_GAZEBO}">
 <group_state name="home" group="chains">
-        <joint name="LHipLat" value="0.0"/>
-        <joint name="LHipSag" value="0.0"/>
-        <joint name="LHipYaw" value="0.0"/>
-        <joint name="LKneePitch" value="0.0"/>
-        <joint name="LAnklePitch" value="0.0"/>
-        <joint name="LAnkleRoll" value="0.0"/>
-        <joint name="RHipLat" value="0.0"/>
-        <joint name="RHipSag" value="0.0"/>
-        <joint name="RHipYaw" value="0.0"/>
-        <joint name="RKneePitch" value="0.0"/>
-        <joint name="RAnklePitch" value="0.0"/>
-        <joint name="RAnkleRoll" value="0.0"/>
-        <joint name="WaistLat" value="0.0"/>
-	<joint name="WaistYaw" value="0.0"/>
-        <joint name="RShSag" value="0.0"/>
-        <joint name="RShLat" value="0.0"/>
-        <joint name="RShYaw" value="0.0"/>
-        <joint name="RElbj" value="0.0"/>
-        <joint name="RForearmPlate" value="0.0"/>
-        <joint name="RWrj1" value="0.0"/>
-        <joint name="RWrj2" value="0.0"/>
-        <joint name="LShSag" value="0.0"/>
-        <joint name="LShLat" value="0.0"/>
-        <joint name="LShYaw" value="0.0"/>
-        <joint name="LElbj" value="0.0"/>
-        <joint name="LForearmPlate" value="0.0"/>
-        <joint name="LWrj1" value="0.0"/>
-        <joint name="LWrj2" value="0.0"/>
+        <joint name="WaistYaw" value="0.0"/>
+    <joint name="WaistLat" value="0.0"/>
+    <joint name="RShSag" value="0.959931"/>
+    <joint name="RShLat" value="-0.007266"/>
+    <joint name="RShYaw" value="-0.0"/>
+    <joint name="RElbj" value="-1.919862"/>
+    <joint name="RForearmPlate" value="0.0"/>
+    <joint name="RWrj1" value="-0.523599"/>
+    <joint name="RWrj2" value="-0.0"/>
+    <joint name="LShSag" value="0.959931"/>
+    <joint name="LShLat" value="0.007266"/>
+    <joint name="LShYaw" value="-0.0"/>
+    <joint name="LElbj" value="-1.919862"/>
+    <joint name="LForearmPlate" value="0.0"/>
+    <joint name="LWrj1" value="-0.523599"/>
+    <joint name="LWrj2" value="-0.0"/>
+    <joint name="RHipLat" value="0.0"/>
+    <joint name="RHipSag" value="-0.363826"/>
+    <joint name="RHipYaw" value="0.0"/>
+    <joint name="RKneePitch" value="0.731245"/>
+    <joint name="RAnklePitch" value="-0.307420"/>
+    <joint name="RAnkleRoll" value="-0.0"/>
+    <joint name="LHipLat" value="-0.0"/>
+    <joint name="LHipSag" value="-0.363826"/>
+    <joint name="LHipYaw" value="0.0"/>
+    <joint name="LKneePitch" value="0.731245"/>
+    <joint name="LAnklePitch" value="-0.307420"/>
+    <joint name="LAnkleRoll" value="0.0"/>
 	<xacro:unless value="${COGIMON_LASER_FIXED}">
     	<xacro:if value="${COGIMON_HEAD}">

Commit message: added head camera and pitch joint

File: cogimon_srdf/srdf/cogimon.srdf.xacro (robot description, xacro)
@@ -67,5 +67,5 @@
     <xacro:if value="${COGIMON_HEAD}">
         <group name="neck">
-            <chain base_link="Neck" tip_link="HeadHokuyo"/>
+            <chain base_link="DWYTorso" tip_link="HeadHokuyo"/>
         </group>
     </xacro:if>

File: cogimon_urdf/urdf/cogimon_config.urdf.xacro (robot description, xacro)
@@ -3,10 +3,11 @@
 <xacro:property name="model_name" value="IIT COGIMON" />
 <xacro:property name="model_version" value="0.1" />
+<xacro:arg name="laser_fixed" default="true"/>
 <!-- ************SELECT PARTS*************-->
 <!-- *************************************-->
 <xacro:property name="COGIMON_HEAD" value="true" />
 <xacro:property name="COGIMON_TORSO" value="true" />
-<xacro:property name="COGIMON_LEFT_ARM" value="true" />
-<xacro:property name="COGIMON_RIGHT_ARM" value="true" />
+<xacro:property name="COGIMON_LEFT_ARM" value="false" />
+<xacro:property name="COGIMON_RIGHT_ARM" value="false" />
 <xacro:property name="COGIMON_LEFT_LEG" value="true" />
 <xacro:property name="COGIMON_RIGHT_LEG" value="true" />
@@ -21,5 +22,5 @@
 -->
 <!-- *************************************-->
-<xacro:property name="COGIMON_LASER_FIXED" value="true" />
+<xacro:property name="COGIMON_LASER_FIXED" value="$(arg laser_fixed)" />
 <!-- ************COGIMON_PENNACCHIO*******-->
 <!--

File: cogimon_urdf/urdf/config/cogimon.urdf.xacro (robot description, xacro)
@@ -21,5 +21,5 @@
 -->
 <!-- *************************************-->
-<xacro:property name="COGIMON_LASER_FIXED" value="true" />
+<xacro:property name="COGIMON_LASER_FIXED" value="false" />
 <!-- ************COGIMON_PENNACCHIO*******-->
 <!--

File: cogimon_urdf/urdf/parts/head.urdf.xacro (robot description, xacro)
@@ -48,8 +48,32 @@
     <child link="HeadHokuyo"/>
     <origin xyz="0.0853 0.0 0.1506" rpy="0 0.3491 0" />
-    <axis xyz="1 0 0" />
-    <limit velocity="6.283" effort="20" lower="-100." upper="100." />
+    <axis xyz="0 1 0" />
+    <limit velocity="6.283" effort="20" lower="-3.14" upper="3.14" />
     <dynamics friction="0" damping="3.0"/>
   </joint>
+  <xacro:include filename="$(find realsense_gazebo_description)/urdf/_d435i.urdf.xacro" />
+  <xacro:property name="d435_head_origin">
+    <origin xyz="0.13015 0 -0.0125" rpy="0 0 0"/>
+  </xacro:property>
+  <xacro:sensor_d435i parent="HeadHokuyo"
+    name="head_camera"
+    topics_ns="head_camera"
+    enable_pointCloud="true"
+    align_depth="true"
+    unite_imu_method="false"
+    visualize="true"
+    accel_fps="300"
+    gyro_fps="300"
+    depth_width="1280"
+    depth_height="720"
+    depth_fps="90"
+    infra_width="1280"
+    infra_height="720"
+    infra_fps="90"
+    color_width="1280"
+    color_height="720"
+    color_fps="30">
+    <xacro:insert_block name="d435_head_origin" />
+  </xacro:sensor_d435i>
 </xacro:unless>
 <link name="HokuyoLaser"/>
@@ -58,5 +82,5 @@
     <child link="HokuyoLaser"/>
     <origin xyz="${65.2577*mmTom} 0.0 0.0" rpy="0 0 0" />
-  </joint>
+</joint>
 </xacro:if>
 </robot>
